File: Hardware/BodyController/BodyController_03/Connectors.sch (KiCad schematic (older format))
At the start: 22 parts, among them J1 7796, J10 Conn_01x01, J11 Conn_01x01, J12 Conn_01x01, J13 Conn_01x01, J14 TEST_1P, J15 TEST_1P, J16 TEST_1P, J17 TEST_1P, J18 TEST_1P, J2 Conn_01x14, J3 Conn_02x10_Top_Bottom, J4 Conn_02x10_Top_Bottom, J5 7796, J6 7796, J7 CONN_01X06, J8 USB_OTG, J9 Conn_01x01

Commit message: Added output files
Parts:
- added TP1, TP7: TEST_1P, Measurement_Points:Test_Point_Keystone_5019_Minature, symbol TEST_1P
- renumbered J14 to TP2, J15 to TP3, J16 to TP4, J17 to TP5, J18 to TP6
Connections:
- net GND: now also TP7.1
- new net +12V: TP1.1
Changed lines of the file:
@@
 $EndDescr
 $Comp
-L GND #PWR0122
+L GND #PWR128
 U 1 1 5995D681
 P 2000 2150
-F 0 "#PWR0122" H 2000 1900 50  0001 C CNN
+F 0 "#PWR128" H 2000 1900 50  0001 C CNN
 F 1 "GND" H 2000 2000 50  0000 C CNN
 F 2 "" H 2000 2150 50  0001 C CNN
@@
 $EndComp
 $Comp
-L +BATT #PWR0123
+L +BATT #PWR127
 U 1 1 5995D6C1
 P 2000 1100
-F 0 "#PWR0123" H 2000 950 50  0001 C CNN
+F 0 "#PWR127" H 2000 950 50  0001 C CNN
 F 1 "+BATT" H 2000 1240 50  0000 C CNN
 F 2 "" H 2000 1100 50  0001 C CNN
@@
 $EndComp
 $Comp
-L +3V3 #PWR0124
+L +3V3 #PWR122
 U 1 1 5997230B
 P 650 2950
-F 0 "#PWR0124" H 650 2800 50  0001 C CNN
+F 0 "#PWR122" H 650 2800 50  0001 C CNN
 F 1 "+3V3" H 650 3090 50  0000 C CNN
 F 2 "" H 650 2950 50  0001 C CNN
@@
 $EndComp
 $Comp
-L GND #PWR0125
+L GND #PWR123
 U 1 1 5997232D
 P 650 3150
-F 0 "#PWR0125" H 650 2900 50  0001 C CNN
+F 0 "#PWR123" H 650 2900 50  0001 C CNN
 F 1 "GND" H 650 3000 50  0000 C CNN
 F 2 "" H 650 3150 50  0001 C CNN
@@
 $EndComp
 $Comp
-L PWR_FLAG #FLG0126
+L PWR_FLAG #FLG3
 U 1 1 59980CA4
 P 1650 1150
-F 0 "#FLG0126" H 1650 1225 50  0001 C CNN
+F 0 "#FLG3" H 1650 1225 50  0001 C CNN
 F 1 "PWR_FLAG" H 1650 1300 50  0000 C CNN
 F 2 "" H 1650 1150 50  0001 C CNN
@@
 $EndComp
 $Comp
-L PWR_FLAG #FLG0127
+L PWR_FLAG #FLG4
 U 1 1 59980CC6
 P 1650 2050
-F 0 "#FLG0127" H 1650 2125 50  0001 C CNN
+F 0 "#FLG4" H 1650 2125 50  0001 C CNN
 F 1 "PWR_FLAG" H 1650 2200 50  0000 C CNN
 F 2 "" H 1650 2050 50  0001 C CNN
@@
 $EndComp
 $Comp
-L GND #PWR0128
+L GND #PWR125
 U 1 1 59A82EC9
 P 1550 5650
-F 0 "#PWR0128" H 1550 5400 50  0001 C CNN
+F 0 "#PWR125" H 1550 5400 50  0001 C CNN
 F 1 "GND" H 1550 5500 50  0000 C CNN
 F 2 "" H 1550 5650 50  0001 C CNN
@@
 $EndComp
 $Comp
-L GND #PWR0129
+L GND #PWR129
 U 1 1 5A49F5A7
 P 4800 3500
-F 0 "#PWR0129" H 4800 3250 50  0001 C CNN
+F 0 "#PWR129" H 4800 3250 50  0001 C CNN
 F 1 "GND" H 4800 3350 50  0000 C CNN
 F 2 "" H 4800 3500 50  0001 C CNN
@@
 $EndComp
 $Comp
-L GND #PWR0130
+L GND #PWR130
 U 1 1 5A49F6E5
 P 5850 6900
-F 0 "#PWR0130" H 5850 6650 50  0001 C CNN
+F 0 "#PWR130" H 5850 6650 50  0001 C CNN
 F 1 "GND" H 5850 6750 50  0000 C CNN
 F 2 "" H 5850 6900 50  0001 C CNN
@@
 $EndComp
 $Comp
-L GND #PWR0131
+L GND #PWR131
 U 1 1 5A49F80B
 P 6400 4600
-F 0 "#PWR0131" H 6400 4350 50  0001 C CNN
+F 0 "#PWR131" H 6400 4350 50  0001 C CNN
 F 1 "GND" H 6400 4450 50  0000 C CNN
 F 2 "" H 6400 4600 50  0001 C CNN
@@
 $EndComp
 $Comp
-L +5VP #PWR0132
+L +5VP #PWR132
 U 1 1 5A49F8B9
 P 6400 5100
-F 0 "#PWR0132" H 6400 4950 50  0001 C CNN
+F 0 "#PWR132" H 6400 4950 50  0001 C CNN
 F 1 "+5VP" H 6400 5240 50  0000 C CNN
 F 2 "" H 6400 5100 50  0001 C CNN
@@
 $EndComp
 $Comp
-L GND #PWR0133
+L GND #PWR124
 U 1 1 5A4AD94A
 P 1550 3850
-F 0 "#PWR0133" H 1550 3600 50  0001 C CNN
+F 0 "#PWR124" H 1550 3600 50  0001 C CNN
 F 1 "GND" H 1550 3700 50  0000 C CNN
 F 2 "" H 1550 3850 50  0001 C CNN
@@
 $EndComp
 $Comp
-L GND #PWR0134
+L GND #PWR126
 U 1 1 5A4AD988
 P 1800 3850
-F 0 "#PWR0134" H 1800 3600 50  0001 C CNN
+F 0 "#PWR126" H 1800 3600 50  0001 C CNN
 F 1 "GND" H 1800 3700 50  0000 C CNN
 F 2 "" H 1800 3850 50  0001 C CNN
@@
 $EndComp
 $Comp
-L TEST_1P J18
+L TEST_1P TP6
 U 1 1 5A527FBB
 P 9400 1100
-F 0 "J18" H 9400 1370 50  0000 C CNN
+F 0 "TP6" H 9400 1370 50  0000 C CNN
 F 1 "TEST_1P" H 9400 1300 50  0000 C CNN
 F 2 "Measurement_Points:Test_Point_Keystone_5019_Minature" H 9600 1100 50  0001 C CNN
@@
 $EndComp
 $Comp
-L TEST_1P J17
+L TEST_1P TP5
 U 1 1 5A5280F8
 P 8950 1100
-F 0 "J17" H 8950 1370 50  0000 C CNN
+F 0 "TP5" H 8950 1370 50  0000 C CNN
 F 1 "TEST_1P" H 8950 1300 50  0000 C CNN
 F 2 "Measurement_Points:Test_Point_Keystone_5019_Minature" H 9150 1100 50  0001 C CNN
@@
 $EndComp
 $Comp
-L TEST_1P J16
+L TEST_1P TP4
 U 1 1 5A528147
 P 8500 1100
-F 0 "J16" H 8500 1370 50  0000 C CNN
+F 0 "TP4" H 8500 1370 50  0000 C CNN
 F 1 "TEST_1P" H 8500 1300 50  0000 C CNN
 F 2 "Measurement_Points:Test_Point_Keystone_5019_Minature" H 8700 1100 50  0001 C CNN
@@
 $EndComp
 $Comp
-L TEST_1P J15
+L TEST_1P TP3
 U 1 1 5A5281E7
 P 8050 1100
-F 0 "J15" H 8050 1370 50  0000 C CNN
+F 0 "TP3" H 8050 1370 50  0000 C CNN
 F 1 "TEST_1P" H 8050 1300 50  0000 C CNN
 F 2 "Measurement_Points:Test_Point_Keystone_5019_Minature" H 8250 1100 50  0001 C CNN
@@
 $EndComp
 $Comp
-L TEST_1P J14
+L TEST_1P TP2
 U 1 1 5A528244
 P 7600 1100
-F 0 "J14" H 7600 1370 50  0000 C CNN
+F 0 "TP2" H 7600 1370 50  0000 C CNN
 F 1 "TEST_1P" H 7600 1300 50  0000 C CNN
 F 2 "Measurement_Points:Test_Point_Keystone_5019_Minature" H 7800 1100 50  0001 C CNN
@@
 $EndComp
 $Comp
-L +5VP #PWR0135
+L +5VP #PWR138
 U 1 1 5A52849A
 P 9400 1100
-F 0 "#PWR0135" H 9400 950 50  0001 C CNN
+F 0 "#PWR138" H 9400 950 50  0001 C CNN
 F 1 "+5VP" H 9400 1240 50  0000 C CNN
 F 2 "" H 9400 1100 50  0001 C CNN
@@
 $EndComp
 $Comp
-L +3.3VP #PWR0136
+L +3.3VP #PWR137
 U 1 1 5A528725
 P 8950 1100
-F 0 "#PWR0136" H 9100 1050 50  0001 C CNN
+F 0 "#PWR137" H 9100 1050 50  0001 C CNN
 F 1 "+3.3VP" H 8950 1200 50  0000 C CNN
 F 2 "" H 8950 1100 50  0001 C CNN
@@
 $EndComp
 $Comp
-L +5V #PWR0137
+L +5V #PWR136
 U 1 1 5A528765
 P 8500 1100
-F 0 "#PWR0137" H 8500 950 50  0001 C CNN
+F 0 "#PWR136" H 8500 950 50  0001 C CNN
 F 1 "+5V" H 8500 1240 50  0000 C CNN
 F 2 "" H 8500 1100 50  0001 C CNN
@@
 $EndComp
 $Comp
-L +3.3V #PWR0138
+L +3.3V #PWR135
 U 1 1 5A5287A5
 P 8050 1100
-F 0 "#PWR0138" H 8050 950 50  0001 C CNN
+F 0 "#PWR135" H 8050 950 50  0001 C CNN
 F 1 "+3.3V" H 8050 1240 50  0000 C CNN
 F 2 "" H 8050 1100 50  0001 C CNN
@@
 $EndComp
 $Comp
-L +12P #PWR0139
+L +12P #PWR134
 U 1 1 5A528E69
 P 7600 1100
-F 0 "#PWR0139" H 7600 950 50  0001 C CNN
+F 0 "#PWR134" H 7600 950 50  0001 C CNN
 F 1 "+12P" H 7600 1240 50  0000 C CNN
 F 2 "" H 7600 1100 50  0001 C CNN
@@
 Text GLabel 6800 5100 3    60   Output ~ 0
 PROXIMITY_IN
+$Comp
+L TEST_1P TP1
+U 1 1 5A57BD55
+P 7150 1100
+F 0 "TP1" H 7150 1370 50  0000 C CNN
+F 1 "TEST_1P" H 7150 1300 50  0000 C CNN
+F 2 "Measurement_Points:Test_Point_Keystone_5019_Minature" H 7350 1100 50  0001 C CNN
+F 3 "" H 7350 1100 50  0001 C CNN
+	1    7150 1100
+	-1   0    0    1
+$EndComp
+$Comp
+L +12V #PWR133
+U 1 1 5A57BE42
+P 7150 1100
+F 0 "#PWR133" H 7150 950 50  0001 C CNN
+F 1 "+12V" H 7150 1240 50  0000 C CNN
+F 2 "" H 7150 1100 50  0001 C CNN
+F 3 "" H 7150 1100 50  0001 C CNN
+	1    7150 1100
+	1    0    0    -1
+$EndComp
+$Comp
+L TEST_1P TP7
+U 1 1 5A57C95A
+P 9800 1100
+F 0 "TP7" H 9800 1370 50  0000 C CNN
+F 1 "TEST_1P" H 9800 1300 50  0000 C CNN
+F 2 "Measurement_Points:Test_Point_Keystone_5019_Minature" H 10000 1100 50  0001 C CNN
+F 3 "" H 10000 1100 50  0001 C CNN
+	1    9800 1100
+	-1   0    0    1
+$EndComp
+$Comp
+L GND #PWR139
+U 1 1 5A57CA66
+P 9800 1100
+F 0 "#PWR139" H 9800 850 50  0001 C CNN
+F 1 "GND" H 9800 950 50  0000 C CNN
+F 2 "" H 9800 1100 50  0001 C CNN
+F 3 "" H 9800 1100 50  0001 C CNN
+	1    9800 1100
+	-1   0    0    1
+$EndComp
 $EndSCHEMATC

Commit message: Added resistor values via BOM importer. Changed layout file to add large CAN resistors and buffer to 1.65V Reference
Parts:
- R109, R110: PartNumber (none) -> AC0603FR-07100RL
Changed lines of the file:
@@
 EESchema Schematic File Version 2
+LIBS:BodyController_03-rescue
 LIBS:power
 LIBS:device
@@
 $EndDescr
 $Comp
-L GND #PWR128
+L GND #PWR0126
 U 1 1 5995D681
 P 2000 2150
-F 0 "#PWR128" H 2000 1900 50  0001 C CNN
+F 0 "#PWR0126" H 2000 1900 50  0001 C CNN
 F 1 "GND" H 2000 2000 50  0000 C CNN
 F 2 "" H 2000 2150 50  0001 C CNN
@@
 $EndComp
 $Comp
-L +BATT #PWR127
+L +BATT #PWR0127
 U 1 1 5995D6C1
 P 2000 1100
-F 0 "#PWR127" H 2000 950 50  0001 C CNN
+F 0 "#PWR0127" H 2000 950 50  0001 C CNN
 F 1 "+BATT" H 2000 1240 50  0000 C CNN
 F 2 "" H 2000 1100 50  0001 C CNN
@@
 $EndComp
 $Comp
-L +3V3 #PWR122
+L +3V3 #PWR0128
 U 1 1 5997230B
 P 650 2950
-F 0 "#PWR122" H 650 2800 50  0001 C CNN
+F 0 "#PWR0128" H 650 2800 50  0001 C CNN
 F 1 "+3V3" H 650 3090 50  0000 C CNN
 F 2 "" H 650 2950 50  0001 C CNN
@@
 $EndComp
 $Comp
-L GND #PWR123
+L GND #PWR0129
 U 1 1 5997232D
 P 650 3150
-F 0 "#PWR123" H 650 2900 50  0001 C CNN
+F 0 "#PWR0129" H 650 2900 50  0001 C CNN
 F 1 "GND" H 650 3000 50  0000 C CNN
 F 2 "" H 650 3150 50  0001 C CNN
@@
 $EndComp
 $Comp
-L PWR_FLAG #FLG3
+L PWR_FLAG #FLG0130
 U 1 1 59980CA4
 P 1650 1150
-F 0 "#FLG3" H 1650 1225 50  0001 C CNN
+F 0 "#FLG0130" H 1650 1225 50  0001 C CNN
 F 1 "PWR_FLAG" H 1650 1300 50  0000 C CNN
 F 2 "" H 1650 1150 50  0001 C CNN
@@
 $EndComp
 $Comp
-L PWR_FLAG #FLG4
+L PWR_FLAG #FLG0131
 U 1 1 59980CC6
 P 1650 2050
-F 0 "#FLG4" H 1650 2125 50  0001 C CNN
+F 0 "#FLG0131" H 1650 2125 50  0001 C CNN
 F 1 "PWR_FLAG" H 1650 2200 50  0000 C CNN
 F 2 "" H 1650 2050 50  0001 C CNN
@@
 $EndComp
 $Comp
-L GND #PWR125
+L GND #PWR0132
 U 1 1 59A82EC9
 P 1550 5650
-F 0 "#PWR125" H 1550 5400 50  0001 C CNN
+F 0 "#PWR0132" H 1550 5400 50  0001 C CNN
 F 1 "GND" H 1550 5500 50  0000 C CNN
 F 2 "" H 1550 5650 50  0001 C CNN
@@
 $EndComp
 $Comp
-L GND #PWR129
+L GND #PWR0133
 U 1 1 5A49F5A7
 P 4800 3500
-F 0 "#PWR129" H 4800 3250 50  0001 C CNN
+F 0 "#PWR0133" H 4800 3250 50  0001 C CNN
 F 1 "GND" H 4800 3350 50  0000 C CNN
 F 2 "" H 4800 3500 50  0001 C CNN
@@
 $EndComp
 $Comp
-L GND #PWR130
+L GND #PWR0134
 U 1 1 5A49F6E5
 P 5850 6900
-F 0 "#PWR130" H 5850 6650 50  0001 C CNN
+F 0 "#PWR0134" H 5850 6650 50  0001 C CNN
 F 1 "GND" H 5850 6750 50  0000 C CNN
 F 2 "" H 5850 6900 50  0001 C CNN
@@
 $EndComp
 $Comp
-L GND #PWR131
+L GND #PWR0135
 U 1 1 5A49F80B
 P 6400 4600
-F 0 "#PWR131" H 6400 4350 50  0001 C CNN
+F 0 "#PWR0135" H 6400 4350 50  0001 C CNN
 F 1 "GND" H 6400 4450 50  0000 C CNN
 F 2 "" H 6400 4600 50  0001 C CNN
@@
 $EndComp
 $Comp
-L +5VP #PWR132
+L +5VP #PWR0136
 U 1 1 5A49F8B9
 P 6400 5100
-F 0 "#PWR132" H 6400 4950 50  0001 C CNN
+F 0 "#PWR0136" H 6400 4950 50  0001 C CNN
 F 1 "+5VP" H 6400 5240 50  0000 C CNN
 F 2 "" H 6400 5100 50  0001 C CNN
@@
 F 1 "100R" V 1600 3200 50  0000 C CNN
 F 2 "Resistors_SMD:R_0603" V 1530 3200 50  0001 C CNN
-F 3 "" H 1600 3200 50  0001 C CNN
+F 3 "http://www.yageo.com/NewPortal/yageodocoutput?fileName=/pdf/R-Chip/PYu-AC_51_RoHS_L_6.pdf" H 1600 3200 50  0001 C CNN
+F 4 "AC0603FR-07100RL" H 0   0   50  0001 C CNN "PartNumber"
 	1    1600 3200
 	0    1    1    0
@@
 F 1 "100R" V 1350 3300 50  0000 C CNN
 F 2 "Resistors_SMD:R_0603" V 1280 3300 50  0001 C CNN
-F 3 "" H 1350 3300 50  0001 C CNN
+F 3 "http://www.yageo.com/NewPortal/yageodocoutput?fileName=/pdf/R-Chip/PYu-AC_51_RoHS_L_6.pdf" H 1350 3300 50  0001 C CNN
+F 4 "AC0603FR-07100RL" H 0   0   50  0001 C CNN "PartNumber"
 	1    1350 3300
 	0    1    1    0
@@
 $EndComp
 $Comp
-L GND #PWR124
+L GND #PWR0137
 U 1 1 5A4AD94A
 P 1550 3850
-F 0 "#PWR124" H 1550 3600 50  0001 C CNN
+F 0 "#PWR0137" H 1550 3600 50  0001 C CNN
 F 1 "GND" H 1550 3700 50  0000 C CNN
 F 2 "" H 1550 3850 50  0001 C CNN
@@
 $EndComp
 $Comp
-L GND #PWR126
+L GND #PWR0138
 U 1 1 5A4AD988
 P 1800 3850
-F 0 "#PWR126" H 1800 3600 50  0001 C CNN
+F 0 "#PWR0138" H 1800 3600 50  0001 C CNN
 F 1 "GND" H 1800 3700 50  0000 C CNN
 F 2 "" H 1800 3850 50  0001 C CNN
@@
 $EndComp
 $Comp
-L +5VP #PWR138
+L +5VP #PWR0139
 U 1 1 5A52849A
 P 9400 1100
-F 0 "#PWR138" H 9400 950 50  0001 C CNN
+F 0 "#PWR0139" H 9400 950 50  0001 C CNN
 F 1 "+5VP" H 9400 1240 50  0000 C CNN
 F 2 "" H 9400 1100 50  0001 C CNN
@@
 $EndComp
 $Comp
-L +3.3VP #PWR137
+L +3.3VP #PWR0140
 U 1 1 5A528725
 P 8950 1100
-F 0 "#PWR137" H 9100 1050 50  0001 C CNN
+F 0 "#PWR0140" H 9100 1050 50  0001 C CNN
 F 1 "+3.3VP" H 8950 1200 50  0000 C CNN
 F 2 "" H 8950 1100 50  0001 C CNN
@@
 $EndComp
 $Comp
-L +5V #PWR136
+L +5V #PWR0141
 U 1 1 5A528765
 P 8500 1100
-F 0 "#PWR136" H 8500 950 50  0001 C CNN
+F 0 "#PWR0141" H 8500 950 50  0001 C CNN
 F 1 "+5V" H 8500 1240 50  0000 C CNN
 F 2 "" H 8500 1100 50  0001 C CNN
@@
 $EndComp
 $Comp
-L +3.3V #PWR135
+L +3.3V #PWR0142
 U 1 1 5A5287A5
 P 8050 1100
-F 0 "#PWR135" H 8050 950 50  0001 C CNN
+F 0 "#PWR0142" H 8050 950 50  0001 C CNN
 F 1 "+3.3V" H 8050 1240 50  0000 C CNN
 F 2 "" H 8050 1100 50  0001 C CNN
@@
 $EndComp
 $Comp
-L +12P #PWR134
+L +12P #PWR0143
 U 1 1 5A528E69
 P 7600 1100
-F 0 "#PWR134" H 7600 950 50  0001 C CNN
+F 0 "#PWR0143" H 7600 950 50  0001 C CNN
 F 1 "+12P" H 7600 1240 50  0000 C CNN
 F 2 "" H 7600 1100 50  0001 C CNN
@@
 	1    7600 1100
 	1    0    0    -1
+$EndComp
+$Comp
+L TEST_1P TP1
+U 1 1 5A57BD55
+P 7150 1100
+F 0 "TP1" H 7150 1370 50  0000 C CNN
+F 1 "TEST_1P" H 7150 1300 50  0000 C CNN
+F 2 "Measurement_Points:Test_Point_Keystone_5019_Minature" H 7350 1100 50  0001 C CNN
+F 3 "" H 7350 1100 50  0001 C CNN
+	1    7150 1100
+	-1   0    0    1
+$EndComp
+$Comp
+L +12V #PWR0144
+U 1 1 5A57BE42
+P 7150 1100
+F 0 "#PWR0144" H 7150 950 50  0001 C CNN
+F 1 "+12V" H 7150 1240 50  0000 C CNN
+F 2 "" H 7150 1100 50  0001 C CNN
+F 3 "" H 7150 1100 50  0001 C CNN
+	1    7150 1100
+	1    0    0    -1
+$EndComp
+$Comp
+L TEST_1P TP7
+U 1 1 5A57C95A
+P 9800 1100
+F 0 "TP7" H 9800 1370 50  0000 C CNN
+F 1 "TEST_1P" H 9800 1300 50  0000 C CNN
+F 2 "Measurement_Points:Test_Point_Keystone_5019_Minature" H 10000 1100 50  0001 C CNN
+F 3 "" H 10000 1100 50  0001 C CNN
+	1    9800 1100
+	-1   0    0    1
+$EndComp
+$Comp
+L GND #PWR0145
+U 1 1 5A57CA66
+P 9800 1100
+F 0 "#PWR0145" H 9800 850 50  0001 C CNN
+F 1 "GND" H 9800 950 50  0000 C CNN
+F 2 "" H 9800 1100 50  0001 C CNN
+F 3 "" H 9800 1100 50  0001 C CNN
+	1    9800 1100
+	-1   0    0    1
 $EndComp
 Text GLabel 4200 4600 1    59   Input ~ 0
@@
 Text GLabel 7300 5100 3    60   Input ~ 0
 DAC_OUT_2
+Text GLabel 6900 5100 3    60   Output ~ 0
+PILOT_IN
+Text GLabel 6800 5100 3    60   Output ~ 0
+PROXIMITY_IN
 Wire Wire Line
 	2000 2050 2000 2150
@@
 Wire Wire Line
 	1800 3500 1800 3200
+Wire Wire Line
+	6600 4600 6600 4450
+Wire Wire Line
+	6600 4450 6400 4450
+Wire Wire Line
+	6400 4450 6400 4600
 Connection ~ 1650 1150
 Connection ~ 1650 2050
@@
 NoConn ~ 10350 1750
 NoConn ~ 10350 2050
-Wire Wire Line
-	6600 4600 6600 4450
-Wire Wire Line
-	6600 4450 6400 4450
-Wire Wire Line
-	6400 4450 6400 4600
-Text GLabel 6900 5100 3    60   Output ~ 0
-PILOT_IN
-Text GLabel 6800 5100 3    60   Output ~ 0
-PROXIMITY_IN
-$Comp
-L TEST_1P TP1
-U 1 1 5A57BD55
-P 7150 1100
-F 0 "TP1" H 7150 1370 50  0000 C CNN
-F 1 "TEST_1P" H 7150 1300 50  0000 C CNN
-F 2 "Measurement_Points:Test_Point_Keystone_5019_Minature" H 7350 1100 50  0001 C CNN
-F 3 "" H 7350 1100 50  0001 C CNN
-	1    7150 1100
-	-1   0    0    1
-$EndComp
-$Comp
-L +12V #PWR133
-U 1 1 5A57BE42
-P 7150 1100
-F 0 "#PWR133" H 7150 950 50  0001 C CNN
-F 1 "+12V" H 7150 1240 50  0000 C CNN
-F 2 "" H 7150 1100 50  0001 C CNN
-F 3 "" H 7150 1100 50  0001 C CNN
-	1    7150 1100
-	1    0    0    -1
-$EndComp
-$Comp
-L TEST_1P TP7
-U 1 1 5A57C95A
-P 9800 1100
-F 0 "TP7" H 9800 1370 50  0000 C CNN
-F 1 "TEST_1P" H 9800 1300 50  0000 C CNN
-F 2 "Measurement_Points:Test_Point_Keystone_5019_Minature" H 10000 1100 50  0001 C CNN
-F 3 "" H 10000 1100 50  0001 C CNN
-	1    9800 1100
-	-1   0    0    1
-$EndComp
-$Comp
-L GND #PWR139
-U 1 1 5A57CA66
-P 9800 1100
-F 0 "#PWR139" H 9800 850 50  0001 C CNN
-F 1 "GND" H 9800 950 50  0000 C CNN
-F 2 "" H 9800 1100 50  0001 C CNN
-F 3 "" H 9800 1100 50  0001 C CNN
-	1    9800 1100
-	-1   0    0    1
-$EndComp
 $EndSCHEMATC
