File: Hardware/BodyController/BodyController_01/Connectors.sch (KiCad schematic (older format))
At the start: 25 parts, among them J1 7796, J10 Conn_01x01, J11 Conn_01x01, J12 Conn_01x01, J13 Conn_01x01, J2 Conn_01x14, J3 Conn_02x10_Top_Bottom, J4 Conn_02x10_Top_Bottom, J5 7796, J6 7796, J7 CONN_01X06, J8 USB_OTG, J9 Conn_01x01

Commit message: New bring-up code for Body Controller
Parts:
- added TP8: TEST_1P, Measurement_Points:Test_Point_Keystone_5019_Minature, symbol TEST_1P
- J2: MPN (none) -> 34772-0140; populate n -> y
- J3: MPN (none) -> 34690-0201; populate n -> y
- J4: MPN (none) -> 34690-0203; populate n -> y
Connections:
- net labels added: DEBUG_PIN
- wire segments 43 -> 45
Changed lines of the file:
@@
 F 2 "Footprints:34772-0140" H 3800 4800 50  0001 C CNN
 F 3 "" H 3800 4800 50  0001 C CNN
-F 4 "n" H 3800 5600 50  0001 C CNN "populate"
+F 4 "y" H 3800 5600 50  0001 C CNN "populate"
+F 5 "34772-0140" H 3800 4800 60  0001 C CNN "MPN"
 	1    3800 4800
 	0    -1   1    0
@@
 F 2 "Footprints:34690-0200" H 5550 4800 50  0001 C CNN
 F 3 "" H 5550 4800 50  0001 C CNN
-F 4 "n" H 5600 5400 50  0001 C CNN "populate"
+F 4 "y" H 5600 5400 50  0001 C CNN "populate"
+F 5 "34690-0201" H 5550 4800 60  0001 C CNN "MPN"
 	1    5550 4800
 	0    -1   1    0
@@
 F 2 "Footprints:34690-0200" H 7000 4800 50  0001 C CNN
 F 3 "" H 7000 4800 50  0001 C CNN
-F 4 "n" H 7050 5400 50  0001 C CNN "populate"
+F 4 "y" H 7050 5400 50  0001 C CNN "populate"
+F 5 "34690-0203" H 7000 4800 60  0001 C CNN "MPN"
 	1    7000 4800
 	0    -1   1    0
@@
 F 3 "" H 9800 1100 50  0001 C CNN
 	1    9800 1100
+	-1   0    0    1
+$EndComp
+$Comp
+L GND #PWR0145
+U 1 1 5A6303D8
+P 10300 2450
+F 0 "#PWR0145" H 10300 2200 50  0001 C CNN
+F 1 "GND" H 10300 2300 50  0000 C CNN
+F 2 "" H 10300 2450 50  0001 C CNN
+F 3 "" H 10300 2450 50  0001 C CNN
+	1    10300 2450
+	1    0    0    -1
+$EndComp
+$Comp
+L GND #PWR0146
+U 1 1 5A6309A6
+P 1300 6050
+F 0 "#PWR0146" H 1300 5800 50  0001 C CNN
+F 1 "GND" H 1300 5900 50  0000 C CNN
+F 2 "" H 1300 6050 50  0001 C CNN
+F 3 "" H 1300 6050 50  0001 C CNN
+	1    1300 6050
+	1    0    0    -1
+$EndComp
+$Comp
+L C C137
+U 1 1 5A630A73
+P 1300 5850
+F 0 "C137" H 1325 5950 50  0000 L CNN
+F 1 "10nF" H 1325 5750 50  0000 L CNN
+F 2 "Capacitors_SMD:C_0603" H 1338 5700 50  0001 C CNN
+F 3 "https://product.tdk.com/info/en/documents/chara_sheet/CGA3E2X7R1H103K080AA.pdf" H 1300 5850 50  0001 C CNN
+F 4 "CGA3E2X7R1H103K080AA" H 1325 6050 50  0001 C CNN "MPN"
+F 5 "y" H 1325 6050 50  0001 C CNN "populate"
+	1    1300 5850
+	1    0    0    -1
+$EndComp
+$Comp
+L TEST_1P TP8
+U 1 1 5A7E886F
+P 6700 1100
+F 0 "TP8" H 6700 1370 50  0000 C CNN
+F 1 "TEST_1P" H 6700 1300 50  0000 C CNN
+F 2 "Measurement_Points:Test_Point_Keystone_5019_Minature" H 6900 1100 50  0001 C CNN
+F 3 "http://www.keyelco.com/product-pdf.cfm?p=1353" H 6900 1100 50  0001 C CNN
+F 4 "5015" H 6700 1470 50  0001 C CNN "MPN"
+F 5 "y" H 6700 1470 50  0001 C CNN "populate"
+	1    6700 1100
 	-1   0    0    1
 $EndComp
@@
 Text GLabel 6900 5100 3    60   Output ~ 0
 PROXIMITY
+Text GLabel 6500 1050 0    60   BiDi ~ 0
+DEBUG_PIN
 Wire Wire Line
 	2000 2050 2000 2150
@@
 Wire Wire Line
 	6400 4450 6400 4600
+Wire Wire Line
+	10300 850  10300 2450
+Wire Wire Line
+	10300 850  10350 850
+Wire Wire Line
+	10350 1150 10300 1150
+Wire Wire Line
+	10350 1450 10300 1450
+Wire Wire Line
+	10350 1750 10300 1750
+Wire Wire Line
+	10350 2050 10300 2050
+Wire Wire Line
+	1600 5600 1600 5650
+Wire Wire Line
+	1500 5600 1500 5650
+Wire Wire Line
+	1500 5650 1300 5650
+Wire Wire Line
+	1300 6000 1300 6050
+Wire Wire Line
+	1300 5650 1300 5700
+Wire Wire Line
+	6500 1050 6700 1050
+Wire Wire Line
+	6700 1050 6700 1100
 Connection ~ 1650 1150
 Connection ~ 1650 2050
@@
 Connection ~ 1550 3300
 Connection ~ 1800 3200
+Connection ~ 10300 1150
+Connection ~ 10300 1450
+Connection ~ 10300 1750
+Connection ~ 10300 2050
 NoConn ~ 1900 3400
 NoConn ~ 1900 5400
-$Comp
-L GND #PWR0145
-U 1 1 5A6303D8
-P 10300 2450
-F 0 "#PWR0145" H 10300 2200 50  0001 C CNN
-F 1 "GND" H 10300 2300 50  0000 C CNN
-F 2 "" H 10300 2450 50  0001 C CNN
-F 3 "" H 10300 2450 50  0001 C CNN
-	1    10300 2450
-	1    0    0    -1
-$EndComp
-Wire Wire Line
-	10300 850  10300 2450
-Wire Wire Line
-	10300 850  10350 850
-Wire Wire Line
-	10350 1150 10300 1150
-Connection ~ 10300 1150
-Wire Wire Line
-	10350 1450 10300 1450
-Connection ~ 10300 1450
-Wire Wire Line
-	10350 1750 10300 1750
-Connection ~ 10300 1750
-Wire Wire Line
-	10350 2050 10300 2050
-Connection ~ 10300 2050
-Wire Wire Line
-	1600 5600 1600 5650
-$Comp
-L GND #PWR0146
-U 1 1 5A6309A6
-P 1300 6050
-F 0 "#PWR0146" H 1300 5800 50  0001 C CNN
-F 1 "GND" H 1300 5900 50  0000 C CNN
-F 2 "" H 1300 6050 50  0001 C CNN
-F 3 "" H 1300 6050 50  0001 C CNN
-	1    1300 6050
-	1    0    0    -1
-$EndComp
-$Comp
-L C C137
-U 1 1 5A630A73
-P 1300 5850
-F 0 "C137" H 1325 5950 50  0000 L CNN
-F 1 "10nF" H 1325 5750 50  0000 L CNN
-F 2 "Capacitors_SMD:C_0603" H 1338 5700 50  0001 C CNN
-F 3 "https://product.tdk.com/info/en/documents/chara_sheet/CGA3E2X7R1H103K080AA.pdf" H 1300 5850 50  0001 C CNN
-F 4 "CGA3E2X7R1H103K080AA" H 1325 6050 50  0001 C CNN "MPN"
-F 5 "y" H 1325 6050 50  0001 C CNN "populate"
-	1    1300 5850
-	1    0    0    -1
-$EndComp
-Wire Wire Line
-	1500 5600 1500 5650
-Wire Wire Line
-	1500 5650 1300 5650
-Wire Wire Line
-	1300 6000 1300 6050
-Wire Wire Line
-	1300 5650 1300 5700
 $EndSCHEMATC

Commit message: too much work to specify all. New Scheduler, new bootloader, added new Hardware projects, updated code for bringup, COnverted kicad files to new version.
Parts:
- C114, C115, C137: symbol C -> BodyController_01-rescue:C-RESCUE-BodyController_01
- J1, J5, J6: symbol 7796 -> BodyController_01-rescue:7796-RESCUE-BodyController_01
- J10, J11, J12, J13, J9: symbol Conn_01x01 -> BodyController_01-rescue:Conn_01x01-RESCUE-BodyController_01
- J2: symbol Conn_01x14 -> BodyController_01-rescue:Conn_01x14-RESCUE-BodyController_01
- J3, J4: symbol Conn_02x10_Top_Bottom -> BodyController_01-rescue:Conn_02x10_Top_Bottom-RESCUE-BodyController_01
- J7: symbol CONN_01X06 -> BodyController_01-rescue:CONN_01X06-RESCUE-BodyController_01
- J8: symbol USB_OTG -> BodyController_01-rescue:USB_OTG-RESCUE-BodyController_01
- R109, R110: symbol R -> BodyController_01-rescue:R-RESCUE-BodyController_01
- TP1, TP2, TP3, TP4, TP5, TP6, TP7, TP8: symbol TEST_1P -> BodyController_01-rescue:TEST_1P-RESCUE-BodyController_01
Changed lines of the file:
@@
-EESchema Schematic File Version 2
-LIBS:switches
-LIBS:power
-LIBS:device
-LIBS:transistors
-LIBS:conn
-LIBS:linear
-LIBS:regul
-LIBS:74xx
-LIBS:cmos4000
-LIBS:adc-dac
-LIBS:memory
-LIBS:xilinx
-LIBS:microcontrollers
-LIBS:dsp
-LIBS:microchip
-LIBS:analog_switches
-LIBS:motorola
-LIBS:texas
-LIBS:intel
-LIBS:audio
-LIBS:interface
-LIBS:digital-audio
-LIBS:philips
-LIBS:display
-LIBS:cypress
-LIBS:siliconi
-LIBS:opto
-LIBS:atmel
-LIBS:contrib
-LIBS:valves
-LIBS:HSD
-LIBS:micros
-LIBS:ICs
-LIBS:Connectors
-LIBS:microchip_dspic33dsc
+EESchema Schematic File Version 4
 LIBS:BodyController_01-cache
-EELAYER 25 0
+EELAYER 26 0
 EELAYER END
 $Descr A4 11693 8268
@@
 $EndDescr
 $Comp
-L GND #PWR0125
+L BodyController_01-rescue:GND-RESCUE-BodyController_01 #PWR0125
 U 1 1 5995D681
 P 2000 2150
@@
 $EndComp
 $Comp
-L +BATT #PWR0126
+L BodyController_01-rescue:+BATT-RESCUE-BodyController_01 #PWR0126
 U 1 1 5995D6C1
 P 2000 1100
@@
 $EndComp
 $Comp
-L CONN_01X06 J7
+L BodyController_01-rescue:CONN_01X06-RESCUE-BodyController_01 J7
 U 1 1 599715F6
 P 2100 3150
@@
 $EndComp
 $Comp
-L +3V3 #PWR0127
+L BodyController_01-rescue:+3V3-RESCUE-BodyController_01 #PWR0127
 U 1 1 5997230B
 P 650 2950
@@
 $EndComp
 $Comp
-L GND #PWR0128
+L BodyController_01-rescue:GND-RESCUE-BodyController_01 #PWR0128
 U 1 1 5997232D
 P 650 3150
@@
 $EndComp
 $Comp
-L PWR_FLAG #FLG0129
+L BodyController_01-rescue:PWR_FLAG-RESCUE-BodyController_01 #FLG0129
 U 1 1 59980CA4
 P 1650 1150
@@
 $EndComp
 $Comp
-L PWR_FLAG #FLG0130
+L BodyController_01-rescue:PWR_FLAG-RESCUE-BodyController_01 #FLG0130
 U 1 1 59980CC6
 P 1650 2050
@@
 $EndComp
 $Comp
-L USB_OTG J8
+L BodyController_01-rescue:USB_OTG-RESCUE-BodyController_01 J8
 U 1 1 59A8218E
 P 1600 5200
@@
 $EndComp
 $Comp
-L GND #PWR0131
+L BodyController_01-rescue:GND-RESCUE-BodyController_01 #PWR0131
 U 1 1 59A82EC9
 P 1600 5650
@@
 $EndComp
 $Comp
-L Conn_01x14 J2
+L BodyController_01-rescue:Conn_01x14-RESCUE-BodyController_01 J2
 U 1 1 5A30D0E9
 P 3800 4800
@@
 $EndComp
 $Comp
-L Conn_02x10_Top_Bottom J3
+L BodyController_01-rescue:Conn_02x10_Top_Bottom-RESCUE-BodyController_01 J3
 U 1 1 5A314BE2
 P 5550 4800
@@
 $EndComp
 $Comp
-L Conn_02x10_Top_Bottom J4
+L BodyController_01-rescue:Conn_02x10_Top_Bottom-RESCUE-BodyController_01 J4
 U 1 1 5A314C2C
 P 7000 4800
@@
 $EndComp
 $Comp
-L 7796 J1
+L BodyController_01-rescue:7796-RESCUE-BodyController_01 J1
 U 1 1 5A393F4B
 P 1400 1250
@@
 $EndComp
 $Comp
-L 7796 J5
+L BodyController_01-rescue:7796-RESCUE-BodyController_01 J5
 U 1 1 5A394530
 P 1400 1700
@@
 $EndComp
 $Comp
-L 7796 J6
+L BodyController_01-rescue:7796-RESCUE-BodyController_01 J6
 U 1 1 5A39455B
 P 1400 2150
@@
 $EndComp
 $Comp
-L Conn_01x01 J9
+L BodyController_01-rescue:Conn_01x01-RESCUE-BodyController_01 J9
 U 1 1 5A465A33
 P 10550 850
@@
 $EndComp
 $Comp
-L Conn_01x01 J10
+L BodyController_01-rescue:Conn_01x01-RESCUE-BodyController_01 J10
 U 1 1 5A465C82
 P 10550 1150
@@
 $EndComp
 $Comp
-L Conn_01x01 J11
+L BodyController_01-rescue:Conn_01x01-RESCUE-BodyController_01 J11
 U 1 1 5A465CB6
 P 10550 1450
@@
 $EndComp
 $Comp
-L Conn_01x01 J12
+L BodyController_01-rescue:Conn_01x01-RESCUE-BodyController_01 J12
 U 1 1 5A465CE9
 P 10550 1750
@@
 $EndComp
 $Comp
-L Conn_01x01 J13
+L BodyController_01-rescue:Conn_01x01-RESCUE-BodyController_01 J13
 U 1 1 5A4665B9
 P 10550 2050
@@
 $EndComp
 $Comp
-L GND #PWR0132
+L BodyController_01-rescue:GND-RESCUE-BodyController_01 #PWR0132
 U 1 1 5A49F5A7
 P 4800 3500
@@
 $EndComp
 $Comp
-L GND #PWR0133
+L BodyController_01-rescue:GND-RESCUE-BodyController_01 #PWR0133
 U 1 1 5A49F6E5
 P 5850 6900
@@
 $EndComp
 $Comp
-L GND #PWR0134
+L BodyController_01-rescue:GND-RESCUE-BodyController_01 #PWR0134
 U 1 1 5A49F80B
 P 6400 4600
@@
 $EndComp
 $Comp
-L +5VP #PWR0135
+L BodyController_01-rescue:+5VP-RESCUE-BodyController_01 #PWR0135
 U 1 1 5A49F8B9
 P 6400 5100
@@
 $EndComp
 $Comp
-L R R110
+L BodyController_01-rescue:R-RESCUE-BodyController_01 R110
 U 1 1 5A4AD53E
 P 1600 3200
@@
 $EndComp
 $Comp
-L R R109
+L BodyController_01-rescue:R-RESCUE-BodyController_01 R109
 U 1 1 5A4AD59D
 P 1350 3300
@@
 $EndComp
 $Comp
-L C C115
+L BodyController_01-rescue:C-RESCUE-BodyController_01 C115
 U 1 1 5A4AD7E0
 P 1800 3650
@@
 $EndComp
 $Comp
-L C C114
+L BodyController_01-rescue:C-RESCUE-BodyController_01 C114
 U 1 1 5A4AD849
 P 1550 3650
@@
 $EndComp
 $Comp
-L GND #PWR0136
+L BodyController_01-rescue:GND-RESCUE-BodyController_01 #PWR0136
 U 1 1 5A4AD94A
 P 1550 3850
@@
 $EndComp
 $Comp
-L GND #PWR0137
+L BodyController_01-rescue:GND-RESCUE-BodyController_01 #PWR0137
 U 1 1 5A4AD988
 P 1800 3850
@@
 $EndComp
 $Comp
-L TEST_1P TP6
+L BodyController_01-rescue:TEST_1P-RESCUE-BodyController_01 TP6
 U 1 1 5A527FBB
 P 9400 1100
@@
 $EndComp
 $Comp
-L TEST_1P TP5
+L BodyController_01-rescue:TEST_1P-RESCUE-BodyController_01 TP5
 U 1 1 5A5280F8
 P 8950 1100
@@
 $EndComp
 $Comp
-L TEST_1P TP4
+L BodyController_01-rescue:TEST_1P-RESCUE-BodyController_01 TP4
 U 1 1 5A528147
 P 8500 1100
@@
 $EndComp
 $Comp
-L TEST_1P TP3
+L BodyController_01-rescue:TEST_1P-RESCUE-BodyController_01 TP3
 U 1 1 5A5281E7
 P 8050 1100
@@
 $EndComp
 $Comp
-L TEST_1P TP2
+L BodyController_01-rescue:TEST_1P-RESCUE-BodyController_01 TP2
 U 1 1 5A528244
 P 7600 1100
@@
 $EndComp
 $Comp
-L +5VP #PWR0138
+L BodyController_01-rescue:+5VP-RESCUE-BodyController_01 #PWR0138
 U 1 1 5A52849A
 P 9400 1100
@@
 $EndComp
 $Comp
-L +3.3VP #PWR0139
+L BodyController_01-rescue:+3.3VP-RESCUE-BodyController_01 #PWR0139
 U 1 1 5A528725
 P 8950 1100
@@
 $EndComp
 $Comp
-L +5V #PWR0140
+L BodyController_01-rescue:+5V-RESCUE-BodyController_01 #PWR0140
 U 1 1 5A528765
 P 8500 1100
@@
 $EndComp
 $Comp
-L +3.3V #PWR0141
+L BodyController_01-rescue:+3.3V-RESCUE-BodyController_01 #PWR0141
 U 1 1 5A5287A5
 P 8050 1100
@@
 $EndComp
 $Comp
-L +12P #PWR0142
+L BodyController_01-rescue:+12P-RESCUE-BodyController_01 #PWR0142
 U 1 1 5A528E69
 P 7600 1100
@@
 $EndComp
 $Comp
-L TEST_1P TP1
+L BodyController_01-rescue:TEST_1P-RESCUE-BodyController_01 TP1
 U 1 1 5A57BD55
 P 7150 1100
@@
 $EndComp
 $Comp
-L +12V #PWR0143
+L BodyController_01-rescue:+12V-RESCUE-BodyController_01 #PWR0143
 U 1 1 5A57BE42
 P 7150 1100
@@
 $EndComp
 $Comp
-L TEST_1P TP7
+L BodyController_01-rescue:TEST_1P-RESCUE-BodyController_01 TP7
 U 1 1 5A57C95A
 P 9800 1100
@@
 $EndComp
 $Comp
-L GND #PWR0144
+L BodyController_01-rescue:GND-RESCUE-BodyController_01 #PWR0144
 U 1 1 5A57CA66
 P 9800 1100
@@
 $EndComp
 $Comp
-L GND #PWR0145
+L BodyController_01-rescue:GND-RESCUE-BodyController_01 #PWR0145
 U 1 1 5A6303D8
 P 10300 2450
@@
 $EndComp
 $Comp
-L GND #PWR0146
+L BodyController_01-rescue:GND-RESCUE-BodyController_01 #PWR0146
 U 1 1 5A6309A6
 P 1300 6050
@@
 $EndComp
 $Comp
-L C C137
+L BodyController_01-rescue:C-RESCUE-BodyController_01 C137
 U 1 1 5A630A73
 P 1300 5850
@@
 $EndComp
 $Comp
-L TEST_1P TP8
+L BodyController_01-rescue:TEST_1P-RESCUE-BodyController_01 TP8
 U 1 1 5A7E886F
 P 6700 1100
