File: Hardware/BodyController/BodyController_01/HighSideDrivers_2.sch (KiCad schematic (older format))
At the start: 25 parts, among them U11 BTS50202EKAXUMA2

Commit message: New bring-up code for Body Controller
Parts:
- C123: MPN CGA5L1X7R1E106M160AC -> C1206C106M3RACAUTO
Changed lines of the file:
@@
 F 1 "10uF" H 5575 1350 50  0000 L CNN
 F 2 "Capacitors_SMD:C_1206" H 5588 1300 50  0001 C CNN
-F 3 "https://product.tdk.com/info/en/documents/chara_sheet/CGA5L1X7R1E106M160AC.pdf" H 5550 1450 50  0001 C CNN
-F 4 "CGA5L1X7R1E106M160AC" H 5575 1650 50  0001 C CNN "MPN"
+F 3 "https://content.kemet.com/datasheets/KEM_C1023_X7R_AUTO_SMD.pdf" H 5550 1450 50  0001 C CNN
+F 4 "C1206C106M3RACAUTO" H 5575 1650 50  0001 C CNN "MPN"
 F 5 "y" H 5575 1650 50  0001 C CNN "populate"
 	1    5550 1450

Commit message: too much work to specify all. New Scheduler, new bootloader, added new Hardware projects, updated code for bringup, COnverted kicad files to new version.
Parts:
- C123, C129, C130, C38, C39, C40, C41, C62, C63, C65: symbol C -> BodyController_01-rescue:C-RESCUE-BodyController_01
- D18, D19: symbol D -> BodyController_01-rescue:D-RESCUE-BodyController_01
- R121, R123, R20, R21, R22, R55, R62, R63, R64, R65, R97, R98: symbol R -> BodyController_01-rescue:R-RESCUE-BodyController_01
- U11: symbol BTS50202EKAXUMA2 -> BodyController_01-rescue:BTS50202EKAXUMA2-RESCUE-BodyController_01
Changed lines of the file:
@@
-EESchema Schematic File Version 2
-LIBS:switches
-LIBS:power
-LIBS:device
-LIBS:transistors
-LIBS:conn
-LIBS:linear
-LIBS:regul
-LIBS:74xx
-LIBS:cmos4000
-LIBS:adc-dac
-LIBS:memory
-LIBS:xilinx
-LIBS:microcontrollers
-LIBS:dsp
-LIBS:microchip
-LIBS:analog_switches
-LIBS:motorola
-LIBS:texas
-LIBS:intel
-LIBS:audio
-LIBS:interface
-LIBS:digital-audio
-LIBS:philips
-LIBS:display
-LIBS:cypress
-LIBS:siliconi
-LIBS:opto
-LIBS:atmel
-LIBS:contrib
-LIBS:valves
-LIBS:HSD
-LIBS:micros
-LIBS:ICs
-LIBS:Connectors
-LIBS:microchip_dspic33dsc
+EESchema Schematic File Version 4
 LIBS:BodyController_01-cache
-EELAYER 25 0
+EELAYER 26 0
 EELAYER END
 $Descr A4 11693 8268
@@
 $EndDescr
 $Comp
-L C C40
+L BodyController_01-rescue:C-RESCUE-BodyController_01 C40
 U 1 1 59913A6A
 P 9250 1550
@@
 $EndComp
 $Comp
-L C C38
+L BodyController_01-rescue:C-RESCUE-BodyController_01 C38
 U 1 1 59913BA9
 P 8350 1550
@@
 $EndComp
 $Comp
-L R R64
+L BodyController_01-rescue:R-RESCUE-BodyController_01 R64
 U 1 1 59913C10
 P 8800 1350
@@
 $EndComp
 $Comp
-L GND #PWR073
+L BodyController_01-rescue:GND-RESCUE-BodyController_01 #PWR073
 U 1 1 599148E7
 P 8350 1750
@@
 $EndComp
 $Comp
-L GND #PWR074
+L BodyController_01-rescue:GND-RESCUE-BodyController_01 #PWR074
 U 1 1 5991493E
 P 9250 1700
@@
 $EndComp
 $Comp
-L C C41
+L BodyController_01-rescue:C-RESCUE-BodyController_01 C41
 U 1 1 59915478
 P 9300 2650
@@
 $EndComp
 $Comp
-L C C39
+L BodyController_01-rescue:C-RESCUE-BodyController_01 C39
 U 1 1 5991547E
 P 8400 2650
@@
 $EndComp
 $Comp
-L R R65
+L BodyController_01-rescue:R-RESCUE-BodyController_01 R65
 U 1 1 59915484
 P 8850 2450
@@
 $EndComp
 $Comp
-L GND #PWR075
+L BodyController_01-rescue:GND-RESCUE-BodyController_01 #PWR075
 U 1 1 5991548C
 P 8400 2900
@@
 $EndComp
 $Comp
-L GND #PWR076
+L BodyController_01-rescue:GND-RESCUE-BodyController_01 #PWR076
 U 1 1 59915493
 P 9300 2800
@@
 $EndComp
 $Comp
-L R R97
+L BodyController_01-rescue:R-RESCUE-BodyController_01 R97
 U 1 1 59979113
 P 9500 1100
@@
 $EndComp
 $Comp
-L R R98
+L BodyController_01-rescue:R-RESCUE-BodyController_01 R98
 U 1 1 59979189
 P 9500 2250
@@
 $EndComp
 $Comp
-L +3.3VP #PWR077
+L BodyController_01-rescue:+3.3VP-RESCUE-BodyController_01 #PWR077
 U 1 1 599A8FBF
 P 9500 850
@@
 $EndComp
 $Comp
-L +3.3VP #PWR078
+L BodyController_01-rescue:+3.3VP-RESCUE-BodyController_01 #PWR078
 U 1 1 599A901C
 P 9500 2000
@@
 $EndComp
 $Comp
-L C C63
+L BodyController_01-rescue:C-RESCUE-BodyController_01 C63
 U 1 1 599FFA4C
 P 8850 3750
@@
 $EndComp
 $Comp
-L R R121
+L BodyController_01-rescue:R-RESCUE-BodyController_01 R121
 U 1 1 599FFA52
 P 8400 3550
@@
 $EndComp
 $Comp
-L GND #PWR079
+L BodyController_01-rescue:GND-RESCUE-BodyController_01 #PWR079
 U 1 1 599FFA58
 P 8850 3900
@@
 $EndComp
 $Comp
-L C C65
+L BodyController_01-rescue:C-RESCUE-BodyController_01 C65
 U 1 1 599FFCCB
 P 8850 4550
@@
 $EndComp
 $Comp
-L R R123
+L BodyController_01-rescue:R-RESCUE-BodyController_01 R123
 U 1 1 599FFCD1
 P 8400 4350
@@
 $EndComp
 $Comp
-L BTS50202EKAXUMA2 U11
+L BodyController_01-rescue:BTS50202EKAXUMA2-RESCUE-BodyController_01 U11
 U 1 1 59A005A4
 P 4200 2050
@@
 $EndComp
 $Comp
-L GND #PWR080
+L BodyController_01-rescue:GND-RESCUE-BodyController_01 #PWR080
 U 1 1 59A005AA
 P 3400 2800
@@
 $EndComp
 $Comp
-L R R63
+L BodyController_01-rescue:R-RESCUE-BodyController_01 R63
 U 1 1 59A005B0
 P 3100 2350
@@
 $EndComp
 $Comp
-L R R22
+L BodyController_01-rescue:R-RESCUE-BodyController_01 R22
 U 1 1 59A005B6
 P 2800 2150
@@
 $EndComp
 $Comp
-L R R21
+L BodyController_01-rescue:R-RESCUE-BodyController_01 R21
 U 1 1 59A005BC
 P 2800 1950
@@
 $EndComp
 $Comp
-L R R62
+L BodyController_01-rescue:R-RESCUE-BodyController_01 R62
 U 1 1 59A005C2
 P 3100 1850
@@
 $EndComp
 $Comp
-L R R20
+L BodyController_01-rescue:R-RESCUE-BodyController_01 R20
 U 1 1 59A005C8
 P 2800 1600
@@
 $EndComp
 $Comp
-L R R55
+L BodyController_01-rescue:R-RESCUE-BodyController_01 R55
 U 1 1 59A005CE
 P 3100 1500
@@
 $EndComp
 $Comp
-L GND #PWR081
+L BodyController_01-rescue:GND-RESCUE-BodyController_01 #PWR081
 U 1 1 59A005D4
 P 3100 2600
@@
 $EndComp
 $Comp
-L C C62
+L BodyController_01-rescue:C-RESCUE-BodyController_01 C62
 U 1 1 59A005DA
 P 2550 2350
@@
 $EndComp
 $Comp
-L GND #PWR082
+L BodyController_01-rescue:GND-RESCUE-BodyController_01 #PWR082
 U 1 1 59A005E0
 P 2550 2600
@@
 $EndComp
 $Comp
-L +12V #PWR083
+L BodyController_01-rescue:+12V-RESCUE-BodyController_01 #PWR083
 U 1 1 59A005E6
 P 5200 1150
@@
 $EndComp
 $Comp
-L D D18
+L BodyController_01-rescue:D-RESCUE-BodyController_01 D18
 U 1 1 59A005EC
 P 5000 2900
@@
 $EndComp
 $Comp
-L D D19
+L BodyController_01-rescue:D-RESCUE-BodyController_01 D19
 U 1 1 59A005F2
 P 5250 2900
@@
 $EndComp
 $Comp
-L GND #PWR084
+L BodyController_01-rescue:GND-RESCUE-BodyController_01 #PWR084
 U 1 1 59A005F8
 P 5000 3100
@@
 $EndComp
 $Comp
-L GND #PWR085
+L BodyController_01-rescue:GND-RESCUE-BodyController_01 #PWR085
 U 1 1 59A005FE
 P 5250 3100
@@
 $EndComp
 $Comp
-L GND #PWR086
+L BodyController_01-rescue:GND-RESCUE-BodyController_01 #PWR086
 U 1 1 59B327F1
 P 9600 1600
@@
 $EndComp
 $Comp
-L GND #PWR087
+L BodyController_01-rescue:GND-RESCUE-BodyController_01 #PWR087
 U 1 1 59B32E08
 P 9650 2700
@@
 $EndComp
 $Comp
-L GND #PWR088
+L BodyController_01-rescue:GND-RESCUE-BodyController_01 #PWR088
 U 1 1 5A2AC1E2
 P 8850 4750
@@
 $EndComp
 $Comp
-L C C123
+L BodyController_01-rescue:C-RESCUE-BodyController_01 C123
 U 1 1 5A4B154C
 P 5550 1450
@@
 $EndComp
 $Comp
-L GND #PWR089
+L BodyController_01-rescue:GND-RESCUE-BodyController_01 #PWR089
 U 1 1 5A4B1661
 P 5550 1650
@@
 $EndComp
 $Comp
-L C C129
+L BodyController_01-rescue:C-RESCUE-BodyController_01 C129
 U 1 1 5A52CED7
 P 8000 3750
@@
 $EndComp
 $Comp
-L GND #PWR090
+L BodyController_01-rescue:GND-RESCUE-BodyController_01 #PWR090
 U 1 1 5A52CEDD
 P 8000 3900
@@
 $EndComp
 $Comp
-L C C130
+L BodyController_01-rescue:C-RESCUE-BodyController_01 C130
 U 1 1 5A52CF54
 P 8000 4550
@@
 $EndComp
 $Comp
-L GND #PWR091
+L BodyController_01-rescue:GND-RESCUE-BodyController_01 #PWR091
 U 1 1 5A52CF5A
 P 8000 4750
