File: Hardware/BodyController/BodyController_01/HighSideDrivers_3.sch (KiCad schematic (older format))
At the start: 49 parts, among them U12 BTS50202EKAXUMA2, U13 BTS50202EKAXUMA2, U15 BTS716G, U22 DRV8872DDARQ1, U23 tps25940-q1

Commit message: New bring-up code for Body Controller
Parts:
- C124, C125, C126, C127, C128: MPN CGA5L1X7R1E106M160AC -> C1206C106M3RACAUTO
- R125: value 487k -> 560k; MPN ERJ-3EKF4873V -> AC0603FR-07560KL
- R126: value 64k9 -> 100k; MPN ERJ-3EKF6492V -> AC0603FR-07100KL
- R127: value 30k9 -> 34k; MPN ERJ-3EKF3092V -> ERJ-3EKF3402V
- R128: value 17k8 -> 22k; MPN RG1608P-3092-B-T5 -> AC0603FR-0722KL
- R129: value 12k7 -> 10k; MPN AC0603FR-0712K7L -> AC0603FR-0710KL
Other:
- note added: "UnderVoltage = 5V\nOverVoltage = 20V\n2A/V\nCurrent Limit = 4A\ndV/dT = 12V/mS"
- note removed: "UnderVoltage = 6V\nOverVoltage = 18.5V\nCurrent Limit = 5A\ndV/dT = 12V/mS"
Changed lines of the file:
@@
 P 6200 3600
 F 0 "R125" V 6280 3600 50  0000 C CNN
-F 1 "487k" V 6200 3600 50  0000 C CNN
+F 1 "560k" V 6200 3600 50  0000 C CNN
 F 2 "Resistors_SMD:R_0603" V 6130 3600 50  0001 C CNN
-F 3 "http://industrial.panasonic.com/www-cgi/jvcr13pz.cgi?E+PZ+3+AOA0002+ERJ3EKF4873V+7+WW" H 6200 3600 50  0001 C CNN
-F 4 "ERJ-3EKF4873V" H 6280 3700 50  0001 C CNN "MPN"
+F 3 "http://www.yageo.com/NewPortal/yageodocoutput?fileName=/pdf/R-Chip/PYu-AC_51_RoHS_L_6.pdf" H 6200 3600 50  0001 C CNN
+F 4 "AC0603FR-07560KL" H 6280 3700 50  0001 C CNN "MPN"
 F 5 "y" H 6280 3700 50  0001 C CNN "populate"
 	1    6200 3600
@@
 P 6200 4100
 F 0 "R126" V 6280 4100 50  0000 C CNN
-F 1 "64k9" V 6200 4100 50  0000 C CNN
+F 1 "100k" V 6200 4100 50  0000 C CNN
 F 2 "Resistors_SMD:R_0603" V 6130 4100 50  0001 C CNN
-F 3 "http://industrial.panasonic.com/www-cgi/jvcr13pz.cgi?E+PZ+3+AOA0002+ERJ3EKF6492V+7+WW" H 6200 4100 50  0001 C CNN
-F 4 "ERJ-3EKF6492V" H 6280 4200 50  0001 C CNN "MPN"
+F 3 "http://www.yageo.com/NewPortal/yageodocoutput?fileName=/pdf/R-Chip/PYu-AC_51_RoHS_L_6.pdf" H 6200 4100 50  0001 C CNN
+F 4 "AC0603FR-07100KL" H 6280 4200 50  0001 C CNN "MPN"
 F 5 "y" H 6280 4200 50  0001 C CNN "populate"
 	1    6200 4100
@@
 P 6200 4650
 F 0 "R127" V 6280 4650 50  0000 C CNN
-F 1 "30k9" V 6200 4650 50  0000 C CNN
+F 1 "34k" V 6200 4650 50  0000 C CNN
 F 2 "Resistors_SMD:R_0603" V 6130 4650 50  0001 C CNN
-F 3 "https://industrial.panasonic.com/ww/products/resistors/chip-resistors/general-purpose-chip-resistors/precision-thick-film-chip-resistors/ERJ3EKF3092V" H 6200 4650 50  0001 C CNN
-F 4 "ERJ-3EKF3092V" H 6280 4750 50  0001 C CNN "MPN"
+F 3 "http://industrial.panasonic.com/www-cgi/jvcr13pz.cgi?E+PZ+3+AOA0002+ERJ3EKF3402V+7+WW" H 6200 4650 50  0001 C CNN
+F 4 "ERJ-3EKF3402V" H 6280 4750 50  0001 C CNN "MPN"
 F 5 "y" H 6280 4750 50  0001 C CNN "populate"
 	1    6200 4650
@@
 P 8900 5000
 F 0 "R129" V 8980 5000 50  0000 C CNN
-F 1 "12k7" V 8900 5000 50  0000 C CNN
+F 1 "10k" V 8900 5000 50  0000 C CNN
 F 2 "Resistors_SMD:R_0603" V 8830 5000 50  0001 C CNN
 F 3 "http://www.yageo.com/NewPortal/yageodocoutput?fileName=/pdf/R-Chip/PYu-AC_51_RoHS_L_6.pdf" H 8900 5000 50  0001 C CNN
-F 4 "AC0603FR-0712K7L" H 8980 5100 50  0001 C CNN "MPN"
+F 4 "AC0603FR-0710KL" H 8980 5100 50  0001 C CNN "MPN"
 F 5 "y" H 8980 5100 50  0001 C CNN "populate"
 	1    8900 5000
@@
 P 6400 4650
 F 0 "R128" V 6480 4650 50  0000 C CNN
-F 1 "17k8" V 6400 4650 50  0000 C CNN
+F 1 "22k" V 6400 4650 50  0000 C CNN
 F 2 "Resistors_SMD:R_0603" V 6330 4650 50  0001 C CNN
-F 3 "http://www.vishay.com/docs/28758/tnpw_e3.pdf" H 6400 4650 50  0001 C CNN
-F 4 "RG1608P-3092-B-T5" H 6480 4750 50  0001 C CNN "MPN"
+F 3 "http://www.yageo.com/NewPortal/yageodocoutput?fileName=/pdf/R-Chip/PYu-AC_51_RoHS_L_6.pdf" H 6400 4650 50  0001 C CNN
+F 4 "AC0603FR-0722KL" H 6480 4750 50  0001 C CNN "MPN"
 F 5 "y" H 6480 4750 50  0001 C CNN "populate"
 	1    6400 4650
@@
 F 1 "10uF" H 9025 650 50  0000 L CNN
 F 2 "Capacitors_SMD:C_1206" H 9038 600 50  0001 C CNN
-F 3 "https://product.tdk.com/info/en/documents/chara_sheet/CGA5L1X7R1E106M160AC.pdf" H 9000 750 50  0001 C CNN
-F 4 "CGA5L1X7R1E106M160AC" H 9025 950 50  0001 C CNN "MPN"
+F 3 "https://content.kemet.com/datasheets/KEM_C1023_X7R_AUTO_SMD.pdf" H 9000 750 50  0001 C CNN
+F 4 "C1206C106M3RACAUTO" H 9025 950 50  0001 C CNN "MPN"
 F 5 "y" H 9025 950 50  0001 C CNN "populate"
 	1    9000 750
@@
 F 1 "10uF" H 4975 3500 50  0000 L CNN
 F 2 "Capacitors_SMD:C_1206" H 4988 3450 50  0001 C CNN
-F 3 "https://product.tdk.com/info/en/documents/chara_sheet/CGA5L1X7R1E106M160AC.pdf" H 4950 3600 50  0001 C CNN
-F 4 "CGA5L1X7R1E106M160AC" H 4975 3800 50  0001 C CNN "MPN"
+F 3 "https://content.kemet.com/datasheets/KEM_C1023_X7R_AUTO_SMD.pdf" H 4950 3600 50  0001 C CNN
+F 4 "C1206C106M3RACAUTO" H 4975 3800 50  0001 C CNN "MPN"
 F 5 "y" H 4975 3800 50  0001 C CNN "populate"
 	1    4950 3600
@@
 F 1 "10uF" H 4175 5450 50  0000 L CNN
 F 2 "Capacitors_SMD:C_1206" H 4188 5400 50  0001 C CNN
-F 3 "https://product.tdk.com/info/en/documents/chara_sheet/CGA5L1X7R1E106M160AC.pdf" H 4150 5550 50  0001 C CNN
-F 4 "CGA5L1X7R1E106M160AC" H 4175 5750 50  0001 C CNN "MPN"
+F 3 "https://content.kemet.com/datasheets/KEM_C1023_X7R_AUTO_SMD.pdf" H 4150 5550 50  0001 C CNN
+F 4 "C1206C106M3RACAUTO" H 4175 5750 50  0001 C CNN "MPN"
 F 5 "y" H 4175 5750 50  0001 C CNN "populate"
 	1    4150 5550
@@
 F 1 "10uF" H 4975 1500 50  0000 L CNN
 F 2 "Capacitors_SMD:C_1206" H 4988 1450 50  0001 C CNN
-F 3 "https://product.tdk.com/info/en/documents/chara_sheet/CGA5L1X7R1E106M160AC.pdf" H 4950 1600 50  0001 C CNN
-F 4 "CGA5L1X7R1E106M160AC" H 4975 1800 50  0001 C CNN "MPN"
+F 3 "https://content.kemet.com/datasheets/KEM_C1023_X7R_AUTO_SMD.pdf" H 4950 1600 50  0001 C CNN
+F 4 "C1206C106M3RACAUTO" H 4975 1800 50  0001 C CNN "MPN"
 F 5 "y" H 4975 1800 50  0001 C CNN "populate"
 	1    4950 1600
@@
 F 1 "10uF" H 5725 3350 50  0000 L CNN
 F 2 "Capacitors_SMD:C_1206" H 5738 3300 50  0001 C CNN
-F 3 "https://product.tdk.com/info/en/documents/chara_sheet/CGA5L1X7R1E106M160AC.pdf" H 5700 3450 50  0001 C CNN
-F 4 "CGA5L1X7R1E106M160AC" H 5725 3650 50  0001 C CNN "MPN"
+F 3 "https://content.kemet.com/datasheets/KEM_C1023_X7R_AUTO_SMD.pdf" H 5700 3450 50  0001 C CNN
+F 4 "C1206C106M3RACAUTO" H 5725 3650 50  0001 C CNN "MPN"
 F 5 "y" H 5725 3650 50  0001 C CNN "populate"
 	1    5700 3450
@@
 31200
 Text Notes 7250 3150 0    60   ~ 0
-UnderVoltage = 6V\nOverVoltage = 18.5V\nCurrent Limit = 5A\ndV/dT = 12V/mS
+UnderVoltage = 5V\nOverVoltage = 20V\n2A/V\nCurrent Limit = 4A\ndV/dT = 12V/mS
 Text GLabel 9650 4700 2    59   Output ~ 0
 IC_CONTROLLER_~FLT

Commit message: too much work to specify all. New Scheduler, new bootloader, added new Hardware projects, updated code for bringup, COnverted kicad files to new version.
Parts:
- C124, C125, C126, C127, C128, C42, C43, C44, C67, C68: symbol C -> BodyController_01-rescue:C-RESCUE-BodyController_01
- D11, D12, D13, D14: symbol D -> BodyController_01-rescue:D-RESCUE-BodyController_01
- R125, R126, R127, R128, R129, R130, R131, R132, R66, R67, R68, R69, R70, R71, R72, R74, R75, R76, R77, R78, R79, R80, R81, R83, R84, R85, R86, R87, R88, R89: symbol R -> BodyController_01-rescue:R-RESCUE-BodyController_01
- U12, U13: symbol BTS50202EKAXUMA2 -> BodyController_01-rescue:BTS50202EKAXUMA2-RESCUE-BodyController_01
- U15: symbol BTS716G -> BodyController_01-rescue:BTS716G-RESCUE-BodyController_01
- U22: symbol DRV8872DDARQ1 -> BodyController_01-rescue:DRV8872DDARQ1-RESCUE-BodyController_01
- U23: symbol tps25940-q1 -> BodyController_01-rescue:tps25940-q1-RESCUE-BodyController_01
