File: Hardware/BodyController/BodyController_01/Communication.sch (KiCad schematic (older format))
At the start: 26 parts, among them U16 MCP2562-H/SN, U29 FT230X

Commit message: New bring-up code for Body Controller
Parts:
- C111, C87: MPN CGA3E2X7R1H104K080AA -> GCM188R71H104KA57D
- C46: MPN CGA5L1X7R1E106M160AC -> C1206C106M3RACAUTO
- D10: MPN PESD24VS1UB,115 -> ESDCAN24-2BLY
- D24: MPN PMEG10010ELRX -> PMEG6020AELRX
- L4: MPN ACT45B-510-2P-TL003 -> B82787C0513H002
- U16: value MCP2562-H/SN -> TCAN1051GVDRQ1; MPN MCP2562-H/SN -> TCAN1051GVDRQ1

Commit message: too much work to specify all. New Scheduler, new bootloader, added new Hardware projects, updated code for bringup, COnverted kicad files to new version.
Parts:
- C111, C112, C133, C134, C135, C136, C45, C46, C85, C86, C87, C88: symbol C -> BodyController_01-rescue:C-RESCUE-BodyController_01
- D10: symbol D_Schottky_x2_ACom_AKK -> BodyController_01-rescue:D_Schottky_x2_ACom_AKK-RESCUE-BodyController_01
- D24: symbol D_Schottky -> BodyController_01-rescue:D_Schottky-RESCUE-BodyController_01
- D4: symbol LED -> BodyController_01-rescue:LED-RESCUE-BodyController_01
- L4: symbol EMI_Filter_CommonMode -> BodyController_01-rescue:EMI_Filter_CommonMode-RESCUE-BodyController_01
- R173, R174, R175, R90, R91, R92, R93, R94: symbol R -> BodyController_01-rescue:R-RESCUE-BodyController_01
- U16: symbol MCP2562-H/SN -> BodyController_01-rescue:MCP2562-H_SN-RESCUE-BodyController_01
- U29: symbol FT230X -> BodyController_01-rescue:FT230X-RESCUE-BodyController_01
Changed lines of the file:
@@
-EESchema Schematic File Version 2
-LIBS:switches
-LIBS:power
-LIBS:device
-LIBS:transistors
-LIBS:conn
-LIBS:linear
-LIBS:regul
-LIBS:74xx
-LIBS:cmos4000
-LIBS:adc-dac
-LIBS:memory
-LIBS:xilinx
-LIBS:microcontrollers
-LIBS:dsp
-LIBS:microchip
-LIBS:analog_switches
-LIBS:motorola
-LIBS:texas
-LIBS:intel
-LIBS:audio
-LIBS:interface
-LIBS:digital-audio
-LIBS:philips
-LIBS:display
-LIBS:cypress
-LIBS:siliconi
-LIBS:opto
-LIBS:atmel
-LIBS:contrib
-LIBS:valves
-LIBS:HSD
-LIBS:micros
-LIBS:ICs
-LIBS:Connectors
-LIBS:microchip_dspic33dsc
+EESchema Schematic File Version 4
 LIBS:BodyController_01-cache
-EELAYER 25 0
+EELAYER 26 0
 EELAYER END
 $Descr A4 11693 8268
@@
 $EndDescr
 $Comp
-L MCP2562-H/SN U16
+L BodyController_01-rescue:MCP2562-H_SN-RESCUE-BodyController_01 U16
 U 1 1 5995476A
 P 7450 2600
@@
 $EndComp
 $Comp
-L GND #PWR0147
+L BodyController_01-rescue:GND-RESCUE-BodyController_01 #PWR0147
 U 1 1 59956B61
 P 7450 3050
@@
 $EndComp
 $Comp
-L +5V #PWR0148
+L BodyController_01-rescue:+5V-RESCUE-BodyController_01 #PWR0148
 U 1 1 59956B7A
 P 7450 1500
@@
 $EndComp
 $Comp
-L C C46
+L BodyController_01-rescue:C-RESCUE-BodyController_01 C46
 U 1 1 59956B93
 P 7150 1700
@@
 $EndComp
 $Comp
-L GND #PWR0149
+L BodyController_01-rescue:GND-RESCUE-BodyController_01 #PWR0149
 U 1 1 59956BCC
 P 7150 1900
@@
 $EndComp
 $Comp
-L R R92
+L BodyController_01-rescue:R-RESCUE-BodyController_01 R92
 U 1 1 59956C83
 P 6500 2400
@@
 $EndComp
 $Comp
-L R R90
+L BodyController_01-rescue:R-RESCUE-BodyController_01 R90
 U 1 1 59956CE0
 P 6100 2500
@@
 $EndComp
 $Comp
-L R R91
+L BodyController_01-rescue:R-RESCUE-BodyController_01 R91
 U 1 1 59956D1A
 P 6100 2800
@@
 $EndComp
 $Comp
-L R R93
+L BodyController_01-rescue:R-RESCUE-BodyController_01 R93
 U 1 1 59956D57
 P 9450 2400
@@
 $EndComp
 $Comp
-L R R94
+L BodyController_01-rescue:R-RESCUE-BodyController_01 R94
 U 1 1 59956DAD
 P 9450 2800
@@
 $EndComp
 $Comp
-L C C45
+L BodyController_01-rescue:C-RESCUE-BodyController_01 C45
 U 1 1 59956F4F
 P 6750 3100
@@
 $EndComp
 $Comp
-L GND #PWR0150
+L BodyController_01-rescue:GND-RESCUE-BodyController_01 #PWR0150
 U 1 1 59956F85
 P 6750 3250
@@
 $EndComp
 $Comp
-L +3V3 #PWR0151
+L BodyController_01-rescue:+3V3-RESCUE-BodyController_01 #PWR0151
 U 1 1 59956FC4
 P 6650 2700
@@
 $EndComp
 $Comp
-L FT230X U29
+L BodyController_01-rescue:FT230X-RESCUE-BodyController_01 U29
 U 1 1 59A81FAF
 P 3950 6200
@@
 $EndComp
 $Comp
-L C C85
+L BodyController_01-rescue:C-RESCUE-BodyController_01 C85
 U 1 1 59A83975
 P 2550 4300
@@
 $EndComp
 $Comp
-L C C87
+L BodyController_01-rescue:C-RESCUE-BodyController_01 C87
 U 1 1 59A839B7
 P 3550 4300
@@
 $EndComp
 $Comp
-L C C86
+L BodyController_01-rescue:C-RESCUE-BodyController_01 C86
 U 1 1 59A84BC7
 P 3250 4300
@@
 $EndComp
 $Comp
-L GND #PWR0152
+L BodyController_01-rescue:GND-RESCUE-BodyController_01 #PWR0152
 U 1 1 59A84C78
 P 3550 4500
@@
 $EndComp
 $Comp
-L GND #PWR0153
+L BodyController_01-rescue:GND-RESCUE-BodyController_01 #PWR0153
 U 1 1 59A84CA7
 P 3250 4500
@@
 $EndComp
 $Comp
-L GND #PWR0154
+L BodyController_01-rescue:GND-RESCUE-BodyController_01 #PWR0154
 U 1 1 59A84D2D
 P 2550 4500
@@
 $EndComp
 $Comp
-L D_Schottky D24
+L BodyController_01-rescue:D_Schottky-RESCUE-BodyController_01 D24
 U 1 1 59A85899
 P 4200 4050
@@
 $EndComp
 $Comp
-L +5V #PWR0155
+L BodyController_01-rescue:+5V-RESCUE-BodyController_01 #PWR0155
 U 1 1 59A85952
 P 4550 4050
@@
 $EndComp
 $Comp
-L GND #PWR0156
+L BodyController_01-rescue:GND-RESCUE-BodyController_01 #PWR0156
 U 1 1 59A86CDB
 P 4050 6800
@@
 $EndComp
 $Comp
-L PWR_FLAG #FLG0157
+L BodyController_01-rescue:PWR_FLAG-RESCUE-BodyController_01 #FLG0157
 U 1 1 59A88735
 P 3150 4050
@@
 $EndComp
 $Comp
-L C C88
+L BodyController_01-rescue:C-RESCUE-BodyController_01 C88
 U 1 1 59A895EF
 P 6800 1700
@@
 $EndComp
 $Comp
-L GND #PWR0158
+L BodyController_01-rescue:GND-RESCUE-BodyController_01 #PWR0158
 U 1 1 59A895F5
 P 6800 1850
@@
 $EndComp
 $Comp
-L C C111
+L BodyController_01-rescue:C-RESCUE-BodyController_01 C111
 U 1 1 5A45C0D4
 P 1600 6350
@@
 $EndComp
 $Comp
-L GND #PWR0159
+L BodyController_01-rescue:GND-RESCUE-BodyController_01 #PWR0159
 U 1 1 5A45C122
 P 1600 6550
@@
 $EndComp
 $Comp
-L LED D4
+L BodyController_01-rescue:LED-RESCUE-BodyController_01 D4
 U 1 1 5A45CB14
 P 9700 5000
@@
 $EndComp
 $Comp
-L R R173
+L BodyController_01-rescue:R-RESCUE-BodyController_01 R173
 U 1 1 5A45CC59
 P 9700 5450
@@
 $EndComp
 $Comp
-L GND #PWR0160
+L BodyController_01-rescue:GND-RESCUE-BodyController_01 #PWR0160
 U 1 1 5A45CD1A
 P 9700 5650
@@
 $EndComp
 $Comp
-L C C112
+L BodyController_01-rescue:C-RESCUE-BodyController_01 C112
 U 1 1 5A45DDEF
 P 9750 2600
@@
 $EndComp
 $Comp
-L GND #PWR0161
+L BodyController_01-rescue:GND-RESCUE-BodyController_01 #PWR0161
 U 1 1 5A45DDF5
 P 9950 2600
@@
 $EndComp
 $Comp
-L R R175
+L BodyController_01-rescue:R-RESCUE-BodyController_01 R175
 U 1 1 5A45ECCD
 P 2850 5650
@@
 $EndComp
 $Comp
-L R R174
+L BodyController_01-rescue:R-RESCUE-BodyController_01 R174
 U 1 1 5A45EF18
 P 2550 5750
@@
 $EndComp
 $Comp
-L EMI_Filter_CommonMode L4
+L BodyController_01-rescue:EMI_Filter_CommonMode-RESCUE-BodyController_01 L4
 U 1 1 5A5FE9AD
 P 8700 2600
@@
 $EndComp
 $Comp
-L C C135
+L BodyController_01-rescue:C-RESCUE-BodyController_01 C135
 U 1 1 5A5FF6F2
 P 9200 2000
@@
 $EndComp
 $Comp
-L C C136
+L BodyController_01-rescue:C-RESCUE-BodyController_01 C136
 U 1 1 5A5FF939
 P 9200 3200
@@
 $EndComp
 $Comp
-L GND #PWR0162
+L BodyController_01-rescue:GND-RESCUE-BodyController_01 #PWR0162
 U 1 1 5A5FFB7F
 P 9200 1850
@@
 $EndComp
 $Comp
-L GND #PWR0163
+L BodyController_01-rescue:GND-RESCUE-BodyController_01 #PWR0163
 U 1 1 5A5FFC84
 P 9200 3350
@@
 $EndComp
 $Comp
-L C C134
+L BodyController_01-rescue:C-RESCUE-BodyController_01 C134
 U 1 1 5A600AF0
 P 8200 3200
@@
 $EndComp
 $Comp
-L GND #PWR0164
+L BodyController_01-rescue:GND-RESCUE-BodyController_01 #PWR0164
 U 1 1 5A600AF6
 P 8200 3350
@@
 $EndComp
 $Comp
-L C C133
+L BodyController_01-rescue:C-RESCUE-BodyController_01 C133
 U 1 1 5A600B61
 P 8200 2000
@@
 $EndComp
 $Comp
-L GND #PWR0165
+L BodyController_01-rescue:GND-RESCUE-BodyController_01 #PWR0165
 U 1 1 5A600B67
 P 8200 1850
@@
 $EndComp
 $Comp
-L D_Schottky_x2_ACom_AKK D10
+L BodyController_01-rescue:D_Schottky_x2_ACom_AKK-RESCUE-BodyController_01 D10
 U 1 1 5A623006
 P 10400 2600
@@
 $EndComp
 $Comp
-L GND #PWR0166
+L BodyController_01-rescue:GND-RESCUE-BodyController_01 #PWR0166
 U 1 1 5A623375
 P 10600 2600

Commit message: changed some directory locations, added new DCDC PBC project, few Body controller light and switches changes
Parts:
- U29: symbol BodyController_01-rescue:FT230X-RESCUE-BodyController_01 -> ftdi:FT230XS
Connections:
- wire segments 55 -> 76
Other:
- moved on the sheet: C85, C86, C87, D24

Commit message: BMS controller. Lots of new FW including bootloaders
Parts:
- U29: symbol ftdi:FT230XS -> BodyController_01-rescue:FT230XS-ftdi
Changed lines of the file:
@@
 $EndComp
 $Comp
-L ftdi:FT230XS U29
+L BodyController_01-rescue:FT230XS-ftdi U29
 U 1 1 59A81FAF
 P 3800 5750
