File: Hardware/BodyController/BodyController_01/PowerRails.sch (KiCad schematic (older format))
At the start: 51 parts, among them Q10 NX1029X,115, Q17 Q_PMOS_GSD, Q5 Q_PMOS_GSD, U17 TPS70950QDBVRQ1, U18 TPS70933QDBVRQ1, U19 TPS70933QDBVRQ1, U20 LMR140x0

Commit message: New bring-up code for Body Controller
Parts:
- C113, C26, C49, C55, C56: MPN CGA5L1X7R1E106M160AC -> C1206C106M3RACAUTO
- C23, C47, C84: value 10uF -> 4u7; MPN CGA5L1X7R1E106M160AC -> CGA5L3X7R1H475K160AE
- C50: value 10nF -> 100nF; MPN CGA3E2X7R1H103K080AA -> GCM188R71H104KA57D
- C53: value 12pF -> 18pF; MPN CGA3E2C0G1H120J080AA -> CGA3E2C0G1H180J080AA
- C83: MPN CGA3E2X7R1H104K080AA -> GCM188R71H104KA57D
- D1, D2, D3, D6, D7: MPN PMEG10010ELRX -> PMEG6020AELRX
- R102, R103: value 10R -> 3R0; MPN AC0603FR-0710RL -> ERJ-3GEYJ3R0V
- R105, R4: value 10k -> 4k7; MPN AC0603FR-0710KL -> AC0603FR-074K7L
- R106: value 20R -> 22R; MPN AC0603FR-0720RL -> AC0603FR-0722RL
- R107: value 10k -> 845k; MPN AC0603FR-0710KL -> RMCF0603FT845K
- R108, R24: value 10k -> 150k; MPN AC0603FR-0710KL -> AC0603FR-07150KL
- R23: value 10k -> 560k; MPN AC0603FR-0710KL -> AC0603FR-07560KL
- R99: value 10k -> 49k9; MPN AC0603FR-0710KL -> AC0603FR-0749K9L
Other:
- note added: "Buck Converter:\n5V 2A Output\n3V UVLO\n500kHz switching frequency\n20mS soft start"
- note removed: "Buck Converter:\n5V 2A Output\n3.3V UVLO\n500kHz switching frequency\n20mS soft start"

Commit message: too much work to specify all. New Scheduler, new bootloader, added new Hardware projects, updated code for bringup, COnverted kicad files to new version.
Parts:
- C10, C113, C23, C25, C26, C27, C28, C29, C47, C48, C49, C50, C51, C52, C53, C54, C55, C56, C83, C84: symbol C -> BodyController_01-rescue:C-RESCUE-BodyController_01
- C24, C30: symbol CP -> BodyController_01-rescue:CP-RESCUE-BodyController_01
- D1, D17, D2, D3, D6, D7: symbol D_Schottky -> BodyController_01-rescue:D_Schottky-RESCUE-BodyController_01
- L2: symbol Ferrite_Bead -> BodyController_01-rescue:Ferrite_Bead-RESCUE-BodyController_01
- L3: symbol L -> BodyController_01-rescue:L-RESCUE-BodyController_01
- Q10: symbol NX1029X,115 -> BodyController_01-rescue:NX1029X,115-RESCUE-BodyController_01
- Q17, Q5: symbol Q_PMOS_GSD -> BodyController_01-rescue:Q_PMOS_GSD-RESCUE-BodyController_01
- R100, R101, R102, R103, R104, R105, R106, R107, R108, R23, R24, R3, R4, R99: symbol R -> BodyController_01-rescue:R-RESCUE-BodyController_01
- U17, U18, U19: symbol TLV70033DDC -> BodyController_01-rescue:TLV70033DDC-RESCUE-BodyController_01
- U20: symbol LMR140x0 -> BodyController_01-rescue:LMR140x0-RESCUE-BodyController_01

Commit message: changed some directory locations, added new DCDC PBC project, few Body controller light and switches changes
Parts:
- U17, U18, U19: symbol BodyController_01-rescue:TLV70033DDC-RESCUE-BodyController_01 -> regul:TLV70033_SOT23-5
- U20: symbol BodyController_01-rescue:LMR140x0-RESCUE-BodyController_01 -> ICs:LMR140x0
Connections:
- wire segments 114 -> 152
Other:
- moved on the sheet: C113, C23, C26, C47, C49, C84, D6, D7

Commit message: BMS controller. Lots of new FW including bootloaders
Parts:
- U17, U18, U19: symbol regul:TLV70033_SOT23-5 -> BodyController_01-rescue:TLV70033_SOT23-5-regul
Changed lines of the file:
@@
 $EndComp
 $Comp
-L regul:TLV70033_SOT23-5 U18
+L BodyController_01-rescue:TLV70033_SOT23-5-regul U18
 U 1 1 59A6966E
 P 2350 6950
@@
 $EndComp
 $Comp
-L regul:TLV70033_SOT23-5 U17
+L BodyController_01-rescue:TLV70033_SOT23-5-regul U17
 U 1 1 5A49C58E
 P 9950 5500
@@
 $EndComp
 $Comp
-L regul:TLV70033_SOT23-5 U19
+L BodyController_01-rescue:TLV70033_SOT23-5-regul U19
 U 1 1 5A4AAC85
 P 5550 6950
