File: Hardware/InterfaceController/InterfaceController_01/Communication.sch (KiCad schematic (older format))
At the start: 26 parts

Commit message: too much work to specify all. New Scheduler, new bootloader, added new Hardware projects, updated code for bringup, COnverted kicad files to new version.
Parts:
- C? (x12): symbol C -> device:C
- D?: symbol D_Schottky -> device:D_Schottky
- D?: symbol LED -> device:LED
- D?: symbol D_Schottky_x2_ACom_AKK -> device:D_Schottky_x2_ACom_AKK
- L?: symbol EMI_Filter_CommonMode -> device:EMI_Filter_CommonMode
- R? (x8): symbol R -> device:R
- U?: symbol MCP2562-H/SN -> IntrefaceController_01-rescue:MCP2562-H_SN-RESCUE-IntrefaceController_01
- U?: symbol FT230XS -> ftdi:FT230XS
