File: Hardware/InterfaceController/InterfaceController_01/MicroController.sch (KiCad schematic (older format))
At the start: 19 parts

Commit message: too much work to specify all. New Scheduler, new bootloader, added new Hardware projects, updated code for bringup, COnverted kicad files to new version.
Parts:
- C? (x11): symbol C -> device:C
- L?: symbol Ferrite_Bead -> device:Ferrite_Bead
- R? (x3): symbol R -> device:R
- SW?: symbol SW_Push -> switches:SW_Push
- U? (x2): symbol PIC33EPxxxMU810 -> micros:PIC33EPxxxMU810
- Y?: symbol Crystal_GND24 -> device:Crystal_GND24
Changed lines of the file:
@@
-EESchema Schematic File Version 2
-LIBS:power
-LIBS:device
-LIBS:switches
-LIBS:relays
-LIBS:motors
-LIBS:transistors
-LIBS:conn
-LIBS:linear
-LIBS:regul
-LIBS:74xx
-LIBS:cmos4000
-LIBS:adc-dac
-LIBS:memory
-LIBS:xilinx
-LIBS:microcontrollers
-LIBS:dsp
-LIBS:microchip
-LIBS:analog_switches
-LIBS:motorola
-LIBS:texas
-LIBS:intel
-LIBS:audio
-LIBS:interface
-LIBS:digital-audio
-LIBS:philips
-LIBS:display
-LIBS:cypress
-LIBS:siliconi
-LIBS:opto
-LIBS:atmel
-LIBS:contrib
-LIBS:valves
-LIBS:Connectors
-LIBS:HSD
-LIBS:ICs
-LIBS:micros
-LIBS:battery_management
-LIBS:ftdi
-LIBS:leds
-LIBS:LEM
-LIBS:microchip_dspic33dsc
-LIBS:modules
-LIBS:rfcom
-LIBS:RFSolutions
-LIBS:sensors
-LIBS:IntrefaceController_01-cache
-EELAYER 25 0
+EESchema Schematic File Version 4
+EELAYER 26 0
 EELAYER END
 $Descr A4 11693 8268
@@
 $EndDescr
 $Comp
-L +3V3 #PWR?
+L power:+3V3 #PWR?
 U 1 1 59953D12
 P 850 4400
@@
 $EndComp
 $Comp
-L GND #PWR?
+L power:GND #PWR?
 U 1 1 59953D98
 P 850 5300
@@
 $EndComp
 $Comp
-L C C?
+L device:C C?
 U 1 1 59954183
 P 950 4850
@@
 $EndComp
 $Comp
-L C C?
+L device:C C?
 U 1 1 599541B1
 P 1150 4850
@@
 $EndComp
 $Comp
-L C C?
+L device:C C?
 U 1 1 599541DB
 P 1350 4850
@@
 $EndComp
 $Comp
-L C C?
+L device:C C?
 U 1 1 599541FC
 P 1550 4850
@@
 $EndComp
 $Comp
-L C C?
+L device:C C?
 U 1 1 59954470
 P 1650 6550
@@
 $EndComp
 $Comp
-L GND #PWR?
+L power:GND #PWR?
 U 1 1 5995450B
 P 1400 6550
@@
 $EndComp
 $Comp
-L C C?
+L device:C C?
 U 1 1 59954578
 P 1650 6100
@@
 $EndComp
 $Comp
-L C C?
+L device:C C?
 U 1 1 59955AC7
 P 850 6100
@@
 $EndComp
 $Comp
-L Ferrite_Bead L?
+L device:Ferrite_Bead L?
 U 1 1 59955DBF
 P 1250 5900
@@
 $EndComp
 $Comp
-L +3V3 #PWR?
+L power:+3V3 #PWR?
 U 1 1 59955FA7
 P 750 5900
@@
 $EndComp
 $Comp
-L GND #PWR?
+L power:GND #PWR?
 U 1 1 59955FD3
 P 750 6300
@@
 $EndComp
 $Comp
-L C C?
+L device:C C?
 U 1 1 599562CF
 P 5300 6650
@@
 $EndComp
 $Comp
-L C C?
+L device:C C?
 U 1 1 59956321
 P 5300 7150
@@
 $EndComp
 $Comp
-L R R?
+L device:R R?
 U 1 1 5995635F
 P 4150 6900
@@
 $EndComp
 $Comp
-L GND #PWR?
+L power:GND #PWR?
 U 1 1 5995664C
 P 5600 6900
@@
 $EndComp
 $Comp
-L +3V3 #PWR?
+L power:+3V3 #PWR?
 U 1 1 59967AA0
 P 1450 7050
@@
 $EndComp
 $Comp
-L R R?
+L device:R R?
 U 1 1 59967AE3
 P 1450 7300
@@
 $EndComp
 $Comp
-L +3.3VA #PWR?
+L power:+3.3VA #PWR?
 U 1 1 59977C27
 P 1800 5850
@@
 $EndComp
 $Comp
-L PWR_FLAG #FLG?
+L power:PWR_FLAG #FLG?
 U 1 1 59980D1B
 P 1500 5750
@@
 $EndComp
 $Comp
-L PIC33EPxxxMU810 U?
+L micros:PIC33EPxxxMU810 U?
 U 1 1 599FC02F
 P 8150 2200
@@
 $EndComp
 $Comp
-L PIC33EPxxxMU810 U?
+L micros:PIC33EPxxxMU810 U?
 U 2 1 599FC07A
 P 2700 3650
@@
 $EndComp
 $Comp
-L C C?
+L device:C C?
 U 1 1 599FDE83
 P 750 4850
@@
 $EndComp
 $Comp
-L C C?
+L device:C C?
 U 1 1 599FDED2
 P 1750 4850
@@
 $EndComp
 $Comp
-L +3V3 #PWR?
+L power:+3V3 #PWR?
 U 1 1 59B2845D
 P 4100 5750
@@
 $EndComp
 $Comp
-L Crystal_GND24 Y?
+L device:Crystal_GND24 Y?
 U 1 1 59BBA021
 P 4700 6900
@@
 $EndComp
 $Comp
-L GND #PWR?
+L power:GND #PWR?
 U 1 1 59BBA3D3
 P 4950 6900
@@
 $EndComp
 $Comp
-L GND #PWR?
+L power:GND #PWR?
 U 1 1 59BBA417
 P 4450 6900
@@
 $EndComp
 $Comp
-L GND #PWR?
+L power:GND #PWR?
 U 1 1 5A45E91E
 P 700 7200
@@
 $EndComp
 $Comp
-L SW_Push SW?
+L switches:SW_Push SW?
 U 1 1 5A45E5E7
 P 950 7200
@@
 $EndComp
 $Comp
-L R R?
+L device:R R?
 U 1 1 5A870904
 P 1700 7600
@@
 DEBUG_PIN
 Wire Wire Line
-	750  5300 2000 5300
-Wire Wire Line
-	750  4400 2000 4400
+	750  5300 850  5300
+Wire Wire Line
+	750  4400 850  4400
 Wire Wire Line
 	950  4700 950  4400
@@
 	1500 6550 1400 6550
 Wire Wire Line
-	1400 5900 1950 5900
+	1400 5900 1500 5900
 Wire Wire Line
 	1650 5950 1650 5900
 Wire Wire Line
-	750  6300 1950 6300
-Wire Wire Line
-	750  5900 1100 5900
+	750  6300 850  6300
+Wire Wire Line
+	750  5900 850  5900
 Wire Wire Line
 	850  6300 850  6250
@@
 	1650 6250 1650 6300
 Wire Wire Line
-	3950 6650 5150 6650
-Wire Wire Line
-	3950 7150 5150 7150
+	3950 6650 4150 6650
+Wire Wire Line
+	3950 7150 4150 7150
 Wire Wire Line
 	4700 7050 4700 7150
@@
 	5500 7150 5450 7150
 Wire Wire Line
-	5500 6650 5500 7150
+	5500 6650 5500 6900
 Wire Wire Line
 	5500 6650 5450 6650
@@
 	1450 7600 1450 7450
 Wire Wire Line
-	850  7600 1550 7600
+	850  7600 1250 7600
 Wire Wire Line
 	1800 5850 1800 5900
@@
 	750  5000 750  5300
 Wire Wire Line
-	2000 4400 2000 4900
-Wire Wire Line
-	2000 5300 2000 5700
+	2000 4400 2000 4500
+Wire Wire Line
+	2000 5300 2000 5400
 Wire Wire Line
 	1950 5900 1950 5950
@@
 Connection ~ 1250 7600
 NoConn ~ 3900 6150
+Wire Wire Line
+	950  4400 1150 4400
+Wire Wire Line
+	1150 4400 1350 4400
+Wire Wire Line
+	1350 4400 1550 4400
+Wire Wire Line
+	1550 4400 1750 4400
+Wire Wire Line
+	950  5300 1150 5300
+Wire Wire Line
+	1150 5300 1350 5300
+Wire Wire Line
+	1350 5300 1550 5300
+Wire Wire Line
+	1550 5300 1750 5300
+Wire Wire Line
+	850  4400 950  4400
+Wire Wire Line
+	1650 5900 1800 5900
+Wire Wire Line
+	850  6300 1650 6300
+Wire Wire Line
+	850  5900 1100 5900
+Wire Wire Line
+	1650 6300 1950 6300
+Wire Wire Line
+	4700 7150 5150 7150
+Wire Wire Line
+	4150 7150 4700 7150
+Wire Wire Line
+	4150 6650 4700 6650
+Wire Wire Line
+	4700 6650 5150 6650
+Wire Wire Line
+	1450 7600 1550 7600
+Wire Wire Line
+	1800 5900 1950 5900
+Wire Wire Line
+	1500 5900 1650 5900
+Wire Wire Line
+	850  5300 950  5300
+Wire Wire Line
+	2000 5400 2000 5500
+Wire Wire Line
+	2000 5500 2000 5600
+Wire Wire Line
+	2000 5600 2000 5700
+Wire Wire Line
+	2000 4800 2000 4900
+Wire Wire Line
+	2000 4700 2000 4800
+Wire Wire Line
+	2000 4600 2000 4700
+Wire Wire Line
+	2000 4500 2000 4600
+Wire Wire Line
+	1750 4400 2000 4400
+Wire Wire Line
+	1750 5300 2000 5300
+Wire Wire Line
+	5500 6900 5500 7150
+Wire Wire Line
+	1250 7600 1450 7600
 $EndSCHEMATC
