File: Hardware/InterfaceController/InterfaceController_01/PowerRails.sch (KiCad schematic (older format))
At the start: 55 parts

Commit message: too much work to specify all. New Scheduler, new bootloader, added new Hardware projects, updated code for bringup, COnverted kicad files to new version.
Parts:
- C? (x20): symbol C -> device:C
- C? (x2): symbol CP -> device:CP
- D? (x6): symbol D_Schottky -> device:D_Schottky
- D?: symbol D_Zener -> device:D_Zener
- L?: symbol Ferrite_Bead -> device:Ferrite_Bead
- L?: symbol L -> device:L
- Q? (x2): symbol NX1029X,115 -> ICs:NX1029X,115
- Q? (x2): symbol Q_PMOS_GSD -> device:Q_PMOS_GSD
- Q?: symbol SQJ423EP-T1_GE3 -> HSD:SQJ423EP-T1_GE3
- R? (x15): symbol R -> device:R
- U?: symbol LMR140x0 -> ICs:LMR140x0
Connections:
- wire segments 170 -> 169
Other:
- note added: "12V_MAIN"
- moved on the sheet: C?, D?, Q?A, Q?B, R?
