File: Hardware/InterfaceController/InterfaceController_01/USB.sch (KiCad schematic (older format))
At the start: 64 parts

Commit message: too much work to specify all. New Scheduler, new bootloader, added new Hardware projects, updated code for bringup, COnverted kicad files to new version.
Parts:
- C? (x2): symbol CP -> device:CP
- C? (x21): symbol C -> device:C
- D? (x4): symbol D_Schottky -> device:D_Schottky
- D? (x2): symbol D_Schottky_x2_ACom_AKK -> device:D_Schottky_x2_ACom_AKK
- L? (x2): symbol Ferrite_Bead -> device:Ferrite_Bead
- L? (x2): symbol L -> device:L
- NT? (x6): symbol Net_Tie-0.5mm -> Connectors:Net_Tie-0.5mm
- R? (x18): symbol R -> device:R
- U? (x2): symbol LMR140x0 -> ICs:LMR140x0
- U?: symbol TPS2513A -> texas:TPS2513A
- U? (x4): symbol INA21x -> ICs:INA21x
