File: Hardware/InterfaceController/InterfaceController_01/file5A8AFC71.sch (KiCad schematic (older format))
At the start: 24 parts

Commit message: too much work to specify all. New Scheduler, new bootloader, added new Hardware projects, updated code for bringup, COnverted kicad files to new version.
Parts:
- C? (x9): symbol C -> device:C
- Q?: symbol Q_Photo_NPN -> device:Q_Photo_NPN
- R? (x14): symbol R -> device:R
Changed lines of the file:
@@
-EESchema Schematic File Version 2
-LIBS:power
-LIBS:device
-LIBS:switches
-LIBS:relays
-LIBS:motors
-LIBS:transistors
-LIBS:conn
-LIBS:linear
-LIBS:regul
-LIBS:74xx
-LIBS:cmos4000
-LIBS:adc-dac
-LIBS:memory
-LIBS:xilinx
-LIBS:microcontrollers
-LIBS:dsp
-LIBS:microchip
-LIBS:analog_switches
-LIBS:motorola
-LIBS:texas
-LIBS:intel
-LIBS:audio
-LIBS:interface
-LIBS:digital-audio
-LIBS:philips
-LIBS:display
-LIBS:cypress
-LIBS:siliconi
-LIBS:opto
-LIBS:atmel
-LIBS:contrib
-LIBS:valves
-LIBS:Connectors
-LIBS:HSD
-LIBS:ICs
-LIBS:micros
-LIBS:battery_management
-LIBS:ftdi
-LIBS:leds
-LIBS:LEM
-LIBS:microchip_dspic33dsc
-LIBS:modules
-LIBS:rfcom
-LIBS:RFSolutions
-LIBS:sensors
-LIBS:IntrefaceController_01-cache
-EELAYER 25 0
+EESchema Schematic File Version 4
+EELAYER 26 0
 EELAYER END
 $Descr A4 11693 8268
@@
 $EndDescr
 $Comp
-L R R?
+L device:R R?
 U 1 1 5A8EE8D0
 P 2850 1350
@@
 $EndComp
 $Comp
-L R R?
+L device:R R?
 U 1 1 5A8EE9AA
 P 2500 1600
@@
 $EndComp
 $Comp
-L C C?
+L device:C C?
 U 1 1 5A8EE9D4
 P 3300 1600
@@
 $EndComp
 $Comp
-L C C?
+L device:C C?
 U 1 1 5A8EEA21
 P 2200 1600
@@
 $EndComp
 $Comp
-L R R?
+L device:R R?
 U 1 1 5A8EEA86
 P 3200 1100
@@
 $EndComp
 $Comp
-L GND #PWR?
+L power:GND #PWR?
 U 1 1 5A8EEB8F
 P 2200 1750
@@
 $EndComp
 $Comp
-L GND #PWR?
+L power:GND #PWR?
 U 1 1 5A8EEBB0
 P 2500 1750
@@
 $EndComp
 $Comp
-L GND #PWR?
+L power:GND #PWR?
 U 1 1 5A8EEBD4
 P 3300 1750
@@
 	3300 1350 3300 1450
 Wire Wire Line
-	3000 1350 3700 1350
+	3000 1350 3200 1350
 Connection ~ 3300 1350
 Wire Wire Line
-	1950 1350 2700 1350
+	1950 1350 2200 1350
 Wire Wire Line
 	2200 1350 2200 1450
@@
 SPARE_IO_1_IN
 $Comp
-L R R?
+L device:R R?
 U 1 1 5A8EF0A4
 P 2850 2850
@@
 $EndComp
 $Comp
-L R R?
+L device:R R?
 U 1 1 5A8EF0AA
 P 2500 3100
@@
 $EndComp
 $Comp
-L C C?
+L device:C C?
 U 1 1 5A8EF0B0
 P 3300 3100
@@
 $EndComp
 $Comp
-L C C?
+L device:C C?
 U 1 1 5A8EF0B6
 P 2200 3100
@@
 $EndComp
 $Comp
-L R R?
+L device:R R?
 U 1 1 5A8EF0BC
 P 3200 2600
@@
 $EndComp
 $Comp
-L GND #PWR?
+L power:GND #PWR?
 U 1 1 5A8EF0C2
 P 2200 3250
@@
 $EndComp
 $Comp
-L GND #PWR?
+L power:GND #PWR?
 U 1 1 5A8EF0C8
 P 2500 3250
@@
 $EndComp
 $Comp
-L GND #PWR?
+L power:GND #PWR?
 U 1 1 5A8EF0CE
 P 3300 3250
@@
 	3300 2850 3300 2950
 Wire Wire Line
-	3000 2850 3700 2850
+	3000 2850 3200 2850
 Connection ~ 3300 2850
 Wire Wire Line
-	1950 2850 2700 2850
+	1950 2850 2200 2850
 Wire Wire Line
 	2200 2850 2200 2950
@@
 SPARE_IO_2_IN
 $Comp
-L Q_Photo_NPN Q?
+L device:Q_Photo_NPN Q?
 U 1 1 5A8EF152
 P 10600 1700
@@
 $EndComp
 $Comp
-L R R?
+L device:R R?
 U 1 1 5A8EF290
 P 10500 1250
@@
 $EndComp
 Wire Wire Line
-	10500 1400 10500 1500
-$Comp
-L GND #PWR?
+	10500 1400 10500 1450
+$Comp
+L power:GND #PWR?
 U 1 1 5A8EF43C
 P 10500 1900
@@
 $EndComp
 $Comp
-L R R?
+L device:R R?
 U 1 1 5A8EF4C2
 P 9900 1450
@@
 $EndComp
 $Comp
-L C C?
+L device:C C?
 U 1 1 5A8EF53F
 P 9550 1750
@@
 $EndComp
 Wire Wire Line
-	9750 1450 9250 1450
+	9750 1450 9550 1450
 Wire Wire Line
 	9550 1600 9550 1450
@@
 Connection ~ 10500 1450
 $Comp
-L GND #PWR?
+L power:GND #PWR?
 U 1 1 5A8EF636
 P 9550 1900
@@
 AMBIENT_LIGHT_AI
 $Comp
-L R R?
+L device:R R?
 U 1 1 5A906AB1
 P 2850 4400
@@
 $EndComp
 $Comp
-L R R?
+L device:R R?
 U 1 1 5A906AB7
 P 2500 4650
@@
 $EndComp
 $Comp
-L C C?
+L device:C C?
 U 1 1 5A906ABD
 P 3300 4650
@@
 $EndComp
 $Comp
-L C C?
+L device:C C?
 U 1 1 5A906AC3
 P 2200 4650
@@
 $EndComp
 $Comp
-L R R?
+L device:R R?
 U 1 1 5A906AC9
 P 3200 4150
@@
 $EndComp
 $Comp
-L GND #PWR?
+L power:GND #PWR?
 U 1 1 5A906ACF
 P 2200 4800
@@
 $EndComp
 $Comp
-L GND #PWR?
+L power:GND #PWR?
 U 1 1 5A906AD5
 P 2500 4800
@@
 $EndComp
 $Comp
-L GND #PWR?
+L power:GND #PWR?
 U 1 1 5A906ADB
 P 3300 4800
@@
 	3300 4400 3300 4500
 Wire Wire Line
-	3000 4400 3700 4400
+	3000 4400 3200 4400
 Connection ~ 3300 4400
 Wire Wire Line
-	1950 4400 2700 4400
+	1950 4400 2200 4400
 Wire Wire Line
 	2200 4400 2200 4500
@@
 SPARE_IO_3_IN
 $Comp
-L R R?
+L device:R R?
 U 1 1 5A906AED
 P 2850 5900
@@
 $EndComp
 $Comp
-L R R?
+L device:R R?
 U 1 1 5A906AF3
 P 2500 6150
@@
 $EndComp
 $Comp
-L C C?
+L device:C C?
 U 1 1 5A906AF9
 P 3300 6150
@@
 $EndComp
 $Comp
-L C C?
+L device:C C?
 U 1 1 5A906AFF
 P 2200 6150
@@
 $EndComp
 $Comp
-L R R?
+L device:R R?
 U 1 1 5A906B05
 P 3200 5650
@@
 $EndComp
 $Comp
-L GND #PWR?
+L power:GND #PWR?
 U 1 1 5A906B0B
 P 2200 6300
@@
 $EndComp
 $Comp
-L GND #PWR?
+L power:GND #PWR?
 U 1 1 5A906B11
 P 2500 6300
@@
 $EndComp
 $Comp
-L GND #PWR?
+L power:GND #PWR?
 U 1 1 5A906B17
 P 3300 6300
@@
 	3300 5900 3300 6000
 Wire Wire Line
-	3000 5900 3700 5900
+	3000 5900 3200 5900
 Connection ~ 3300 5900
 Wire Wire Line
-	1950 5900 2700 5900
+	1950 5900 2200 5900
 Wire Wire Line
 	2200 5900 2200 6000
@@
 SPARE_IO_4_IN
 $Comp
-L +3.3VP #PWR?
+L power:+3.3VP #PWR?
 U 1 1 5A907122
 P 3200 950
@@
 $EndComp
 $Comp
-L +3.3VP #PWR?
+L power:+3.3VP #PWR?
 U 1 1 5A9071BA
 P 3200 2450
@@
 $EndComp
 $Comp
-L +3.3VP #PWR?
+L power:+3.3VP #PWR?
 U 1 1 5A90729A
 P 3200 4000
@@
 $EndComp
 $Comp
-L +3.3VP #PWR?
+L power:+3.3VP #PWR?
 U 1 1 5A9072ED
 P 3200 5500
@@
 	1    0    0    -1
 $EndComp
+Wire Wire Line
+	3300 1350 3700 1350
+Wire Wire Line
+	2500 1350 2700 1350
+Wire Wire Line
+	2200 1350 2500 1350
+Wire Wire Line
+	3200 1350 3300 1350
+Wire Wire Line
+	3300 2850 3700 2850
+Wire Wire Line
+	2500 2850 2700 2850
+Wire Wire Line
+	2200 2850 2500 2850
+Wire Wire Line
+	3200 2850 3300 2850
+Wire Wire Line
+	9550 1450 9250 1450
+Wire Wire Line
+	10500 1450 10500 1500
+Wire Wire Line
+	3300 4400 3700 4400
+Wire Wire Line
+	2500 4400 2700 4400
+Wire Wire Line
+	2200 4400 2500 4400
+Wire Wire Line
+	3200 4400 3300 4400
+Wire Wire Line
+	3300 5900 3700 5900
+Wire Wire Line
+	2500 5900 2700 5900
+Wire Wire Line
+	2200 5900 2500 5900
+Wire Wire Line
+	3200 5900 3300 5900
 $EndSCHEMATC
