File: Hardware/DCDC/DCDC_01/Connectors.sch (KiCad schematic (older format))
At the start: 8 parts, among them J1 USB_B_Micro, J2 Conn_01x04, J3 Conn_01x02, J4 Conn_01x02, J5 Conn_01x06

Commit message: Mostly finished DCDC schematic, still needs some values and maybe a soft-start circuit that can be bypassed with 0ohm resister in case it doesn't work.
Parts:
- added R72, R73: 100R, Resistors_SMD:R_0603, symbol device:R
- C82: DNP (none) -> (none); Voltage (none) -> 50V
- D7, D8, J1, J2, J3, J4, J5: DNP (none) -> (none)
Connections:
- wire segments 23 -> 26
Changed lines of the file:
@@
 $Descr A4 11693 8268
 encoding utf-8
-Sheet 7 7
+Sheet 8 8
 Title ""
 Date ""
@@
 F 2 "" H 8550 4850 50  0001 C CNN
 F 3 "~" H 8550 4850 50  0001 C CNN
+F 4 " " H 0   0   50  0001 C CNN "DNP"
 	1    8400 4900
 	1    0    0    -1
 $EndComp
-Text GLabel 8700 4700 2    60   Output ~ 0
-USB_5V
-Text GLabel 8700 4900 2    60   BiDi ~ 0
-USB_D+
-Text GLabel 8700 5000 2    60   BiDi ~ 0
-USB_D-
 $Comp
 L power:GND #PWR0124
@@
 F 2 "" H 7988 5450 50  0001 C CNN
 F 3 "~" H 7950 5600 50  0001 C CNN
+F 4 " " H 0   0   50  0001 C CNN "DNP"
+F 5 "50V" H 0   0   50  0001 C CNN "Voltage"
 	1    7950 5600
 	1    0    0    -1
 $EndComp
-Wire Wire Line
-	8300 5300 8300 5350
-Wire Wire Line
-	8300 5350 7950 5350
-Wire Wire Line
-	7950 5350 7950 5450
-NoConn ~ 8700 5100
 $Comp
 L Connector_Generic:Conn_01x04 J2
@@
 F 2 "" H 3950 5100 50  0001 C CNN
 F 3 "~" H 3950 5100 50  0001 C CNN
+F 4 " " H 0   0   50  0001 C CNN "DNP"
 	1    3950 5100
 	1    0    0    -1
@@
 	1    0    0    -1
 $EndComp
-Wire Wire Line
-	3650 5400 3650 5300
-Wire Wire Line
-	3650 5300 3750 5300
-Text GLabel 3750 5100 0    60   BiDi ~ 0
-CAN_P
-Text GLabel 3750 5200 0    60   BiDi ~ 0
-CAN_N
-Text GLabel 3750 5000 0    50   Output ~ 0
-ENABLE_STBY_SUPPLY
 $Comp
 L Connector_Generic:Conn_01x02 J3
@@
 F 2 "" H 2800 1950 50  0001 C CNN
 F 3 "~" H 2800 1950 50  0001 C CNN
+F 4 " " H 0   0   50  0001 C CNN "DNP"
 	1    2800 1950
 	1    0    0    -1
@@
 F 2 "" H 3800 1950 50  0001 C CNN
 F 3 "~" H 3800 1950 50  0001 C CNN
+F 4 " " H 0   0   50  0001 C CNN "DNP"
 	1    3800 1950
 	-1   0    0    -1
@@
 	1    0    0    -1
 $EndComp
-Wire Wire Line
-	2600 1950 2200 1950
-Wire Wire Line
-	2200 1950 2200 1800
 $Comp
 L power:GND #PWR0128
@@
 	1    0    0    -1
 $EndComp
-Wire Wire Line
-	2500 2150 2500 2050
-Wire Wire Line
-	2500 2050 2600 2050
 $Comp
 L power:GND #PWR0129
@@
 	-1   0    0    -1
 $EndComp
-Wire Wire Line
-	4100 2150 4100 2050
-Wire Wire Line
-	4100 2050 4000 2050
 $Comp
 L power:+12V #PWR0130
@@
 	1    0    0    -1
 $EndComp
-Wire Wire Line
-	4250 1850 4250 1950
-Wire Wire Line
-	4250 1950 4000 1950
 $Comp
 L Connector_Generic:Conn_01x06 J5
@@
 F 2 "" H 8800 1900 50  0001 C CNN
 F 3 "~" H 8800 1900 50  0001 C CNN
+F 4 " " H 0   0   50  0001 C CNN "DNP"
 	1    8800 1900
 	1    0    0    -1
@@
 L power:+3V3 #PWR0131
 U 1 1 5C4905F0
-P 7850 1700
-F 0 "#PWR0131" H 7850 1550 50  0001 C CNN
-F 1 "+3V3" H 7865 1873 50  0000 C CNN
-F 2 "" H 7850 1700 50  0001 C CNN
-F 3 "" H 7850 1700 50  0001 C CNN
-	1    7850 1700
-	1    0    0    -1
-$EndComp
-Wire Wire Line
-	7850 1700 7850 1800
-Wire Wire Line
-	7850 1800 8600 1800
+P 7300 1700
+F 0 "#PWR0131" H 7300 1550 50  0001 C CNN
+F 1 "+3V3" H 7315 1873 50  0000 C CNN
+F 2 "" H 7300 1700 50  0001 C CNN
+F 3 "" H 7300 1700 50  0001 C CNN
+	1    7300 1700
+	1    0    0    -1
+$EndComp
 $Comp
 L power:GND #PWR0132
 U 1 1 5C490708
-P 7850 2400
-F 0 "#PWR0132" H 7850 2150 50  0001 C CNN
-F 1 "GND" H 7855 2227 50  0000 C CNN
-F 2 "" H 7850 2400 50  0001 C CNN
-F 3 "" H 7850 2400 50  0001 C CNN
-	1    7850 2400
-	1    0    0    -1
-$EndComp
-Wire Wire Line
-	7850 2400 7850 1900
-Wire Wire Line
-	7850 1900 8600 1900
-Text GLabel 8100 2000 0    49   Output ~ 0
-PGED
-Text GLabel 8100 2100 0    49   Output ~ 0
-PGEC
-Text GLabel 8600 1700 0    49   Output ~ 0
-nRESET
-NoConn ~ 8600 2200
+P 7300 2400
+F 0 "#PWR0132" H 7300 2150 50  0001 C CNN
+F 1 "GND" H 7305 2227 50  0000 C CNN
+F 2 "" H 7300 2400 50  0001 C CNN
+F 3 "" H 7300 2400 50  0001 C CNN
+	1    7300 2400
+	1    0    0    -1
+$EndComp
 $Comp
 L device:D_TVS D7
@@
 F 2 "" H 8200 2400 50  0001 C CNN
 F 3 "~" H 8200 2400 50  0001 C CNN
+F 4 " " H 0   0   50  0001 C CNN "DNP"
 	1    8200 2400
 	0    1    1    0
@@
 F 2 "" H 8400 2700 50  0001 C CNN
 F 3 "~" H 8400 2700 50  0001 C CNN
+F 4 " " H 0   0   50  0001 C CNN "DNP"
 	1    8400 2700
 	0    1    1    0
 $EndComp
-Wire Wire Line
-	8200 2250 8200 2000
-Wire Wire Line
-	8200 2000 8100 2000
-Wire Wire Line
-	8200 2000 8600 2000
-Connection ~ 8200 2000
-Wire Wire Line
-	8600 2100 8400 2100
 $Comp
 L power:GND #PWR0133
@@
 	1    0    0    -1
 $EndComp
-Wire Wire Line
-	8400 2550 8400 2100
-Connection ~ 8400 2100
-Wire Wire Line
-	8400 2100 8100 2100
+Text GLabel 8700 4700 2    60   Output ~ 0
+USB_5V
+Text GLabel 8700 4900 2    60   BiDi ~ 0
+USB_D+
+Text GLabel 8700 5000 2    60   BiDi ~ 0
+USB_D-
+Text GLabel 3750 5100 0    60   BiDi ~ 0
+CAN_P
+Text GLabel 3750 5200 0    60   BiDi ~ 0
+CAN_N
+Text GLabel 3750 5000 0    50   Output ~ 0
+ENABLE_STBY_SUPPLY
+Text GLabel 7550 2000 0    49   Output ~ 0
+PGED
+Text GLabel 7550 2100 0    49   Output ~ 0
+PGEC
+Text GLabel 8600 1700 0    49   Output ~ 0
+nRESET
 Text Notes 2850 1450 0    197  ~ 0
 POWER
@@
 Text Notes 8100 4200 0    197  ~ 0
 USB
+Wire Wire Line
+	8300 5300 8300 5350
+Wire Wire Line
+	8300 5350 7950 5350
+Wire Wire Line
+	7950 5350 7950 5450
+Wire Wire Line
+	3650 5400 3650 5300
+Wire Wire Line
+	3650 5300 3750 5300
+Wire Wire Line
+	2600 1950 2450 1950
+Wire Wire Line
+	2200 1950 2200 1800
+Wire Wire Line
+	2500 2150 2500 2050
+Wire Wire Line
+	2500 2050 2600 2050
+Wire Wire Line
+	4100 2150 4100 2050
+Wire Wire Line
+	4100 2050 4000 2050
+Wire Wire Line
+	4250 1850 4250 1950
+Wire Wire Line
+	4250 1950 4000 1950
+Wire Wire Line
+	7300 1700 7300 1800
+Wire Wire Line
+	7300 1800 8600 1800
+Wire Wire Line
+	7300 2400 7300 1900
+Wire Wire Line
+	7300 1900 8600 1900
+Wire Wire Line
+	8200 2250 8200 2000
+Wire Wire Line
+	8200 2000 8150 2000
+Wire Wire Line
+	8200 2000 8600 2000
+Wire Wire Line
+	8600 2100 8400 2100
+Wire Wire Line
+	8400 2550 8400 2100
+Wire Wire Line
+	8400 2100 7900 2100
+Connection ~ 8200 2000
+Connection ~ 8400 2100
+NoConn ~ 8700 5100
+NoConn ~ 8600 2200
+$Comp
+L device:R R?
+U 1 1 5B5C8B23
+P 8000 2000
+AR Path="/5B2FB0D8/5B5C8B23" Ref="R?"  Part="1"
+AR Path="/5BC21A84/5B5C8B23" Ref="R?"  Part="1"
+AR Path="/5C8FC872/5C8FC88B/5B5C8B23" Ref="R?"  Part="1"
+AR Path="/5C8FC872/5C8FC88D/5B5C8B23" Ref="R73"  Part="1"
+F 0 "R73" V 7900 2000 50  0000 C CNN
+F 1 "100R" V 8000 2000 50  0000 C CNN
+F 2 "Resistors_SMD:R_0603" V 7930 2000 50  0001 C CNN
+F 3 "~" H 8000 2000 50  0001 C CNN
+F 4 " " H 0   300 50  0001 C CNN "DNP"
+	1    8000 2000
+	0    1    1    0
+$EndComp
+Wire Wire Line
+	7850 2000 7550 2000
+$Comp
+L device:R R?
+U 1 1 5B5C912B
+P 7750 2100
+AR Path="/5B2FB0D8/5B5C912B" Ref="R?"  Part="1"
+AR Path="/5BC21A84/5B5C912B" Ref="R?"  Part="1"
+AR Path="/5C8FC872/5C8FC88B/5B5C912B" Ref="R?"  Part="1"
+AR Path="/5C8FC872/5C8FC88D/5B5C912B" Ref="R72"  Part="1"
+F 0 "R72" V 7650 2100 50  0000 C CNN
+F 1 "100R" V 7750 2100 50  0000 C CNN
+F 2 "Resistors_SMD:R_0603" V 7680 2100 50  0001 C CNN
+F 3 "~" H 7750 2100 50  0001 C CNN
+F 4 " " H -250 400 50  0001 C CNN "DNP"
+	1    7750 2100
+	0    1    1    0
+$EndComp
+Wire Wire Line
+	7600 2100 7550 2100
+$Comp
+L power:PWR_FLAG #FLG0110
+U 1 1 5B60E1EA
+P 2450 1950
+F 0 "#FLG0110" H 2450 2025 50  0001 C CNN
+F 1 "PWR_FLAG" H 2450 2124 50  0000 C CNN
+F 2 "" H 2450 1950 50  0001 C CNN
+F 3 "~" H 2450 1950 50  0001 C CNN
+	1    2450 1950
+	1    0    0    -1
+$EndComp
+Connection ~ 2450 1950
+Wire Wire Line
+	2450 1950 2200 1950
 $EndSCHEMATC
