File: Hardware/DCDC/DCDC_01/DCDC_Controller_old.sch (KiCad schematic (older format))
At the start: 62 parts, among them Q3 Q_NMOS_GDS, U10 OPA320-Q1, U11 TPL0401B-10-Q1, U3 LTC7810

Commit message: Mostly finished DCDC schematic, still needs some values and maybe a soft-start circuit that can be bypassed with 0ohm resister in case it doesn't work.
Parts:
- C24: value 100nF -> 1uF; Voltage 250V -> 50V
- C25: Voltage 250V -> 240V
- C27: value 1uF -> 10uF
- C28, C39: DNP X -> (none)
- C30, C32, C33: value 1uF -> 10uF; Voltage 250V -> 50V
- C34, C35, C37: Voltage 250V -> 50V
- C38: value 1uF -> 4.7uF; Voltage 250V -> 50V
- C78: value 1uF -> C
- C79, C81: value 100nF -> C
- L4, L5: footprint Inductors_SMD:L_0603_HandSoldering -> (none); MPN MPZ1608S300ATAH0 -> (none)
- L6, L7, L8: footprint Inductors_SMD:L_0603_HandSoldering -> (none); MPN MMZ1608B121CTDH5 -> (none)
- Q3: value Q_NMOS_GDS -> Q_NMOS_DGS; footprint TO_SOT_Packages_SMD:TO-263-2 -> (none); symbol device:Q_NMOS_GDS -> device:Q_NMOS_DGS; MPN FDB2532-F085 -> (none)
- R16, R19, R20, R21, R23, R24, R26, R27, R29: footprint Resistors_SMD:R_0603 -> (none)
- R17, R18, R25, R28, R30, R31: value 0R0 -> R; footprint Resistors_SMD:R_0603 -> (none)
- R32: value 20R -> R; footprint Resistors_SMD:R_0603 -> (none)
- R33: value 100k -> R; footprint Resistors_SMD:R_0603 -> (none)
- R34: value 10k -> R; footprint Resistors_SMD:R_0603 -> (none)
- R77: value 22k -> R; footprint Resistors_SMD:R_0603 -> (none)
- U10: footprint TO_SOT_Packages_SMD:SOT-23-5 -> (none); MPN OPA320AQDBVRQ1 -> (none)
- U3: footprint Housings_QFP:TQFP-48-1EP_7x7mm_Pitch0.5mm -> Package_QFP:LQFP-48-1EP_7x7mm_P0.5mm_EP3.6x3.6mm
Connections:
- wire segments 177 -> 174
