File: Hardware/DCDC/DCDC_01/DCDC_Controller.sch (KiCad schematic (older format))
At the start: 62 parts, among them Q3 Q_NMOS_GDS, U10 OPA320-Q1, U11 TPL0401B-10-Q1, U3 LTC7810

Commit message: Updated DCDC schematic with footprints. Moving onto BMS as higher priority. Footprints added, 5V regulator updated
Parts:
- added C84: 100uF, Capacitors_THT:CP_Radial_D16.0mm_P7.50mm, symbol device:CP
- added C85, C86, C87, C88: 1uF, Capacitors_SMD:C_2220, symbol device:C
- added C89: 100nF, Capacitors_SMD:C_0805, symbol device:C
- added C90: 10nF, Capacitors_SMD:C_0805, symbol device:C
- added C91, C92, C93, C94, C95, C96: 10uF, Capacitors_SMD:C_1206, symbol device:C
- added L13, L14: Ferrite_Bead, Inductors_SMD:L_0603_HandSoldering, symbol device:Ferrite_Bead
- added R91, R92: R, symbol device:R
- C21, C22, C26, C28, C29, C31, C36, C40, C49, C50, C79, C81: footprint (none) -> Capacitors_SMD:C_0603
- C23, C45, C46, C47, C48: footprint (none) -> Capacitors_SMD:C_1206
- C25: footprint (none) -> Capacitors_THT:CP_Radial_D16.0mm_P7.50mm
- C27, C30, C32, C33: footprint (none) -> Capacitors_SMD:C_2220
- C34, C35, C78: footprint (none) -> Capacitors_SMD:C_0805
- C39: footprint (none) -> Capacitors_SMD:C_0603; DNP X -> (none)
- C41, C44: footprint (none) -> Capacitors_SMD:CP_Elec_10x10
- U11: footprint Package_TO_SOT_SMD:Texas_R-PDSO-G6 -> TO_SOT_Packages_SMD:Texas_R-PDSO-G6
Connections:
- net labels added: 12V_OLVO_HV, 12V_ULVO_HV, VBATT_FILT_NDRV_HV, VBATT_FILT_PHASE_1_HV, VBATT_FILT_PHASE_2_HV, Vin_HV
- net labels removed: VBATT_FILT, VBATT_FILT_NDRV, Vin
- wire segments 177 -> 234
Other:
- note added: "High Voltage"
- moved on the sheet: U11
