File: Hardware/DCDC/DCDC_01/MicroController.sch (KiCad schematic (older format))
At the start: 0 parts

Commit message: DCDC schematic update and first pass completion. Still needs review and component values
Parts:
- added C1, C2, C3, C4, C5, C6, C7, C9: 100nF, Capacitors_SMD:C_0603, symbol device:C
- added C10, C11: 18pF, Capacitors_SMD:C_0603, symbol device:C
- added C8: 10uF, Capacitors_SMD:C_1206, symbol device:C
- added L1: Ferrite_Bead, Inductors_SMD:L_0603, symbol device:Ferrite_Bead
- added R1, R2: 10k, Resistors_SMD:R_0603, symbol device:R
- added R3: 1M, Resistors_SMD:R_0603, symbol device:R
- added R71, R72, R73: R, symbol device:R
- added SW1: PTS645SM43SMTR92 LFS, Buttons_Switches_SMD:SW_SPST_EVQP0, symbol Switch:SW_Push
- added U1: PIC33EPxxxMU810, Housings_QFP:TQFP-100_14x14mm_Pitch0.5mm, symbol micros:PIC33EPxxxMU810
- added Y1: 8MHz, Crystals:Crystal_SMD_7050-4pin_7.0x5.0mm, symbol device:Crystal_GND24
Connections:
- net labels added: +3.3VA, +3V3, 12V_MONITOR_AI, 5V_MONITOR_AI, CAN_RX, CAN_SLEEP, CAN_TX, DEBUG_LED, DEBUG_PIN, GND, PGEC, PGED, Phase1_Isense_AI, Phase2_Isense_AI, RUN_LTC, SPI_CLK, SPI_DATA, SW_EN, UART_RX, UART_TX, Voltage_Digipot_CS, nRESET
- wire segments 0 -> 172
- no-connect marks 0 -> 64
Other:
- note added: "TO ADD"

Commit message: Mostly finished DCDC schematic, still needs some values and maybe a soft-start circuit that can be bypassed with 0ohm resister in case it doesn't work.
Parts:
- removed R71, R72, R73: R, symbol device:R
- C1, C10, C11, C2, C3, C4, C5, C6, C7, C8, C9: DNP (none) -> (none); Voltage (none) -> 50V; populate y -> (none)
- L1: footprint Inductors_SMD:L_0603 -> Inductors_SMD:L_0603_HandSoldering; DNP (none) -> (none); MPN MPZ1608S300ATDH5 -> MMZ1608B121CTDH5; populate y -> (none)
- R1, R2, R3, SW1, U1, Y1: DNP (none) -> (none); populate y -> (none)
Connections:
- net labels added: I2C_SCL, I2C_SDA
- net labels removed: SPI_CLK, SPI_DATA, Voltage_Digipot_CS
- wire segments 172 -> 169
- no-connect marks 64 -> 65

Commit message: Updated DCDC schematic with footprints. Moving onto BMS as higher priority. Footprints added, 5V regulator updated
Connections:
- net labels added: VBATT_MONITOR_AI
- no-connect marks 65 -> 64
Changed lines of the file:
@@
 Text GLabel 10000 1200 2    59   Output ~ 0
 CAN_SLEEP
-Text GLabel 5600 3700 0    59   Input ~ 0
+Text GLabel 5600 3200 0    59   Input ~ 0
 5V_MONITOR_AI
 Text GLabel 5600 3000 0    59   Input ~ 0
 12V_MONITOR_AI
-Text GLabel 10000 1800 2    60   Output ~ 0
+Text GLabel 10000 1800 2    59   Output ~ 0
 CAN_TX
-Text GLabel 10000 1900 2    60   Input ~ 0
+Text GLabel 10000 1900 2    59   Input ~ 0
 CAN_RX
 Text Notes 1700 950  2    60   ~ 0
@@
 Text GLabel 850  7600 0    60   Input ~ 0
 nRESET
-Text GLabel 5600 4100 0    60   Input ~ 0
+Text GLabel 5600 4100 0    59   Input ~ 0
 PGED
-Text GLabel 5600 4200 0    60   Input ~ 0
+Text GLabel 5600 4200 0    59   Input ~ 0
 PGEC
-Text GLabel 10000 2000 2    60   Output ~ 0
+Text GLabel 10000 2000 2    59   Output ~ 0
 UART_TX
-Text GLabel 10000 2100 2    60   Input ~ 0
+Text GLabel 10000 2100 2    59   Input ~ 0
 UART_RX
 Text GLabel 5600 700  0    60   Output ~ 0
@@
 Text GLabel 5600 2900 0    59   Input ~ 0
 Phase2_Isense_AI
-Text GLabel 10000 2950 2    50   BiDi ~ 0
+Text GLabel 10000 2950 2    59   BiDi ~ 0
 I2C_SCL
-Text GLabel 10000 2850 2    50   BiDi ~ 0
+Text GLabel 10000 2850 2    59   BiDi ~ 0
 I2C_SDA
-Text GLabel 10000 900  2    50   Output ~ 0
+Text GLabel 10000 900  2    59   Output ~ 0
 RUN_LTC
 Wire Wire Line
@@
 NoConn ~ 5600 2600
 NoConn ~ 5600 2700
-NoConn ~ 5600 3200
+NoConn ~ 5600 3700
 NoConn ~ 5600 3300
 NoConn ~ 5600 3400
@@
 NoConn ~ 10000 1000
 NoConn ~ 10000 800
-NoConn ~ 5600 3100
 NoConn ~ 9950 3050
+Text GLabel 5600 3100 0    59   Input ~ 0
+VBATT_MONITOR_AI
 $EndSCHEMATC
