File: Hardware/DCDC/DCDC_01/PowerRails.sch (KiCad schematic (older format))
At the start: 0 parts

Commit message: DCDC schematic update and first pass completion. Still needs review and component values
Parts:
- added C12, C13, C14, C15, C16, C17, C18, C19, C20, C42, C74, C75, C76, C77: C, symbol device:C
- added D1: D_Schottky, symbol device:D_Schottky
- added L2: Ferrite_Bead, symbol device:Ferrite_Bead
- added L3: L, symbol device:L
- added Q1, Q15, Q4: Q_PMOS_DGS, symbol device:Q_PMOS_DGS
- added Q14, Q2, Q5: Q_NMOS_DGS, symbol device:Q_NMOS_DGS
- added R10, R11, R12, R13, R14, R15, R35, R36, R37, R38, R4, R5, R6, R7, R74, R79, R8, R80, R81, R9: R, symbol device:R
- added U2: LTC3638, Package_SO:Linear_MSOP-12-16-1EP_3x4mm_P0.5mm, symbol Regulator_Switching:LTC3638
- added U8, U9: TPS73633DBV, Package_TO_SOT_SMD:SOT-23-5, symbol Regulator_Linear:TPS73633DBV
Connections:
- net labels added: +12P, +12V, +3.3VP, +3V3, +5V, +5VP, +BATT, 12V_MONITOR_AI, 5V_MONITOR_AI, ENABLE_STBY_SUPPLY, GND, SW_EN, VBATT_FILT_5V
- wire segments 0 -> 106
- no-connect marks 0 -> 2
Other:
- note added: "3V3_Always_On"
- note added: "3V3_Switched_power"
- note added: "5V_Always_On"

Commit message: Mostly finished DCDC schematic, still needs some values and maybe a soft-start circuit that can be bypassed with 0ohm resister in case it doesn't work.
Parts:
- removed R11: R, symbol device:R
- added NT9: Net-Tie_2, symbol device:Net-Tie_2
- added R78: 10k, Resistors_SMD:R_0603, symbol device:R
- C12: DNP (none) -> (none); Voltage (none) -> 50V
- C13: value C -> 100nF; DNP (none) -> (none); Voltage (none) -> 250V
- C14: value C -> 10uF; DNP (none) -> (none); Voltage (none) -> 250V
- C15: value C -> 330pF; DNP (none) -> (none); Voltage (none) -> 50V
- C16, C17, C74, C75, C76, C77: value C -> 10uF; DNP (none) -> (none); Voltage (none) -> 50V
- C18, C20, C42: value C -> 100nF; DNP (none) -> (none); Voltage (none) -> 50V
- C19: value C -> 10nF; DNP (none) -> (none); Voltage (none) -> 50V
- D1, L3, Q1, Q14, Q15, Q2, Q4, Q5, R4, R5, R6, R7, R8, R80, R81, R9, U2, U8, U9: DNP (none) -> (none)
- L2: footprint (none) -> Inductors_SMD:L_0603_HandSoldering; DNP (none) -> (none); MPN (none) -> MMZ1608B121CTDH5
- R10: value R -> 3R3; footprint (none) -> Resistors_SMD:R_0603; DNP (none) -> (none)
- R12, R35: value R -> 100k; footprint (none) -> Resistors_SMD:R_0603; DNP (none) -> (none)
- R13: value R -> 47k; footprint (none) -> Resistors_SMD:R_0603; DNP (none) -> (none)
- R14, R36, R37: value R -> 10k; footprint (none) -> Resistors_SMD:R_0603; DNP (none) -> (none)
- R15, R38, R74, R79: value R -> 100R; footprint (none) -> Resistors_SMD:R_0603; DNP (none) -> (none)
Connections:
- wire segments 106 -> 109

Commit message: Updated DCDC schematic with footprints. Moving onto BMS as higher priority. Footprints added, 5V regulator updated
Parts:
- removed Q1: Q_PMOS_DGS, symbol device:Q_PMOS_DGS
- removed Q2, Q5: Q_NMOS_DGS, symbol device:Q_NMOS_DGS
- added C80: 280pF, symbol device:C
- added C83: 100nF, Capacitors_SMD:C_0603, symbol device:C
- added D10, D11, D9: 15V, symbol device:D_Zener
- added Q1: Q_NMOS_DGS, symbol device:Q_NMOS_DGS
- added Q2, Q5: NX1029X,115, symbol ICs:NX1029X,115
- added R82, R85, R89, R90: 10k, Resistors_SMD:R_0603, symbol device:R
- added R83, R87: 100k, Resistors_SMD:R_0603, symbol device:R
- added R84, R88: 47k, Resistors_SMD:R_0603, symbol device:R
- added R86: 100k, symbol device:R
- C12: value C -> 500nF; footprint (none) -> Capacitors_SMD:C_0603
- C14: value 10uF -> 1uF
- C15, C18, C19, C20, C42: footprint (none) -> Capacitors_SMD:C_0603
- C16, C74, C75, C76, C77: footprint (none) -> Capacitors_SMD:C_1206
- C17: footprint (none) -> 1206
- L3: value L -> 220u
- Q14, Q15, R79: DNP (none) -> X
- Q4: DNP (none) -> (none)
- R4: value R -> 1M49; DNP (none) -> X
- R5: value R -> 32k
- R6: value R -> 100R; footprint (none) -> Resistors_SMD:R_0603
- R7: value R -> 1M49
- R8: value R -> 13k
- R80: value R -> 100k; DNP (none) -> X
- R81: value R -> 10k; DNP (none) -> X
- R9: value R -> 176k
- U8, U9: footprint Package_TO_SOT_SMD:SOT-23-5 -> TO_SOT_Packages_SMD:SOT-23-5
Connections:
- net labels added: +BATT_SW_FET_HV, +BATT_SW_GATE_HV, +BATT_SW_HV, 5V_OVLO_HV, 5V_RUN_HV, 5V_SNUB_HV, 5V_SW_NODE_HV, ENABLE_STBY_SUPPLY_PMOS_GATE_HV, VBATT_FILT_5V_HV, VBATT_MONITOR_AI
- net labels removed: VBATT_FILT_5V
- wire segments 109 -> 145
- no-connect marks 2 -> 3
Other:
- note added: "High Voltage"
- note added: "Vin_HV: 40V - 140V\nVout: 5V\nSwitching Freq: 100kHz\nRMS Current: 200mA\nSoftStart 100mS"
- moved on the sheet: U8, U9

Commit message: Too much stuff to list
Parts:
- L3: footprint (none) -> Inductors:Inductor_Taiyo-Yuden_NR-50xx
Changed lines of the file:
@@
 F 0 "L3" V 6490 1850 50  0000 C CNN
 F 1 "220u" V 6399 1850 50  0000 C CNN
-F 2 "" H 6300 1850 50  0001 C CNN
+F 2 "Inductors:Inductor_Taiyo-Yuden_NR-50xx" H 6300 1850 50  0001 C CNN
 F 3 "~" H 6300 1850 50  0001 C CNN
 F 4 " " H 0   0   50  0001 C CNN "DNP"
