File: Hardware/Welder/Welder/Connectors.sch (KiCad schematic (older format))
At the start: 11 parts, among them J1 Conn_01x08, J2 Screw_Terminal_01x03, J3 Screw_Terminal_01x02, J4 Screw_Terminal_01x02

Commit message: Layout for Welder almost complete
Parts:
- added MK1, MK2, MK3, MK4: Mounting_Hole_PAD, symbol mechanical:Mounting_Hole_PAD
Changed lines of the file:
@@
 EESchema Schematic File Version 4
+LIBS:Welder-cache
 EELAYER 26 0
 EELAYER END
@@
 Text Notes 1150 4450 0    98   ~ 0
 HIGH VOLTAGE
+$Comp
+L mechanical:Mounting_Hole_PAD MK1
+U 1 1 5D28CEA3
+P 5250 5350
+F 0 "MK1" H 5350 5401 50  0000 L CNN
+F 1 "Mounting_Hole_PAD" H 5350 5310 50  0000 L CNN
+F 2 "" H 5250 5350 50  0001 C CNN
+F 3 "" H 5250 5350 50  0001 C CNN
+	1    5250 5350
+	1    0    0    -1
+$EndComp
+$Comp
+L power:GND #PWR070
+U 1 1 5D28D3F6
+P 5250 5450
+F 0 "#PWR070" H 5250 5200 50  0001 C CNN
+F 1 "GND" H 5255 5277 50  0000 C CNN
+F 2 "" H 5250 5450 50  0001 C CNN
+F 3 "" H 5250 5450 50  0001 C CNN
+	1    5250 5450
+	1    0    0    -1
+$EndComp
+$Comp
+L mechanical:Mounting_Hole_PAD MK2
+U 1 1 5D28D4D0
+P 5250 5850
+F 0 "MK2" H 5350 5901 50  0000 L CNN
+F 1 "Mounting_Hole_PAD" H 5350 5810 50  0000 L CNN
+F 2 "" H 5250 5850 50  0001 C CNN
+F 3 "" H 5250 5850 50  0001 C CNN
+	1    5250 5850
+	1    0    0    -1
+$EndComp
+$Comp
+L power:GND #PWR071
+U 1 1 5D28D4D7
+P 5250 5950
+F 0 "#PWR071" H 5250 5700 50  0001 C CNN
+F 1 "GND" H 5255 5777 50  0000 C CNN
+F 2 "" H 5250 5950 50  0001 C CNN
+F 3 "" H 5250 5950 50  0001 C CNN
+	1    5250 5950
+	1    0    0    -1
+$EndComp
+$Comp
+L mechanical:Mounting_Hole_PAD MK3
+U 1 1 5D28D6EC
+P 5250 6350
+F 0 "MK3" H 5350 6401 50  0000 L CNN
+F 1 "Mounting_Hole_PAD" H 5350 6310 50  0000 L CNN
+F 2 "" H 5250 6350 50  0001 C CNN
+F 3 "" H 5250 6350 50  0001 C CNN
+	1    5250 6350
+	1    0    0    -1
+$EndComp
+$Comp
+L power:GND #PWR072
+U 1 1 5D28D6F3
+P 5250 6450
+F 0 "#PWR072" H 5250 6200 50  0001 C CNN
+F 1 "GND" H 5255 6277 50  0000 C CNN
+F 2 "" H 5250 6450 50  0001 C CNN
+F 3 "" H 5250 6450 50  0001 C CNN
+	1    5250 6450
+	1    0    0    -1
+$EndComp
+$Comp
+L mechanical:Mounting_Hole_PAD MK4
+U 1 1 5D28D8F5
+P 5250 6850
+F 0 "MK4" H 5350 6901 50  0000 L CNN
+F 1 "Mounting_Hole_PAD" H 5350 6810 50  0000 L CNN
+F 2 "" H 5250 6850 50  0001 C CNN
+F 3 "" H 5250 6850 50  0001 C CNN
+	1    5250 6850
+	1    0    0    -1
+$EndComp
+$Comp
+L power:GND #PWR073
+U 1 1 5D28D8FC
+P 5250 6950
+F 0 "#PWR073" H 5250 6700 50  0001 C CNN
+F 1 "GND" H 5255 6777 50  0000 C CNN
+F 2 "" H 5250 6950 50  0001 C CNN
+F 3 "" H 5250 6950 50  0001 C CNN
+	1    5250 6950
+	1    0    0    -1
+$EndComp
 $EndSCHEMATC

Commit message: a few last layout items
Parts:
- MK1, MK2, MK3, MK4: footprint (none) -> Mounting_Holes:MountingHole_4.3mm_M4_Pad_Via
Changed lines of the file:
@@
 F 2 "Connectors_Samtec:SL-108-X-XX_1x08" H 1850 3400 50  0001 C CNN
 F 3 "~" H 1850 3400 50  0001 C CNN
+F 4 "~" H 0   0   50  0001 C CNN "PartNumber"
 	1    1850 3400
 	-1   0    0    1
@@
 F 0 "MK1" H 5350 5401 50  0000 L CNN
 F 1 "Mounting_Hole_PAD" H 5350 5310 50  0000 L CNN
-F 2 "" H 5250 5350 50  0001 C CNN
-F 3 "" H 5250 5350 50  0001 C CNN
+F 2 "Mounting_Holes:MountingHole_4.3mm_M4_Pad_Via" H 5250 5350 50  0001 C CNN
+F 3 "~" H 5250 5350 50  0001 C CNN
+F 4 "~" H 0   0   50  0001 C CNN "PartNumber"
 	1    5250 5350
 	1    0    0    -1
@@
 F 0 "MK2" H 5350 5901 50  0000 L CNN
 F 1 "Mounting_Hole_PAD" H 5350 5810 50  0000 L CNN
-F 2 "" H 5250 5850 50  0001 C CNN
-F 3 "" H 5250 5850 50  0001 C CNN
+F 2 "Mounting_Holes:MountingHole_4.3mm_M4_Pad_Via" H 5250 5850 50  0001 C CNN
+F 3 "~" H 5250 5850 50  0001 C CNN
+F 4 "~" H 0   0   50  0001 C CNN "PartNumber"
 	1    5250 5850
 	1    0    0    -1
@@
 F 0 "MK3" H 5350 6401 50  0000 L CNN
 F 1 "Mounting_Hole_PAD" H 5350 6310 50  0000 L CNN
-F 2 "" H 5250 6350 50  0001 C CNN
-F 3 "" H 5250 6350 50  0001 C CNN
+F 2 "Mounting_Holes:MountingHole_4.3mm_M4_Pad_Via" H 5250 6350 50  0001 C CNN
+F 3 "~" H 5250 6350 50  0001 C CNN
+F 4 "~" H 0   0   50  0001 C CNN "PartNumber"
 	1    5250 6350
 	1    0    0    -1
@@
 F 0 "MK4" H 5350 6901 50  0000 L CNN
 F 1 "Mounting_Hole_PAD" H 5350 6810 50  0000 L CNN
-F 2 "" H 5250 6850 50  0001 C CNN
-F 3 "" H 5250 6850 50  0001 C CNN
+F 2 "Mounting_Holes:MountingHole_4.3mm_M4_Pad_Via" H 5250 6850 50  0001 C CNN
+F 3 "~" H 5250 6850 50  0001 C CNN
+F 4 "~" H 0   0   50  0001 C CNN "PartNumber"
 	1    5250 6850
 	1    0    0    -1
