File: Hardware/Welder/Welder/Power.sch (KiCad schematic (older format))
At the start: 7 parts, among them U1 LM7805_TO220

Commit message: major CAD update
Parts:
- TR1: footprint Transformers_THT:Transformer_Breve_TEZ-22x24 -> Footprints:FS20-120-C2
Changed lines of the file:
@@
 F 0 "TR1" H 4050 3832 50  0000 C CNN
 F 1 "TRANSF6" H 4050 3741 50  0000 C CNN
-F 2 "Transformers_THT:Transformer_Breve_TEZ-22x24" H 4050 3350 50  0001 C CNN
+F 2 "Footprints:FS20-120-C2" H 4050 3350 50  0001 C CNN
 F 3 "http://catalog.triadmagnetics.com/Asset/FS20-120-C2.pdf" H 4050 3350 50  0001 C CNN
 F 4 "FS20-120-C2" H 2400 2150 50  0001 C CNN "PartNumber"
