File: Hardware/Welder/Welder/Welder.kicad_pcb (KiCad board)
At the start: 2 copper layers, 165 x 95 mm, 70 parts, among them J1 Conn_01x08, J2 Screw_Terminal_01x03, J3 Screw_Terminal_01x02, J4 Screw_Terminal_01x02, Q1 Q_NMOS_GSD, Q2 Q_NMOS_GSD, SW1 SW_Push, SW2 SW_Push, SW3 SW_Push, U1 LM7805_TO220, U2 MOC3052M

Commit message: Layout for Welder almost complete
Parts:
- added C13: 10nF, Capacitors_SMD:C_0603, F.Cu at (98.0, 63.8)
- moved R29 106.2 mm to (112.0, 68.6), turned to 270 degrees
- moved D4 104.4 mm to (94.0, 62.8), turned to 270 degrees
- moved D15 102.2 mm to (112.0, 72.7), turned to 270 degrees
- moved R28 100.4 mm to (115.5, 68.5), turned to 270 degrees
- moved C9 100.2 mm to (147.0, 65.2), turned to 270 degrees
- moved D3 97.7 mm to (96.0, 71.0), turned to 270 degrees
- moved D14 96.1 mm to (115.5, 72.6), turned to 270 degrees
- moved C10 90.3 mm to (133.0, 65.2), turned to 270 degrees
- moved C8 90.3 mm to (119.8, 65.0), turned to 270 degrees
- moved R16 89.3 mm to (85.5, 73.8), turned to 180 degrees
- moved R11 87.5 mm to (121.5, 61.2), turned to 270 degrees
- moved R26 86.7 mm to (97.8, 82.0), turned to 180 degrees
- moved R20 84.8 mm to (89.5, 65.5), turned to 180 degrees
- moved R21 84.7 mm to (93.8, 65.5), turned to 180 degrees
- moved R14 84.7 mm to (133.0, 61.5), turned to 90 degrees
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Routing:
- net +5V: track 0.00 -> 322.4 mm, vias 0 -> 21
- net ZERO_CROSS: track 0.00 -> 80.4 mm
- net GND: track 0.00 -> 80.4 mm, vias 0 -> 28
- net PRI_LO: track 0.00 -> 55.6 mm, vias 0 -> 1
- net MOT_EN: track 0.00 -> 53.4 mm
- net Net-(D2-Pad3): track 0.00 -> 51.6 mm, vias 0 -> 1
- net PRIMARY_A_AI: track 0.00 -> 43.2 mm
- net SDA: track 0.00 -> 41.6 mm
- net SCL: track 0.00 -> 41.6 mm
- net PRIMARY_B_AI: track 0.00 -> 40.5 mm
- net CLK: track 0.00 -> 40.1 mm
- net WELD_BUTTON: track 0.00 -> 37.5 mm, vias 0 -> 2
- net WELD_BUTTON_OUT: track 0.00 -> 37.1 mm
- net Net-(D1-Pad3): track 0.00 -> 35.9 mm
- net Net-(C5-Pad1): track 0.00 -> 34.1 mm
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- added copper zone on B.Cu, net GND
- added copper zone on F.Cu, net GND
- added copper zone on F.Cu, net MOT_+
- added copper zone on F.Cu, net Net-(C1-Pad1)
- added copper zone on F.Cu, net PRI_HI
- added copper zone on F.Cu, net PRI_LO
Other:
- board size 165 x 95 mm -> 125 x 77.2 mm
- net class 5V added: clearance 0.2, trace_width 0.5, via_dia 0.8, via_drill 0.4
- board text added: "5V"
- board text added: "CLK"
- board text added: "CS"
- board text added: "GND"
- board text added: "MISO"
- board text added: "MODE"
- board text added: "MOSI"
- board text added: "MOT WELDER V1.0 2019 ZSL"
- board text added: "MOT+"
- board text added: "PRI_HI"
- board text added: "PRI_LO"
- board text added: "SCL"
- board text added: "SDA"
- board text added: "SELECT"
- board text added: "WELD"

Commit message: a few last layout items
Parts:
- added MK1: Mounting_Hole_PAD, Mounting_Holes:MountingHole_4.3mm_M4_Pad_Via, F.Cu at (164.2, 53.8)
- added MK2: Mounting_Hole_PAD, Mounting_Holes:MountingHole_4.3mm_M4_Pad_Via, F.Cu at (164.2, 119.5)
- added MK3: Mounting_Hole_PAD, Mounting_Holes:MountingHole_4.3mm_M4_Pad_Via, F.Cu at (51.0, 54.0)
- added MK4: Mounting_Hole_PAD, Mounting_Holes:MountingHole_4.3mm_M4_Pad_Via, F.Cu at (51.0, 119.0)
Changed lines of the file:
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@@
     (tracks 468)
     (zones 0)
-    (modules 71)
+    (modules 75)
     (nets 59)
   )
@@
     (last_trace_width 0.25)
     (trace_clearance 0.2)
-    (zone_clearance 1)
+    (zone_clearance 0.508)
     (zone_45_only no)
     (trace_min 0.2)
@@
     (add_net +5V)
   )
+  (module Mounting_Holes:MountingHole_4.3mm_M4_Pad_Via (layer F.Cu)
+    (at 164.25 53.75)
+    (descr "Mounting Hole 4.3mm, M4")
+    (tags "mounting hole 4.3mm m4")
+    (attr virtual)
+    (fp_text reference MK1 (at 0 -5.3) (layer F.SilkS)
+      (effects (font (size 1 1) (thickness 0.15)))
+    )
+    (fp_text value Mounting_Hole_PAD (at 0 5.3) (layer F.Fab)
+      (effects (font (size 1 1) (thickness 0.15)))
+    )
+    (fp_text user %R (at 0.3 0) (layer F.Fab)
+      (effects (font (size 1 1) (thickness 0.15)))
+    )
+    (fp_circle (center 0 0) (end 4.3 0) (layer Cmts.User) (width 0.15))
+    (fp_circle (center 0 0) (end 4.55 0) (layer F.CrtYd) (width 0.05))
+    (pad 1 thru_hole circle (at 0 0) (size 8.6 8.6) (drill 4.3) (layers *.Cu *.Mask)
+      (net 4 GND))
+    (pad 1 thru_hole circle (at 3.225 0) (size 0.9 0.9) (drill 0.6) (layers *.Cu *.Mask)
+      (net 4 GND))
+    (pad 1 thru_hole circle (at 2.280419 2.280419) (size 0.9 0.9) (drill 0.6) (layers *.Cu *.Mask)
+      (net 4 GND))
+    (pad 1 thru_hole circle (at 0 3.225) (size 0.9 0.9) (drill 0.6) (layers *.Cu *.Mask)
+      (net 4 GND))
+    (pad 1 thru_hole circle (at -2.280419 2.280419) (size 0.9 0.9) (drill 0.6) (layers *.Cu *.Mask)
+      (net 4 GND))
+    (pad 1 thru_hole circle (at -3.225 0) (size 0.9 0.9) (drill 0.6) (layers *.Cu *.Mask)
+      (net 4 GND))
+    (pad 1 thru_hole circle (at -2.280419 -2.280419) (size 0.9 0.9) (drill 0.6) (layers *.Cu *.Mask)
+      (net 4 GND))
+    (pad 1 thru_hole circle (at 0 -3.225) (size 0.9 0.9) (drill 0.6) (layers *.Cu *.Mask)
+      (net 4 GND))
+    (pad 1 thru_hole circle (at 2.280419 -2.280419) (size 0.9 0.9) (drill 0.6) (layers *.Cu *.Mask)
+      (net 4 GND))
+  )
+  (module Mounting_Holes:MountingHole_4.3mm_M4_Pad_Via (layer F.Cu)
+    (at 164.25 119.5)
+    (descr "Mounting Hole 4.3mm, M4")
+    (tags "mounting hole 4.3mm m4")
+    (attr virtual)
+    (fp_text reference MK2 (at 0 -5.3) (layer F.SilkS)
+      (effects (font (size 1 1) (thickness 0.15)))
+    )
+    (fp_text value Mounting_Hole_PAD (at 0 5.3) (layer F.Fab)
+      (effects (font (size 1 1) (thickness 0.15)))
+    )
+    (fp_circle (center 0 0) (end 4.55 0) (layer F.CrtYd) (width 0.05))
+    (fp_circle (center 0 0) (end 4.3 0) (layer Cmts.User) (width 0.15))
+    (fp_text user %R (at 0.3 0) (layer F.Fab)
+      (effects (font (size 1 1) (thickness 0.15)))
+    )
+    (pad 1 thru_hole circle (at 2.280419 -2.280419) (size 0.9 0.9) (drill 0.6) (layers *.Cu *.Mask)
+      (net 4 GND))
+    (pad 1 thru_hole circle (at 0 -3.225) (size 0.9 0.9) (drill 0.6) (layers *.Cu *.Mask)
+      (net 4 GND))
+    (pad 1 thru_hole circle (at -2.280419 -2.280419) (size 0.9 0.9) (drill 0.6) (layers *.Cu *.Mask)
+      (net 4 GND))
+    (pad 1 thru_hole circle (at -3.225 0) (size 0.9 0.9) (drill 0.6) (layers *.Cu *.Mask)
+      (net 4 GND))
+    (pad 1 thru_hole circle (at -2.280419 2.280419) (size 0.9 0.9) (drill 0.6) (layers *.Cu *.Mask)
+      (net 4 GND))
+    (pad 1 thru_hole circle (at 0 3.225) (size 0.9 0.9) (drill 0.6) (layers *.Cu *.Mask)
+      (net 4 GND))
+    (pad 1 thru_hole circle (at 2.280419 2.280419) (size 0.9 0.9) (drill 0.6) (layers *.Cu *.Mask)
+      (net 4 GND))
+    (pad 1 thru_hole circle (at 3.225 0) (size 0.9 0.9) (drill 0.6) (layers *.Cu *.Mask)
+      (net 4 GND))
+    (pad 1 thru_hole circle (at 0 0) (size 8.6 8.6) (drill 4.3) (layers *.Cu *.Mask)
+      (net 4 GND))
+  )
+  (module Mounting_Holes:MountingHole_4.3mm_M4_Pad_Via (layer F.Cu)
+    (at 51 54)
+    (descr "Mounting Hole 4.3mm, M4")
+    (tags "mounting hole 4.3mm m4")
+    (attr virtual)
+    (fp_text reference MK3 (at 0 -5.3) (layer F.SilkS)
+      (effects (font (size 1 1) (thickness 0.15)))
+    )
+    (fp_text value Mounting_Hole_PAD (at 0 5.3) (layer F.Fab)
+      (effects (font (size 1 1) (thickness 0.15)))
+    )
+    (fp_circle (center 0 0) (end 4.55 0) (layer F.CrtYd) (width 0.05))
+    (fp_circle (center 0 0) (end 4.3 0) (layer Cmts.User) (width 0.15))
+    (fp_text user %R (at 0.3 0) (layer F.Fab)
+      (effects (font (size 1 1) (thickness 0.15)))
+    )
+    (pad 1 thru_hole circle (at 2.280419 -2.280419) (size 0.9 0.9) (drill 0.6) (layers *.Cu *.Mask)
+      (net 4 GND))
+    (pad 1 thru_hole circle (at 0 -3.225) (size 0.9 0.9) (drill 0.6) (layers *.Cu *.Mask)
+      (net 4 GND))
+    (pad 1 thru_hole circle (at -2.280419 -2.280419) (size 0.9 0.9) (drill 0.6) (layers *.Cu *.Mask)
+      (net 4 GND))
+    (pad 1 thru_hole circle (at -3.225 0) (size 0.9 0.9) (drill 0.6) (layers *.Cu *.Mask)
+      (net 4 GND))
+    (pad 1 thru_hole circle (at -2.280419 2.280419) (size 0.9 0.9) (drill 0.6) (layers *.Cu *.Mask)
+      (net 4 GND))
+    (pad 1 thru_hole circle (at 0 3.225) (size 0.9 0.9) (drill 0.6) (layers *.Cu *.Mask)
+      (net 4 GND))
+    (pad 1 thru_hole circle (at 2.280419 2.280419) (size 0.9 0.9) (drill 0.6) (layers *.Cu *.Mask)
+      (net 4 GND))
+    (pad 1 thru_hole circle (at 3.225 0) (size 0.9 0.9) (drill 0.6) (layers *.Cu *.Mask)
+      (net 4 GND))
+    (pad 1 thru_hole circle (at 0 0) (size 8.6 8.6) (drill 4.3) (layers *.Cu *.Mask)
+      (net 4 GND))
+  )
+  (module Mounting_Holes:MountingHole_4.3mm_M4_Pad_Via (layer F.Cu)
+    (at 51 119)
+    (descr "Mounting Hole 4.3mm, M4")
+    (tags "mounting hole 4.3mm m4")
+    (attr virtual)
+    (fp_text reference MK4 (at 0 -5.3) (layer F.SilkS)
+      (effects (font (size 1 1) (thickness 0.15)))
+    )
+    (fp_text value Mounting_Hole_PAD (at 0 5.3) (layer F.Fab)
+      (effects (font (size 1 1) (thickness 0.15)))
+    )
+    (fp_circle (center 0 0) (end 4.55 0) (layer F.CrtYd) (width 0.05))
+    (fp_circle (center 0 0) (end 4.3 0) (layer Cmts.User) (width 0.15))
+    (fp_text user %R (at 0.3 0) (layer F.Fab)
+      (effects (font (size 1 1) (thickness 0.15)))
+    )
+    (pad 1 thru_hole circle (at 2.280419 -2.280419) (size 0.9 0.9) (drill 0.6) (layers *.Cu *.Mask)
+      (net 4 GND))
+    (pad 1 thru_hole circle (at 0 -3.225) (size 0.9 0.9) (drill 0.6) (layers *.Cu *.Mask)
+      (net 4 GND))
+    (pad 1 thru_hole circle (at -2.280419 -2.280419) (size 0.9 0.9) (drill 0.6) (layers *.Cu *.Mask)
+      (net 4 GND))
+    (pad 1 thru_hole circle (at -3.225 0) (size 0.9 0.9) (drill 0.6) (layers *.Cu *.Mask)
+      (net 4 GND))
+    (pad 1 thru_hole circle (at -2.280419 2.280419) (size 0.9 0.9) (drill 0.6) (layers *.Cu *.Mask)
+      (net 4 GND))
+    (pad 1 thru_hole circle (at 0 3.225) (size 0.9 0.9) (drill 0.6) (layers *.Cu *.Mask)
+      (net 4 GND))
+    (pad 1 thru_hole circle (at 2.280419 2.280419) (size 0.9 0.9) (drill 0.6) (layers *.Cu *.Mask)
+      (net 4 GND))
+    (pad 1 thru_hole circle (at 3.225 0) (size 0.9 0.9) (drill 0.6) (layers *.Cu *.Mask)
+      (net 4 GND))
+    (pad 1 thru_hole circle (at 0 0) (size 8.6 8.6) (drill 4.3) (layers *.Cu *.Mask)
+      (net 4 GND))
+  )
   (module Resistors_THT:R_Axial_DIN0414_L11.9mm_D4.5mm_P15.24mm_Horizontal (layer F.Cu)
     (at 67.5 79.75 270)
@@
     (polygon
       (pts
-        (xy 170 47.75) (xy 170 125) (xy 89.25 125) (xy 89.25 47.75)
-      )
-    )
-  )
-  (zone (net 4) (net_name GND) (layer F.Cu) (hatch edge 0.508)
-    (connect_pads yes (clearance 2))
-    (min_thickness 0.254)
-    (fill yes (arc_segments 16) (thermal_gap 0.508) (thermal_bridge_width 0.508))
-    (polygon
-      (pts
-        (xy 89.28579 125) (xy 45.15579 125) (xy 45.15579 47.75) (xy 89.40579 47.75)
+        (xy 170 125) (xy 45 125) (xy 45 47.75) (xy 170 47.75)
       )
     )

Commit message: major CAD update
Parts:
- TR1: footprint Transformers_THT:Transformer_Breve_TEZ-22x24 -> Footprints:FS20-120-C2
- moved TR1 10.0 mm to (92.7, 95.5)
- moved R3 5.00 mm to (52.5, 105.2)
- moved U1 3.02 mm to (118.0, 87.4)
- moved D1 2.60 mm to (118.0, 106.0)
- moved C1 1.95 mm to (115.0, 98.0)
- moved C2 1.90 mm to (115.0, 92.2)
- moved C4 1.75 mm to (112.2, 84.2)
- moved C3 0.75 mm to (113.0, 82.0)
Routing:
- net Net-(D1-Pad4): track 19.6 -> 44.6 mm
- net Net-(D1-Pad3): track 35.9 -> 12.0 mm
- net GND: track 80.4 -> 69.9 mm, vias 28 -> 69
- net PRI_HI: track 17.6 -> 9.96 mm
- net Net-(C5-Pad1): track 34.1 -> 39.9 mm
- net Net-(R3-Pad2): track 28.8 -> 23.8 mm
- net +5V: track 322.4 -> 326.2 mm
- net MOT_EN: track 53.4 -> 55.2 mm
- net Net-(TR1-Pad6): track 5.00 -> 6.35 mm
- net ZERO_CROSS: track 80.4 -> 79.1 mm
- net MODE_BUTTON: track 31.2 -> 32.4 mm
- net PRI_LO: track 55.6 -> 54.7 mm
Other:
- board text added: "!!!HIGH VOLTAGE!!!"
