File: Hardware/BMS/BMS_01/BattStack.sch (KiCad schematic (older format))
At the start: 23 parts, among them U3 LTC6802-1

Commit message: Updated DCDC schematic with footprints. Moving onto BMS as higher priority. Footprints added, 5V regulator updated
Parts:
- C24: renamed from C16; value C -> 100nF; footprint (none) -> Capacitors_SMD:C_0805
- C25, C26, C27, C28: renamed from C?; footprint (none) -> Capacitors_SMD:C_0603
- L4: renamed from L?; footprint (none) -> Inductors_SMD:L_0603_HandSoldering
- Q1: renamed from Q?; value Q_NMOS_DSG -> Q_NMOS_GSD; footprint (none) -> TO_SOT_Packages_SMD:SOT-23; symbol device:Q_NMOS_DSG -> device:Q_NMOS_GSD
- Q2: renamed from Q?; value Q_PMOS_DGS -> Q_PMOS_GSD; footprint (none) -> TO_SOT_Packages_SMD:SOT-23; symbol device:Q_PMOS_DGS -> device:Q_PMOS_GSD
- R10, R11, R12, R13, R14, R15, R16, R8, R9: renamed from R?; footprint (none) -> Resistors_SMD:R_0603_HandSoldering
- R7: renamed from R2; value R -> 20R0; footprint (none) -> Capacitors_SMD:C_0805
- TH1: renamed from TH?; footprint (none) -> Resistors_SMD:R_0603_HandSoldering
- U5: renamed from U3; footprint (none) -> Housings_SSOP:TSSOP-44_4.4x11.2mm_Pitch0.5mm
- gave numbers to parts that had none: 3
Connections:
- wire segments 200 -> 235

Commit message: Added foorprints for BMS schematics
Parts:
- removed D7: D_Zener, symbol device:D_Zener
- added D6: LED, Diodes_SMD:D_0603, symbol device:LED
- added Q1: Q_NMOS_GSD, TO_SOT_Packages_SMD:SOT-23, symbol device:Q_NMOS_GSD
- added R10, R11: R, Resistors_SMD:R_0603_HandSoldering, symbol device:R
- D7: renamed from D6; value D_Zener -> 15V; footprint (none) -> Diodes_SMD:D_SOD-123
- R20: renamed from R16; value R -> 10k
- renumbered C24 to C26, C25 to C27, C26 to C28, C27 to C29, C28 to C30, Q1 to Q2, Q2 to Q3, R8 to R12, R9 to R13, R10 to R14, R11 to R15, R12 to R16, R13 to R17, R14 to R18, R15 to R19, R7 to R9
Connections:
- net labels added: GPO_LED
- wire segments 235 -> 234

Commit message: Too much stuff to list
Parts:
- L5: renamed from L4; footprint Inductors_SMD:L_0603_HandSoldering -> Inductors_SMD:L_0603
- R70: renamed from R10; footprint Resistors_SMD:R_0603_HandSoldering -> Footprints:R_0603_Standard
- R71: renamed from R11; footprint Resistors_SMD:R_0603_HandSoldering -> Footprints:R_0603_Standard
- R72: renamed from R12; footprint Resistors_SMD:R_0603_HandSoldering -> Footprints:R_0603_Standard
- R73: renamed from R13; footprint Resistors_SMD:R_0603_HandSoldering -> Footprints:R_0603_Standard
- R74: renamed from R14; footprint Resistors_SMD:R_0603_HandSoldering -> Footprints:R_0603_Standard
- R75: renamed from R15; footprint Resistors_SMD:R_0603_HandSoldering -> Footprints:R_0603_Standard
- R76: renamed from R16; footprint Resistors_SMD:R_0603_HandSoldering -> Footprints:R_0603_Standard
- R77: renamed from R17; footprint Resistors_SMD:R_0603_HandSoldering -> Footprints:R_0603_Standard
- R78: renamed from R18; footprint Resistors_SMD:R_0603_HandSoldering -> Footprints:R_0603_Standard
- R79: renamed from R19; footprint Resistors_SMD:R_0603_HandSoldering -> Footprints:R_0603_Standard
- R80: renamed from R20; footprint Resistors_SMD:R_0603_HandSoldering -> Footprints:R_0603_Standard
- TH2: renamed from TH1; footprint Resistors_SMD:R_0603_HandSoldering -> Footprints:R_0603_Standard
- renumbered C26 to C43, C27 to C44, C28 to C45, C29 to C46, C30 to C47, D5 to D44, D6 to D45, D7 to D46, Q1 to Q16, Q2 to Q17, Q3 to Q18, R9 to R69, U5 to U6
Connections:
- wire segments 234 -> 235

Commit message: created HV penthouse. Complete Battery Assembly
Parts:
- C43: footprint Capacitors_SMD:C_0805 -> Capacitor_SMD:C_0805_2012Metric; symbol device:C -> Device:C
- C44, C45, C46, C47: footprint Capacitors_SMD:C_0603 -> Capacitor_SMD:C_0603_1608Metric; symbol device:C -> Device:C
- D44: symbol device:D_TVS -> Device:D_TVS
- D45: footprint Diodes_SMD:D_0603 -> Diode_SMD:D_0603_1608Metric; symbol device:LED -> Device:LED
- D46: footprint Diodes_SMD:D_SOD-123 -> Diode_SMD:D_SOD-123; symbol device:D_Zener -> Device:D_Zener
- L5: footprint Inductors_SMD:L_0603 -> Inductor_SMD:L_0603_1608Metric; symbol device:Ferrite_Bead -> Device:Ferrite_Bead
- Q16, Q17: footprint TO_SOT_Packages_SMD:SOT-23 -> Package_TO_SOT_SMD:SOT-23; symbol device:Q_NMOS_GSD -> Device:Q_NMOS_GSD
- Q18: footprint TO_SOT_Packages_SMD:SOT-23 -> Package_TO_SOT_SMD:SOT-23; symbol device:Q_PMOS_GSD -> Device:Q_PMOS_GSD
- R69: footprint Capacitors_SMD:C_0805 -> Resistor_SMD:R_0603_1608Metric; symbol device:R -> Device:R
- R70, R71, R72, R73, R74, R75, R76, R77, R78, R79: footprint Footprints:R_0603_Standard -> Resistor_SMD:R_0603_1608Metric; symbol device:R -> Device:R
- R80: footprint Footprints:R_0603_Standard -> Resistor_SMD:R_0603_1608Metric; symbol device:R -> Device:R; MPN (none) -> AC0603FR-0710KL
- TH2: footprint Footprints:R_0603_Standard -> Resistor_SMD:R_0603_1608Metric; symbol device:Thermistor_NTC -> Device:Thermistor_NTC
- U6: footprint Housings_SSOP:TSSOP-44_4.4x11.2mm_Pitch0.5mm -> Package_SO:TSSOP-44_4.4x11.2mm_P0.5mm
Connections:
- net labels added: Stack_Top
- wire segments 235 -> 236

Commit message: BMS controller. Lots of new FW including bootloaders
Parts:
- removed C44, C47: C, Capacitor_SMD:C_0603_1608Metric, symbol Device:C
- removed D44: D_TVS, symbol Device:D_TVS
- removed Q16: Q_NMOS_GSD, Package_TO_SOT_SMD:SOT-23, symbol Device:Q_NMOS_GSD
- removed R70, R71, R74: R, Resistor_SMD:R_0603_1608Metric, symbol Device:R
- removed R72: 1M, Resistor_SMD:R_0603_1608Metric, symbol Device:R
- removed R80: 10k, Resistor_SMD:R_0603_1608Metric, symbol Device:R
- removed U6: LTC6802-1, Package_SO:TSSOP-44_4.4x11.2mm_P0.5mm, symbol ICs:LTC6802-1
- added C19, C30: 100nF, Capacitor_SMD:C_0603_1608Metric, symbol Device:C
- added D32: D_Schottky, Diode_SMD:D_SOD-123F, symbol Device:D_Schottky
- added D5: D_TVS, Diode_SMD:D_SMA, symbol Device:D_Zener
- added Q63, Q64, Q65: Q_NPN_BEC, Package_TO_SOT_SMD:SOT-23, symbol Device:Q_NPN_BEC
- added R284, R285, R286: 2k2, Resistor_SMD:R_0603_1608Metric, symbol Device:R
- added U11: LTC6802-2, Package_SO:TSSOP-44_4.4x11.2mm_P0.5mm, symbol ICs:LTC6802-2
- C43: footprint Capacitor_SMD:C_0805_2012Metric -> Capacitor_SMD:C_1206_3216Metric; Digikey_PN (none) -> 445-5851-1-ND; MPN (none) -> CGA5L3X7R2E104K160AA; Part Number (none) -> CGA5L3X7R2E104K160AA
- C45, C46: value C -> 1uF; Digikey_PN (none) -> 445-12539-1-ND; Part Number (none) -> CGA3E1X7R1C105K080AC
- D45: value LED -> D_LED; Digikey_PN (none) -> 160-1447-1-ND; MPN (none) -> LTST-C191KRKT; Part Number (none) -> LTST-C191KRKT
- D46: value 15V -> 12V; footprint Diode_SMD:D_SOD-123 -> Diode_SMD:D_SOD-323F; Digikey_PN (none) -> MM3Z12VCCT-ND; MPN (none) -> MM3Z12VC; Part Number (none) -> MM3Z12VC
- L5: Digikey_PN (none) -> 732-1591-1-ND; MPN (none) -> 742792609; Part Number (none) -> 742792609
- Q17: Digikey_PN (none) -> TN5335K1-GCT-ND; MPN (none) -> TN5335K1-G; Part Number (none) -> TN5335K1-G
- Q18: Digikey_PN (none) -> TP5335K1-GCT-ND; MPN (none) -> TP5335K1-G; Part Number (none) -> TP5335K1-G
- R69: Digikey_PN (none) -> RMCF0603FT20R0CT-ND; MPN (none) -> RMCF0603FT20R0; Part Number (none) -> RMCF0603FT20R0
- R73: value R -> 100R; Digikey_PN (none) -> YAG3561CT-ND; MPN (none) -> AC0603FR-07100RL; Part Number (none) -> AC0603FR-07100RL
- R75: value R -> 10k0; DNP (none) -> < ... >; Digikey_PN (none) -> 311-10KLDCT-ND; MPN (none) -> AC0603FR-0710KL; Part Number (none) -> AC0603FR-0710KL
- R76: value R -> 32k0; Digikey_PN (none) -> 2019-RN73R1JTTD3202B25CT-ND; MPN (none) -> RN73R1JTTD3202B25; Part Number (none) -> RN73R1JTTD3202B25
- R77: value R -> 100k; Digikey_PN (none) -> RMCF0603FT100KCT-ND; MPN (none) -> RMCF0603FT100K; Part Number (none) -> RMCF0603FT100K
- R78: value R -> 499k; Digikey_PN (none) -> RMCF0603FT499KCT-ND; MPN (none) -> RMCF0603FT499K; Part Number (none) -> RMCF0603FT499K
- R79: value R -> 26k1 0.1%; Digikey_PN (none) -> A140602CT-ND; Part Number (none) -> RQ73C1J26K1BTD
- TH2: Digikey_PN (none) -> 495-76084-1-ND; MPN (none) -> B57355V5104F360; Part Number (none) -> B57355V5104F360
Connections:
- net labels added: A0, CSB, CSB_daisy, SCK, SCK_daisy, SDI_daisy, SDO_daisy, Top_of_stack, WDT, ground
- net labels removed: CSBO, GPO_LED, Mode, SCKO, SDIO, Stack_top
- wire segments 236 -> 251
- no-connect marks 0 -> 1
