File: Hardware/BMS/BMS_01/Connectors.sch (KiCad schematic (older format))
At the start: 10 parts

Commit message: BMS Connectors
Connections:
- net labels added: BANK_01, BANK_02, BANK_03, BANK_04, BANK_05, BANK_06, BANK_07, BANK_08, BANK_09, BANK_10, BANK_11, BANK_12
Changed lines of the file:
@@
 L power:+BATT #PWR?
 U 1 1 5C1B76AE
-P 1050 1700
-F 0 "#PWR?" H 1050 1550 50  0001 C CNN
-F 1 "+BATT" H 1065 1873 50  0000 C CNN
-F 2 "" H 1050 1700 50  0001 C CNN
-F 3 "" H 1050 1700 50  0001 C CNN
-	1    1050 1700
+P 900 1200
+F 0 "#PWR?" H 900 1050 50  0001 C CNN
+F 1 "+BATT" H 915 1373 50  0000 C CNN
+F 2 "" H 900 1200 50  0001 C CNN
+F 3 "" H 900 1200 50  0001 C CNN
+	1    900  1200
 	1    0    0    -1
 $EndComp
@@
 L power:GND #PWR?
 U 1 1 5C1B7790
-P 1600 4500
-F 0 "#PWR?" H 1600 4250 50  0001 C CNN
-F 1 "GND" H 1605 4327 50  0000 C CNN
-F 2 "" H 1600 4500 50  0001 C CNN
-F 3 "" H 1600 4500 50  0001 C CNN
-	1    1600 4500
+P 1250 4750
+F 0 "#PWR?" H 1250 4500 50  0001 C CNN
+F 1 "GND" H 1255 4577 50  0000 C CNN
+F 2 "" H 1250 4750 50  0001 C CNN
+F 3 "" H 1250 4750 50  0001 C CNN
+	1    1250 4750
 	1    0    0    -1
 $EndComp
@@
 	3650 5300 3750 5300
 Wire Wire Line
-	1050 1850 1050 1700
-Wire Wire Line
-	1600 4500 1600 4400
-Wire Wire Line
-	1600 4400 1700 4400
+	900  1350 900  1200
+Wire Wire Line
+	1250 4750 1250 4650
+Wire Wire Line
+	1250 4650 1350 4650
 Wire Wire Line
 	7300 1700 7300 1800
@@
 AR Path="/5C8FC872/5C8FC88B/5B5C8B23" Ref="R?"  Part="1"
 AR Path="/5C8FC872/5C8FC88D/5B5C8B23" Ref="R?"  Part="1"
+AR Path="/5B64EF74/5B5C8B23" Ref="R?"  Part="1"
 F 0 "R?" V 7900 2000 50  0000 C CNN
 F 1 "100R" V 8000 2000 50  0000 C CNN
@@
 AR Path="/5C8FC872/5C8FC88B/5B5C912B" Ref="R?"  Part="1"
 AR Path="/5C8FC872/5C8FC88D/5B5C912B" Ref="R?"  Part="1"
+AR Path="/5B64EF74/5B5C912B" Ref="R?"  Part="1"
 F 0 "R?" V 7650 2100 50  0000 C CNN
 F 1 "100R" V 7750 2100 50  0000 C CNN
@@
 L power:PWR_FLAG #FLG?
 U 1 1 5B60E1EA
-P 1300 1850
-F 0 "#FLG?" H 1300 1925 50  0001 C CNN
-F 1 "PWR_FLAG" H 1300 2024 50  0000 C CNN
-F 2 "" H 1300 1850 50  0001 C CNN
-F 3 "~" H 1300 1850 50  0001 C CNN
-	1    1300 1850
-	1    0    0    -1
-$EndComp
-Connection ~ 1300 1850
-Wire Wire Line
-	1300 1850 1050 1850
+P 1150 1350
+F 0 "#FLG?" H 1150 1425 50  0001 C CNN
+F 1 "PWR_FLAG" H 1150 1524 50  0000 C CNN
+F 2 "" H 1150 1350 50  0001 C CNN
+F 3 "~" H 1150 1350 50  0001 C CNN
+	1    1150 1350
+	1    0    0    -1
+$EndComp
+Connection ~ 1150 1350
+Wire Wire Line
+	1150 1350 900  1350
 $Comp
 L Connector_Generic:Conn_01x12 J?
 U 1 1 5B64F388
-P 1900 3900
-F 0 "J?" H 1819 3075 50  0000 C CNN
-F 1 "Conn_01x12" H 1819 3166 50  0000 C CNN
-F 2 "" H 1900 3900 50  0001 C CNN
-F 3 "~" H 1900 3900 50  0001 C CNN
-	1    1900 3900
+P 1900 3950
+F 0 "J?" H 1819 3125 50  0000 C CNN
+F 1 "Conn_01x12" H 1819 3216 50  0000 C CNN
+F 2 "" H 1900 3950 50  0001 C CNN
+F 3 "~" H 1900 3950 50  0001 C CNN
+	1    1900 3950
 	1    0    0    1
 $EndComp
@@
 $EndComp
 Wire Wire Line
-	1300 1850 1700 1850
+	1150 1350 1550 1350
+Text GLabel 1550 3350 0    50   Input ~ 0
+BANK_12
+Text GLabel 1550 3450 0    50   Input ~ 0
+BANK_11
+Text GLabel 1550 3550 0    50   Input ~ 0
+BANK_10
+Text GLabel 1550 3650 0    50   Input ~ 0
+BANK_09
+Text GLabel 1550 3750 0    50   Input ~ 0
+BANK_08
+Text GLabel 1550 3850 0    50   Input ~ 0
+BANK_07
+Text GLabel 1550 3950 0    50   Input ~ 0
+BANK_06
+Text GLabel 1550 4050 0    50   Input ~ 0
+BANK_05
+Text GLabel 1550 4150 0    50   Input ~ 0
+BANK_04
+Text GLabel 1550 4250 0    50   Input ~ 0
+BANK_03
+Text GLabel 1550 4350 0    50   Input ~ 0
+BANK_02
+Text GLabel 1550 4450 0    50   Input ~ 0
+BANK_01
 $EndSCHEMATC

Commit message: Too much stuff to list
Parts:
- removed J? (x2): Conn_01x12, symbol Connector_Generic:Conn_01x12
- removed J?: Conn_01x04, symbol Connector_Generic:Conn_01x04
- added J1, J2: Conn_01x13, Connectors_Molex:Molex_KK-6410-13_13x2.54mm_Straight, symbol Connector_Generic:Conn_01x13
- added J3, J4: Conn_02x12_Top_Bottom, Connectors_Molex:Molex_Microfit3_Header_02x12_Angled_43045-240x, symbol Connector_Generic:Conn_02x12_Top_Bottom
- added J7: Conn_01x16, symbol Connector_Generic:Conn_01x16
- C96: renamed from C?; footprint (none) -> Capacitors_SMD:C_0603
- D86, D87: renamed from D?; footprint (none) -> Diodes_SMD:D_0603
- J5: renamed from J?; footprint (none) -> Connectors:USB_Micro-B_10103594-0001LF
- J6: renamed from J?; footprint (none) -> Connectors_Molex:Molex_KK-6410-06_06x2.54mm_Straight
- R187, R188: renamed from R?; footprint Resistors_SMD:R_0603 -> Footprints:R_0603_Standard
Connections:
- net labels added: BANK_13, BANK_14, BANK_15, BANK_16, BANK_17, BANK_18, BANK_19, BANK_20, BANK_21, BANK_22, BANK_23, BANK_24, NTC_10_OUT, NTC_10_RTN, NTC_11_OUT, NTC_11_RTN, NTC_12_OUT, NTC_12_RTN, NTC_13_OUT, NTC_13_RTN, NTC_14_OUT, NTC_14_RTN, NTC_15_OUT, NTC_15_RTN, NTC_16_OUT, NTC_16_RTN, NTC_17_OUT, NTC_17_RTN, NTC_18_OUT, NTC_18_RTN, NTC_19_OUT, NTC_19_RTN, NTC_1_OUT, NTC_1_RTN, NTC_20_OUT, NTC_20_RTN, NTC_21_OUT, NTC_21_RTN, NTC_22_OUT, NTC_22_RTN, NTC_23_OUT, NTC_23_RTN, NTC_24_OUT, NTC_24_RTN, NTC_2_OUT, NTC_2_RTN, NTC_3_OUT, NTC_3_RTN, NTC_4_OUT, NTC_4_RTN, NTC_5_OUT, NTC_5_RTN, NTC_6_OUT, NTC_6_RTN, NTC_7_OUT, NTC_7_RTN, NTC_8_OUT, NTC_8_RTN, NTC_9_OUT, NTC_9_RTN, Transducer_Input, Transducer_Pwr, Transducer_Ref
- net labels removed: ENABLE_STBY_SUPPLY
- wire segments 22 -> 23
- no-connect marks 2 -> 12
Other:
- note added: "CAN"
- note added: "DEBUG/JTAG"
- note added: "NTCs"
- note removed: "DEBUG"
- note removed: "SIGNAL"

Commit message: created HV penthouse. Complete Battery Assembly
Parts:
- removed J1, J2: Conn_01x13, Connectors_Molex:Molex_KK-6410-13_13x2.54mm_Straight, symbol Connector_Generic:Conn_01x13
- removed J3, J4: Conn_02x12_Top_Bottom, Connectors_Molex:Molex_Microfit3_Header_02x12_Angled_43045-240x, symbol Connector_Generic:Conn_02x12_Top_Bottom
- removed J7: Conn_01x16, symbol Connector_Generic:Conn_01x16
- added J1, J2, J3, J4: Conn_01x07, Connector_JST:JST_GH_BM08B-GHS-TBT_1x08-1MP_P1.25mm_Vertical, symbol Connector_Generic:Conn_01x07
- added J10: Conn_01x02, Connector_JST:JST_EH_B2B-EH-A_1x02_P2.50mm_Vertical, symbol Connector_Generic:Conn_01x02
- added J11, J9: Conn_01x04, Connector_JST:JST_SH_BM04B-SRSS-TB_1x04-1MP_P1.00mm_Vertical, symbol Connector_Generic:Conn_01x04
- added J12: Conn_01x02, Connector_JST:JST_EH_B3B-EH-A_1x03_P2.50mm_Vertical, symbol Connector_Generic:Conn_01x03
- added J5, J6, J7, J8: Conn_02x06_Top_Bottom, Connector_JST:JST_SH_BM12B-SRSS-TB_1x12-1MP_P1.00mm_Vertical, symbol Connector_Generic:Conn_02x06_Top_Bottom
- C96: footprint Capacitors_SMD:C_0603 -> Capacitor_SMD:C_0603_1608Metric; symbol device:C -> Device:C
- D86, D87: footprint Diodes_SMD:D_0603 -> Diode_SMD:D_0603_1608Metric; symbol device:D_TVS -> Device:D_TVS
- J13: renamed from J6; footprint Connectors_Molex:Molex_KK-6410-06_06x2.54mm_Straight -> Connector_Molex:Molex_KK-254_AE-6410-06A_1x06_P2.54mm_Vertical
- J14: renamed from J5; footprint Connectors:USB_Micro-B_10103594-0001LF -> Connector_USB:USB_Micro-B_Molex-105017-0001
- R187, R188: footprint Footprints:R_0603_Standard -> Resistor_SMD:R_0603_1608Metric; symbol device:R -> Device:R; MPN (none) -> AC0603FR-07100RL
Connections:
- net labels added: 12V_POWER, BANK_00, CONTACTOR_PWM_OUT, PRE_CHARGE_OUT
- no-connect marks 12 -> 2
Other:
- note added: "Balancing"

Commit message: BMS controller. Lots of new FW including bootloaders
Parts:
- removed D86, D87: D_TVS, Diode_SMD:D_0603_1608Metric, symbol Device:D_TVS
- removed J10: Conn_01x02, Connector_JST:JST_EH_B2B-EH-A_1x02_P2.50mm_Vertical, symbol Connector_Generic:Conn_01x02
- removed J12: Conn_01x02, Connector_JST:JST_EH_B3B-EH-A_1x03_P2.50mm_Vertical, symbol Connector_Generic:Conn_01x03
- removed J5, J6, J7, J8: Conn_02x06_Top_Bottom, Connector_JST:JST_SH_BM12B-SRSS-TB_1x12-1MP_P1.00mm_Vertical, symbol Connector_Generic:Conn_02x06_Top_Bottom
- added D28, D29: D_Schottky_x2_ACom_AKK, Footprints:D_SOT-23_ANK, symbol Device:D_Schottky_x2_ACom_AKK
- added J10, J17, J18, J19: 7807, Footprints:7807, symbol Connectors:7807
- added J12, J15, J16, J20: Conn_01x02, Connector_JST:JST_XH_B2B-XH-A_1x02_P2.50mm_Vertical, symbol Connector_Generic:Conn_01x02
- added J5, J6, J7, J8: Conn_02x06_Odd_Even, Connector_PinHeader_2.54mm:PinHeader_2x06_P2.54mm_Vertical, symbol Connector_Generic:Conn_02x06_Odd_Even
- C96: value C -> 100nF; Digikey_PN (none) -> 490-4779-1-ND; MPN (none) -> GCM188R71H104KA57D; Part Number (none) -> GCM188R71H104KA57D
- J1: footprint Connector_JST:JST_GH_BM08B-GHS-TBT_1x08-1MP_P1.25mm_Vertical -> Connector_JST:JST_XH_B7B-XH-A_1x07_P2.50mm_Vertical
- J11, J9: footprint Connector_JST:JST_SH_BM04B-SRSS-TB_1x04-1MP_P1.00mm_Vertical -> Connector_JST:JST_XH_B4B-XH-A_1x04_P2.50mm_Vertical
- J13: footprint Connector_Molex:Molex_KK-254_AE-6410-06A_1x06_P2.54mm_Vertical -> Connector_JST:JST_XH_B6B-XH-A_1x06_P2.50mm_Vertical
- J2, J3, J4: value Conn_01x07 -> Conn_01x06; footprint Connector_JST:JST_GH_BM08B-GHS-TBT_1x08-1MP_P1.25mm_Vertical -> Connector_JST:JST_XH_B6B-XH-A_1x06_P2.50mm_Vertical; symbol Connector_Generic:Conn_01x07 -> Connector_Generic:Conn_01x06
- R187, R188: Digikey_PN (none) -> YAG3561CT-ND; Part Number (none) -> AC0603FR-07100RL
Connections:
- net labels added: CONTACTOR_PWM_1_OUT, CONTACTOR_PWM_2_OUT, GND1, HV_DCDC_OUTPUT, HV_EV_CHARGER_INPUT, HV_PRECHARGE_OUT, SHUNT_N, SHUNT_P
- net labels removed: BANK_00, CONTACTOR_PWM_OUT, NTC_10_RTN, NTC_11_RTN, NTC_12_RTN, NTC_13_RTN, NTC_14_RTN, NTC_15_RTN, NTC_16_RTN, NTC_17_RTN, NTC_18_RTN, NTC_19_RTN, NTC_1_RTN, NTC_20_RTN, NTC_21_RTN, NTC_22_RTN, NTC_23_RTN, NTC_24_RTN, NTC_2_RTN, NTC_3_RTN, NTC_4_RTN, NTC_5_RTN, NTC_6_RTN, NTC_7_RTN, NTC_8_RTN, NTC_9_RTN, PRE_CHARGE_OUT
- wire segments 23 -> 59
- no-connect marks 2 -> 3
