File: Hardware/BMS/BMS_01/Contactor.sch (KiCad schematic (older format))
At the start: 21 parts, among them Q31 MMBTA42-7-F, Q32 SQJ431EP-T1_GE3, U11 BTS3050EJXUMA1

Commit message: BMS controller. Lots of new FW including bootloaders
Parts:
- removed C107: 10n, Capacitor_SMD:C_0603_1608Metric, symbol Device:C
- removed Q32: SQJ431EP-T1_GE3, Package_SO:PowerPAK_SO-8_Single, symbol ICs:BUK9Y3R0-40E,115
- removed R102, R98: R, Resistor_SMD:R_0603_1608Metric, symbol Device:R
- removed R106, R66, R82, R86: 10k, Resistor_SMD:R_0603_1608Metric, symbol Device:R
- removed U11: BTS3050EJXUMA1, Package_SO:TI_SO-PowerPAD-8_ThermalVias, symbol HSD:BTS3050EJXUMA1
- added C117, C118: 10nF, Capacitor_SMD:C_0603_1608Metric, symbol Device:C
- added D10: 12V, Diode_SMD:D_SOD-323F, symbol Device:D_Zener
- added D11, D13: D_Schottky, Diode_SMD:D_SMA, symbol Device:D_Schottky
- added D22: D_TVS, Diode_SMD:D_SMB, symbol Device:D_Zener
- added Q34: Q_NPN_BEC, Package_TO_SOT_SMD:SOT-23, symbol Device:Q_NPN_BEC
- added Q35: Q_PMOS_GDS, Package_TO_SOT_SMD:TO-263-2, symbol Device:Q_PMOS_GDS
- added Q36: TPH3300CNH,L1Q, Package_SO:PowerPAK_SO-8_Single, symbol ICs:Q_NMOS_SSSGD
- added Q58, Q59: RQ3G100GNTB, Package_TO_SOT_SMD:LFPAK33, symbol ICs:Q_NMOS_SSSGD
- added R122, R126, R134, R203, R206: 10k0, Resistor_SMD:R_0603_1608Metric, symbol Device:R
- added R193, R269: 100k, Resistor_SMD:R_0603_1608Metric, symbol Device:R
- added R204, R205: 100R, Resistor_SMD:R_0603_1608Metric, symbol Device:R
- added R208: 1M, Resistor_SMD:R_0603_1608Metric, symbol Device:R
- added U15, U16: TLX9185A(GBTPL,F, Package_SO:SO-4_4.4x3.9mm_P2.54mm, symbol Isolator:SFH617A-1
- C106: value 10n -> 10nF; Digikey_PN (none) -> 490-4781-1-ND; MPN (none) -> GCM188R72A103KA37D; Part Number (none) -> GCM188R72A103KA37D
- Q31: value MMBTA42-7-F -> Q_NPN_BEC; Digikey_PN (none) -> FMMTA42CT-ND; MPN (none) -> MMBTA42-7-F; Part Number (none) -> MMBTA42-7-F
- R34, R94: value 10k -> 10k0; Digikey_PN (none) -> 311-10KLDCT-ND; Part Number (none) -> AC0603FR-0710KL
- R38, R42, R46, R62: value R -> 100k; Digikey_PN (none) -> RMCF0603FT100KCT-ND; MPN (none) -> RMCF0603FT100K; Part Number (none) -> RMCF0603FT100K
- R50: value 1k -> 100R; footprint Resistor_THT:R_Axial_Power_L38.0mm_W9.0mm_P45.72mm -> Resistor_THT:R_Axial_Power_L50.0mm_W9.0mm_P55.88mm; Digikey_PN (none) -> 100W-10-ND; MPN (none) -> SQP10AJB-100R; Part Number (none) -> SQP10AJB-100R
- R54, R58: value R -> 1M; DNP (none) -> < ... >; Digikey_PN (none) -> 311-1MLDCT-ND; MPN (none) -> AC0603FR-071ML; Part Number (none) -> AC0603FR-071ML
- R90: value 10k -> 100k; Digikey_PN (none) -> RMCF0603FT100KCT-ND; MPN AC0603FR-0710KL -> RMCF0603FT100K; Part Number (none) -> RMCF0603FT100K
Connections:
- net labels added: +5VL, CONTACTOR_PWM_1, CONTACTOR_PWM_1_OUT, CONTACTOR_PWM_2, CONTACTOR_PWM_2_OUT, DISCHARGE_EN, GND1, HV_BUS_VOLTAGE_AI, HV_PRECHARGE_OUT, HV_precharge_gate, HV_precharge_switch
- net labels removed: +3.3V, 12V_POWER_MONITOR_AI, CONTACTOR_PWM, CONTACTOR_PWM_OUT, CONTACTOR_STATUS, HV_BUS_MONITOR_AI, PRE_CHARGE_OUT
- wire segments 52 -> 88
Other:
- note added: "Circuit sized for minimum 100 ohm series resistor."
- note added: "LOW VOLTAGE DOMAIN"
- note removed: "Contactor 12V Monitor"
- note removed: "Wrong symbol but OK because footprint is correct"
