File: Hardware/BMS/BMS_01/NTC.sch (KiCad schematic (older format))
At the start: 3 parts

Commit message: Too much stuff to list
Parts:
- R171: renamed from R139; footprint Resistors_SMD:R_0603_HandSoldering -> Footprints:R_0603_Standard
- R172: renamed from R140; footprint Resistors_SMD:R_0603_HandSoldering -> Footprints:R_0603_Standard
- renumbered C72 to C88

Commit message: created HV penthouse. Complete Battery Assembly
Parts:
- C88: value C -> 10n; footprint Capacitors_SMD:C_0603 -> Capacitor_SMD:C_0603_1608Metric; symbol device:C -> Device:C
- R171, R172: value R -> 10k; footprint Footprints:R_0603_Standard -> Resistor_SMD:R_0603_1608Metric; symbol device:R -> Device:R; MPN (none) -> AC0603FR-0710KL
Changed lines of the file:
@@
 $Descr A4 11693 8268
 encoding utf-8
-Sheet 42 58
+Sheet 44 59
 Title ""
 Date ""
@@
 $EndDescr
 $Comp
-L device:R R?
+L Device:R R?
 U 1 1 5B579950
 P 5850 3550
@@
 AR Path="/5B5CD4CD/5B5CD608/5B5E0A0D/5B579950" Ref="R186"  Part="1"
 F 0 "R186" H 5920 3596 50  0000 L CNN
-F 1 "R" H 5920 3505 50  0000 L CNN
-F 2 "Footprints:R_0603_Standard" V 5780 3550 50  0001 C CNN
-F 3 "~" H 5850 3550 50  0001 C CNN
+F 1 "10k" H 5920 3505 50  0000 L CNN
+F 2 "Resistor_SMD:R_0603_1608Metric" V 5780 3550 50  0001 C CNN
+F 3 "http://www.yageo.com/NewPortal/yageodocoutput?fileName=/pdf/R-Chip/PYu-AC_51_RoHS_L_6.pdf" H 5850 3550 50  0001 C CNN
+F 4 "AC0603FR-0710KL" H 0   0   50  0001 C CNN "MPN"
 	1    5850 3550
 	1    0    0    -1
 $EndComp
 $Comp
-L device:R R?
+L Device:R R?
 U 1 1 5B57995D
 P 5600 3800
@@
 AR Path="/5B5CD4CD/5B5CD608/5B5E0A0D/5B57995D" Ref="R185"  Part="1"
 F 0 "R185" V 5393 3800 50  0000 C CNN
-F 1 "R" V 5484 3800 50  0000 C CNN
-F 2 "Footprints:R_0603_Standard" V 5530 3800 50  0001 C CNN
-F 3 "~" H 5600 3800 50  0001 C CNN
+F 1 "10k" V 5484 3800 50  0000 C CNN
+F 2 "Resistor_SMD:R_0603_1608Metric" V 5530 3800 50  0001 C CNN
+F 3 "http://www.yageo.com/NewPortal/yageodocoutput?fileName=/pdf/R-Chip/PYu-AC_51_RoHS_L_6.pdf" H 5600 3800 50  0001 C CNN
+F 4 "AC0603FR-0710KL" H 0   0   50  0001 C CNN "MPN"
 	1    5600 3800
 	0    1    1    0
 $EndComp
 $Comp
-L device:C C?
+L Device:C C?
 U 1 1 5B579964
 P 5250 4050
@@
 AR Path="/5B5CD4CD/5B5CD608/5B5E0A0D/5B579964" Ref="C95"  Part="1"
 F 0 "C95" H 5365 4096 50  0000 L CNN
-F 1 "C" H 5365 4005 50  0000 L CNN
-F 2 "Capacitors_SMD:C_0603" H 5288 3900 50  0001 C CNN
+F 1 "10n" H 5365 4005 50  0000 L CNN
+F 2 "Capacitor_SMD:C_0603_1608Metric" H 5288 3900 50  0001 C CNN
 F 3 "~" H 5250 4050 50  0001 C CNN
 	1    5250 4050

Commit message: BMS controller. Lots of new FW including bootloaders
Parts:
- C88: value 10n -> 10nF; Digikey_PN (none) -> 490-4781-1-ND; MPN (none) -> GCM188R72A103KA37D; Part Number (none) -> GCM188R72A103KA37D
- R171, R172: value 10k -> 10k0; Digikey_PN (none) -> 311-10KLDCT-ND; Part Number (none) -> AC0603FR-0710KL
Changed lines of the file:
@@
 $Descr A4 11693 8268
 encoding utf-8
-Sheet 44 59
+Sheet 54 61
 Title ""
 Date ""
@@
 AR Path="/5B5CD4CD/5B5CD608/5B5E0A0D/5B579950" Ref="R186"  Part="1"
 F 0 "R186" H 5920 3596 50  0000 L CNN
-F 1 "10k" H 5920 3505 50  0000 L CNN
+F 1 "10k0" H 5920 3505 50  0000 L CNN
 F 2 "Resistor_SMD:R_0603_1608Metric" V 5780 3550 50  0001 C CNN
 F 3 "http://www.yageo.com/NewPortal/yageodocoutput?fileName=/pdf/R-Chip/PYu-AC_51_RoHS_L_6.pdf" H 5850 3550 50  0001 C CNN
 F 4 "AC0603FR-0710KL" H 0   0   50  0001 C CNN "MPN"
+F 5 "AC0603FR-0710KL" H 0   0   50  0001 C CNN "Part Number"
+F 6 "311-10KLDCT-ND" H 0   0   50  0001 C CNN "Digikey_PN"
 	1    5850 3550
 	1    0    0    -1
@@
 AR Path="/5B5CD4CD/5B5CD608/5B5E0A0D/5B57995D" Ref="R185"  Part="1"
 F 0 "R185" V 5393 3800 50  0000 C CNN
-F 1 "10k" V 5484 3800 50  0000 C CNN
+F 1 "10k0" V 5484 3800 50  0000 C CNN
 F 2 "Resistor_SMD:R_0603_1608Metric" V 5530 3800 50  0001 C CNN
 F 3 "http://www.yageo.com/NewPortal/yageodocoutput?fileName=/pdf/R-Chip/PYu-AC_51_RoHS_L_6.pdf" H 5600 3800 50  0001 C CNN
 F 4 "AC0603FR-0710KL" H 0   0   50  0001 C CNN "MPN"
+F 5 "AC0603FR-0710KL" H 0   0   50  0001 C CNN "Part Number"
+F 6 "311-10KLDCT-ND" H 0   0   50  0001 C CNN "Digikey_PN"
 	1    5600 3800
 	0    1    1    0
@@
 AR Path="/5B5CD4CD/5B5CD608/5B5E0A0D/5B579964" Ref="C95"  Part="1"
 F 0 "C95" H 5365 4096 50  0000 L CNN
-F 1 "10n" H 5365 4005 50  0000 L CNN
+F 1 "10nF" H 5365 4005 50  0000 L CNN
 F 2 "Capacitor_SMD:C_0603_1608Metric" H 5288 3900 50  0001 C CNN
 F 3 "~" H 5250 4050 50  0001 C CNN
+F 4 "GCM188R72A103KA37D" H 0   0   50  0001 C CNN "MPN"
+F 5 "GCM188R72A103KA37D" H 0   0   50  0001 C CNN "Part Number"
+F 6 "490-4781-1-ND" H 0   0   50  0001 C CNN "Digikey_PN"
 	1    5250 4050
 	1    0    0    -1
