File: Hardware/BMS/BMS_01/PowerRails.sch (KiCad schematic (older format))
At the start: 15 parts, among them U2 LTC3639

Commit message: Updated DCDC schematic with footprints. Moving onto BMS as higher priority. Footprints added, 5V regulator updated
Parts:
- removed C? (x2): C, symbol device:C
- removed U2: LTC3639, symbol ICs:LTC3639
- removed U?: TPS76350, TO_SOT_Packages_SMD:SOT-23-5, symbol regul:TPS76350
- added C10, C12, C15, C16: 10uF, Capacitors_SMD:C_1206, symbol device:C
- added C17: 500nF, Capacitors_SMD:C_0603, symbol device:C
- added C18: 280pF, Capacitors_SMD:C_0603, symbol device:C
- added C19: C, Capacitors_SMD:C_0603, symbol device:C
- added C23: 10nF, Capacitors_SMD:C_0603, symbol device:C
- added D4: D_Schottky, symbol device:D_Schottky
- added R5: 176k, Resistors_SMD:R_0603_HandSoldering, symbol device:R
- added R6: 3R3, Resistors_SMD:R_0603_HandSoldering, symbol device:R
- added U2, U3: TPS73633DBV, Package_TO_SOT_SMD:SOT-23-5, symbol Regulator_Linear:TPS73633DBV
- added U4: LTC3638, Package_SO:Linear_MSOP-12-16-1EP_3x4mm_P0.5mm, symbol Regulator_Switching:LTC3638
- C11: renamed from C10; value C -> 100nF; footprint (none) -> Capacitors_SMD:C_1206
- C13: renamed from C11; value C -> 100nF; footprint (none) -> Capacitors_SMD:C_1206
- C14: renamed from C12; value C -> 1uF; footprint (none) -> Capacitors_SMD:C_2220
- C20: renamed from C13; value C -> 10uF; footprint (none) -> Capacitors_SMD:C_1206
- C21: renamed from C14; value C -> 10uF; footprint (none) -> Capacitors_SMD:C_1206
- C22: renamed from C15; value C -> 100nF; footprint (none) -> Capacitors_SMD:C_0603
- L2: footprint (none) -> Inductors_SMD:L_1206
- L3: value 470uH -> 220u; MPN SRR0745A-471M -> (none)
- R2: renamed from R?; value R -> 1M49; footprint (none) -> Resistors_SMD:R_0603_HandSoldering
- R3: renamed from R?; value R -> 32k0; footprint (none) -> Resistors_SMD:R_0603_HandSoldering
- R4: renamed from R?; value R -> 13k0; footprint (none) -> Resistors_SMD:R_0603_HandSoldering
Connections:
- net labels added: +3.3V, SW_EN
- net labels removed: +12VA, +5VA
- wire segments 44 -> 66
- no-connect marks 0 -> 1
Other:
- note added: "3V3 Always On"
- note added: "3V3 Switched (External)"
- note added: "5V Always On"
- note added: "Vin_HV: 40V - 140V\nVout: 5V\nSwitching Freq: 100kHz\nRMS Current: 200mA\nSoftStart 100mS"

Commit message: Added foorprints for BMS schematics
Parts:
- U2, U3: footprint Package_TO_SOT_SMD:SOT-23-5 -> TO_SOT_Packages_SMD:SOT-23-5
- U4: footprint Package_SO:Linear_MSOP-12-16-1EP_3x4mm_P0.5mm -> Housings_SSOP:Linear_MSOP-12-16-1EP_3x4mm_Pitch0.5mm
- renumbered C10 to C12, C11 to C13, C12 to C14, C13 to C15, C14 to C16, C15 to C17, C16 to C18, C17 to C19, C18 to C20, C19 to C21, C20 to C22, C21 to C23, C22 to C24, C23 to C25, R2 to R4, R3 to R5, R4 to R6, R5 to R7, R6 to R8
Connections:
- net labels added: +3.3VP, +BATT
- wire segments 66 -> 67

Commit message: Too much stuff to list
Parts:
- added C103, C97: C, Capacitors_SMD:C_0603, symbol device:C
- added L7, L8: Ferrite_Bead, Inductors_SMD:L_0603, symbol device:Ferrite_Bead
- added NT1: Net-Tie_2, Footprints:Net_Tie-0.5mm, symbol device:Net-Tie_2
- added R193, R199: 100R, Footprints:R_0603_Standard, symbol device:R
- added R200, R201: 10k0, Footprints:R_0603_Standard, symbol device:R
- added R202: R, Footprints:R_0603_Standard, symbol device:R
- added U9: TPS2551-Q1, TO_SOT_Packages_SMD:SOT-23-6, symbol HSD:TPS2551-Q1
- D4: footprint (none) -> Diodes_SMD:D_SOD-123F; MPN (none) -> ACDBMT1200-HF
- L2: footprint Inductors_SMD:L_1206 -> Inductors_SMD:L_0603
- L3: footprint (none) -> Inductors:Inductor_Taiyo-Yuden_NR-60xx; MPN (none) -> TYS6045221M-10
- R4, R5, R6, R7, R8: footprint Resistors_SMD:R_0603_HandSoldering -> Footprints:R_0603_Standard
Connections:
- net labels added: +5VP, 5V_SW_nFAULT, FB_5V, SWITCH_NODE_5V, VBATT_FILT_5V_IN
- wire segments 67 -> 98
- no-connect marks 1 -> 3
Other:
- note added: "5V Switched (External)"
- note added: "TODO:\nUpdate Diode Footprint"
- moved on the sheet: U2

Commit message: created HV penthouse. Complete Battery Assembly
Parts:
- added C104: 100nF, Capacitor_SMD:C_1206_3216Metric, symbol Device:C
- added C105: 100nF, Capacitor_SMD:C_0805_2012Metric, symbol Device:C
- added D8: D_TVS, symbol Device:D_TVS
- C103, C19, C20, C21, C24, C25, C97: footprint Capacitors_SMD:C_0603 -> Capacitor_SMD:C_0603_1608Metric; symbol device:C -> Device:C
- C12, C13, C14, C15, C17, C18, C22, C23: footprint Capacitors_SMD:C_1206 -> Capacitor_SMD:C_1206_3216Metric; symbol device:C -> Device:C
- C16: footprint Capacitors_SMD:C_2220 -> Capacitor_SMD:C_2220_5650Metric; symbol device:C -> Device:C
- D4: footprint Diodes_SMD:D_SOD-123F -> Diode_SMD:D_SOD-123F; symbol device:D_Schottky -> Device:D_Schottky
- L2, L7, L8: footprint Inductors_SMD:L_0603 -> Inductor_SMD:L_0603_1608Metric; symbol device:Ferrite_Bead -> Device:Ferrite_Bead
- L3: symbol device:L -> Device:L
- NT1: symbol device:Net-Tie_2 -> Device:Net-Tie_2
- R193, R199: footprint Footprints:R_0603_Standard -> Resistor_SMD:R_0603_1608Metric; symbol device:R -> Device:R; MPN (none) -> AC0603FR-07100RL
- R200, R201, R202, R4, R5, R6, R7, R8: footprint Footprints:R_0603_Standard -> Resistor_SMD:R_0603_1608Metric; symbol device:R -> Device:R
- U2, U3: footprint TO_SOT_Packages_SMD:SOT-23-5 -> Package_TO_SOT_SMD:SOT-23-5
- U4: footprint Housings_SSOP:Linear_MSOP-12-16-1EP_3x4mm_Pitch0.5mm -> Package_SO:Linear_MSOP-12-16-1EP_3x4mm_P0.5mm
- U9: footprint TO_SOT_Packages_SMD:SOT-23-6 -> Package_TO_SOT_SMD:SOT-23-6
Connections:
- wire segments 98 -> 110
Other:
- note added: "TODO:\ncheck diode footprint\nAdd Electrolytic output cap (10-20uF)"
- note removed: "TODO:\nUpdate Diode Footprint"

Commit message: BMS controller. Lots of new FW including bootloaders
Parts:
- removed C104: 100nF, Capacitor_SMD:C_1206_3216Metric, symbol Device:C
- removed C105: 100nF, Capacitor_SMD:C_0805_2012Metric, symbol Device:C
- removed C19: 500nF, Capacitor_SMD:C_0603_1608Metric, symbol Device:C
- removed C20: 280pF, Capacitor_SMD:C_0603_1608Metric, symbol Device:C
- removed D8: D_TVS, symbol Device:D_TVS
- removed L7: Ferrite_Bead, Inductor_SMD:L_0603_1608Metric, symbol Device:Ferrite_Bead
- removed R193: 100R, Resistor_SMD:R_0603_1608Metric, symbol Device:R
- removed R7: 176k, Resistor_SMD:R_0603_1608Metric, symbol Device:R
- removed U2: TPS73633DBV, Package_TO_SOT_SMD:SOT-23-5, symbol Regulator_Linear:TPS73633DBV
- added C108, C109, C111, C112: 100nF, Capacitor_SMD:C_0603_1608Metric, symbol Device:C
- added D8: D_TVS, Diode_SMD:D_SMB, symbol Device:D_Zener
- added Q32, Q33: Q_DUAL_NMOS_PMOS, Package_TO_SOT_SMD:SOT-363_SC-70-6, symbol ICs:Q_DUAL_NMOS_PMOS
- added R102, R267, R274, R279, R280, R66, R86: 10k0, Resistor_SMD:R_0603_1608Metric, symbol Device:R
- added R230: 499k, Resistor_SMD:R_0603_1608Metric, symbol Device:R
- added R82, R98: 100R, Resistor_SMD:R_0603_1608Metric, symbol Device:R
- added U12: TLX9185A(GBTPL,F, Package_SO:SO-4_4.4x3.9mm_P2.54mm, symbol Isolator:SFH617A-1
- added U2: LM2931-5.0_SO8, Package_SO:SOIC-8_3.9x4.9mm_P1.27mm, symbol Regulator_Linear:LM2931-5.0_SO8
- C103, C97: value C -> 100nF; Digikey_PN (none) -> 490-4779-1-ND; MPN (none) -> GCM188R71H104KA57D; Part Number (none) -> GCM188R71H104KA57D
- C12, C17: value 10uF -> 100nF; Digikey_PN (none) -> 445-5851-1-ND; MPN (none) -> CGA5L3X7R2E104K160AA; Part Number (none) -> CGA5L3X7R2E104K160AA
- C13, C15: Digikey_PN (none) -> 445-5851-1-ND; MPN (none) -> CGA5L3X7R2E104K160AA; Part Number (none) -> CGA5L3X7R2E104K160AA
- C14, C18: value 10uF -> 100nF; footprint Capacitor_SMD:C_1206_3216Metric -> Capacitor_SMD:C_0603_1608Metric; Digikey_PN (none) -> 490-4779-1-ND; MPN (none) -> GCM188R71H104KA57D; Part Number (none) -> GCM188R71H104KA57D
- C16: value 1uF -> 100nF; footprint Capacitor_SMD:C_2220_5650Metric -> Capacitor_SMD:C_1206_3216Metric; Digikey_PN (none) -> 445-5851-1-ND; MPN (none) -> CGA5L3X7R2E104K160AA; Part Number (none) -> CGA5L3X7R2E104K160AA
- C21: value C -> 18pF; Digikey_PN (none) -> 445-5631-1-ND; MPN (none) -> CGA3E2C0G1H180J080AA; Part Number (none) -> CGA3E2C0G1H180J080AA
- C22, C23: Digikey_PN (none) -> 1276-6797-1-ND; MPN (none) -> CL31B106KOHVPNE; Part Number (none) -> CL31B106KOHVPNE
- C24: Digikey_PN (none) -> 490-4779-1-ND; MPN (none) -> GCM188R71H104KA57D; Part Number (none) -> GCM188R71H104KA57D
- C25: Digikey_PN (none) -> 490-4781-1-ND; MPN (none) -> GCM188R72A103KA37D; Part Number (none) -> GCM188R72A103KA37D
- D4: footprint Diode_SMD:D_SOD-123F -> Diode_SMD:D_SMA; Digikey_PN (none) -> 497-7545-1-ND; MPN ACDBMT1200-HF -> STPS1150A; Part Number (none) -> STPS1150A
- L2, L8: Digikey_PN (none) -> 732-1591-1-ND; MPN (none) -> 742792609; Part Number (none) -> 742792609
- L3: Digikey_PN (none) -> 240-2742-1-ND; Part Number (none) -> TYS6045221M-10
- R199: Digikey_PN (none) -> YAG3561CT-ND; Part Number (none) -> AC0603FR-07100RL
- R200, R201: DNP (none) -> < ... >; Digikey_PN (none) -> 311-10KLDCT-ND; MPN (none) -> AC0603FR-0710KL; Part Number (none) -> AC0603FR-0710KL
- R202: value R -> 3R3; Digikey_PN (none) -> RHM303DCT-ND; MPN (none) -> ESR03EZPJ3R3; Part Number (none) -> ESR03EZPJ3R3
- R4: value 1M49 -> 1M; DNP (none) -> < ... >; Digikey_PN (none) -> 311-1MLDCT-ND; MPN (none) -> AC0603FR-071ML; Part Number (none) -> AC0603FR-071ML
- R5: Digikey_PN (none) -> 2019-RN73R1JTTD3202B25CT-ND; MPN (none) -> RN73R1JTTD3202B25; Part Number (none) -> RN73R1JTTD3202B25
- R6: Digikey_PN (none) -> RMCF0603FT13K0CT-ND; MPN (none) -> RMCF0603FT13K0; Part Number (none) -> RMCF0603FT13K0
- R8: Digikey_PN (none) -> RHM303DCT-ND; MPN (none) -> ESR03EZPJ3R3; Part Number (none) -> ESR03EZPJ3R3
- U3: Alternate (none) -> TLV733P-Q1; Digikey_PN (none) -> 296-TLV73330PQDBVRQ1CT-ND; Part Number (none) -> TLV733P-Q1
- U4: Part Number (none) -> LTC3638
- U9: Alternate (none) -> AP22652W6-7; Digikey_PN (none) -> 31-AP22652AW6-7CT-ND; Part Number (none) -> AP22652W6-7
Connections:
- net labels added: +3.3VA, +5VA, +5VL, 12V_POWER, 12V_POWER_STATUS, 5V_N_SW_EN, GND1, HV_VBATT_FILT_5V_IN
- net labels removed: +3.3VP, VBATT_FILT_5V_IN
- wire segments 110 -> 141
Other:
- note added: "3V3 Switched"
- note added: "5V Comms"
- note added: "5V Switched"
- note added: "Do Not populate R280"
- note added: "LOW VOLTAGE DOMAIN"
- note added: "Vin_HV: 40V - 140V\nVout: 5V\nSwitching Freq: 100kHz\nRMS Current: 200mA\nSoftStart 1mS"
- note removed: "3V3 Switched (External)"
- note removed: "TODO:\ncheck diode footprint\nAdd Electrolytic output cap (10-20uF)"
- note removed: "Vin_HV: 40V - 140V\nVout: 5V\nSwitching Freq: 100kHz\nRMS Current: 200mA\nSoftStart 100mS"
- moved on the sheet: U3
