File: Hardware/BMS/BMS_01/TempSensors.sch (KiCad schematic (older format))
At the start: 0 parts

Commit message: Too much stuff to list
Connections:
- net labels added: NTC_10_AI, NTC_10_OUT, NTC_10_RTN, NTC_11_AI, NTC_11_OUT, NTC_11_RTN, NTC_12_AI, NTC_12_OUT, NTC_12_RTN, NTC_13_AI, NTC_13_OUT, NTC_13_RTN, NTC_14_AI, NTC_14_OUT, NTC_14_RTN, NTC_15_AI, NTC_15_OUT, NTC_15_RTN, NTC_16_AI, NTC_16_OUT, NTC_16_RTN, NTC_17_AI, NTC_17_OUT, NTC_17_RTN, NTC_18_AI, NTC_18_OUT, NTC_18_RTN, NTC_19_AI, NTC_19_OUT, NTC_19_RTN, NTC_1_AI, NTC_1_OUT, NTC_1_RTN, NTC_20_AI, NTC_20_OUT, NTC_20_RTN, NTC_21_AI, NTC_21_OUT, NTC_21_RTN, NTC_22_AI, NTC_22_OUT, NTC_22_RTN, NTC_23_AI, NTC_23_OUT, NTC_23_RTN, NTC_24_AI, NTC_24_OUT, NTC_24_RTN, NTC_2_AI, NTC_2_OUT, NTC_2_RTN, NTC_3_AI, NTC_3_OUT, NTC_3_RTN, NTC_4_AI, NTC_4_OUT, NTC_4_RTN, NTC_5_AI, NTC_5_OUT, NTC_5_RTN, NTC_6_AI, NTC_6_OUT, NTC_6_RTN, NTC_7_AI, NTC_7_OUT, NTC_7_RTN, NTC_8_AI, NTC_8_OUT, NTC_8_RTN, NTC_9_AI, NTC_9_OUT, NTC_9_RTN
- wire segments 40 -> 120

Commit message: BMS controller. Lots of new FW including bootloaders
Connections:
- net labels added: +3.3VA, GND
- net labels removed: +3.3VP, NTC_10_RTN, NTC_11_RTN, NTC_12_RTN, NTC_13_RTN, NTC_14_RTN, NTC_15_RTN, NTC_16_RTN, NTC_17_RTN, NTC_18_RTN, NTC_19_RTN, NTC_1_RTN, NTC_20_RTN, NTC_21_RTN, NTC_22_RTN, NTC_23_RTN, NTC_24_RTN, NTC_2_RTN, NTC_3_RTN, NTC_4_RTN, NTC_5_RTN, NTC_6_RTN, NTC_7_RTN, NTC_8_RTN, NTC_9_RTN
- wire segments 120 -> 123
