File: Hardware/BMS/BMS_01/TopLevel.sch (KiCad schematic (older format))
At the start: 7 parts

Commit message: created HV penthouse. Complete Battery Assembly
Parts:
- added R22, R30: 100R, Resistor_SMD:R_0603_1608Metric, symbol Device:R
- added R26: 20R, Resistor_SMD:R_0603_1608Metric, symbol Device:R
- added SYM1: SYM_Flash_Small, Symbol:Symbol_HighVoltage_Type2_CopperTop_VerySmall, symbol Graphic:SYM_Flash_Large
- D1, D2, D3: footprint Diodes_SMD:D_SOD-123F -> Diode_SMD:D_SOD-123F; symbol device:D -> Device:D; MPN (none) -> RS1GFA
- R189, R191, R192: footprint Footprints:R_0603_Standard -> Resistor_SMD:R_0603_1608Metric; symbol device:R -> Device:R; MPN (none) -> AC0603FR-07100RL
- R190: value 100R -> 20R; footprint Footprints:R_0603_Standard -> Resistor_SMD:R_0603_1608Metric; symbol device:R -> Device:R
Connections:
- net labels added: BANK_00
- wire segments 52 -> 60

Commit message: BMS controller. Lots of new FW including bootloaders
Parts:
- removed R189, R191, R192: 100R, Resistor_SMD:R_0603_1608Metric, symbol Device:R
- removed R190: 20R, Resistor_SMD:R_0603_1608Metric, symbol Device:R
- removed SYM1: SYM_Flash_Small, Symbol:Symbol_HighVoltage_Type2_CopperTop_VerySmall, symbol Graphic:SYM_Flash_Large
- added C125, C126, C128, C135, C137: 10nF, Capacitor_SMD:C_0603_1608Metric, symbol Device:C
- added D31: D_Schottky, Diode_SMD:D_SOD-123F, symbol Device:D_Schottky
- added H1, H2, H3, H4, H5: MountingHole_Pad, Footprints:MountingHole_3.2mm_M3_Pad_Via, symbol Mechanical:MountingHole_Pad
- added Q60: Q_NPN_BEC, Package_TO_SOT_SMD:SOT-23, symbol Device:Q_NPN_BEC
- added Q61: Q_NMOS_GSD, Package_TO_SOT_SMD:SOT-23, symbol Device:Q_NMOS_GSD
- added Q62: Q_PNP_BEC, Package_TO_SOT_SMD:SOT-23, symbol Device:Q_PNP_BEC
- added R12: 1M, Resistor_SMD:R_0603_1608Metric, symbol Device:R
- D1, D2, D3: value D -> D_Schottky; symbol Device:D -> Device:D_Schottky; Digikey_PN (none) -> S215FACT-ND; Part Number (none) -> RS1GFA
- R22: value 100R -> 1k8; Digikey_PN (none) -> RMCF0603JG1K80CT-ND; MPN AC0603FR-07100RL -> RMCF0603JG1K80; Part Number (none) -> RMCF0603JG1K80
- R26: value 20R -> 100R; Digikey_PN (none) -> YAG3561CT-ND; MPN (none) -> AC0603FR-07100RL; Part Number (none) -> AC0603FR-07100RL
- R30: value 100R -> 2k2; Digikey_PN (none) -> RMCF0603FT2K20CT-ND; MPN AC0603FR-07100RL -> RMCF0603FT2K20; Part Number (none) -> RMCF0603FT2K20
Connections:
- net labels added: GND1, SPI_MIPO, SPI_MOPI, vreg_s2, wd_s2
- net labels removed: BANK_00, SPI_SDI, SPI_SDO
- wire segments 60 -> 78
- no-connect marks 4 -> 1
