File: Hardware/BMS/BMS_02/ChargerAndDCDC.kicad_sch (KiCad schematic)
At the start: 114 parts, among them Q16 Q_Dual_NMOS_S1G1D2S2G2D1, Q31 Q_Dual_NMOS_S1G1D2S2G2D1, Q37 Q_NMOS_GSD, Q38 Q_PMOS_GSD, Q40 Q_Dual_NPN_PNP_E1B1C2E2B2C1, Q41 Q_NMOS_GSD, Q42 NTB5D0N15MC, Q43 NTB5D0N15MC, Q44 Q_DUAL_NMOS_PMOS, Q45 NTB5D0N15MC, Q46 NTB5D0N15MC, Q47 NTB5D0N15MC, Q48 NTB5D0N15MC, Q49 NTB5D0N15MC, Q50 NTB5D0N15MC, Q52 Q_Dual_NPN_PNP_E1B1C2E2B2C1, Q53 Q_NMOS_GSD, Q54 Q_DUAL_NMOS_PMOS, Q55 TPH3300CNH,L1Q, Q56 TPH3300CNH,L1Q, U18 FAN3216TMX-F085, U19 ACS72981LLRATR-100B5, U20 CT415-HSN820DR, U21 LMV393

Commit message: bms 02 build and code bring up. Board is built, bootloader is stable and uploads app flawlessly.
Parts:
- removed C121: 4u7, Capacitor_SMD:C_1206_3216Metric, symbol Device:C
- removed C131: 100nF, Capacitor_SMD:C_0603_1608Metric, symbol Device:C
- removed D14: 12V, Diode_SMD:D_SOD-323F, symbol Device:D_Zener
- removed D17, D19: (no value), symbol Device:D_Schottky_Dual_Series_AKC
- removed D20: D_Schottky, Diode_SMD:D_SMA, symbol Device:D_Schottky
- removed Q16, Q31: Q_Dual_NMOS_S1G1D2S2G2D1, Package_TO_SOT_SMD:SOT-23-6, symbol Device:Q_Dual_NMOS_S1G1D2S2G2D1
- removed Q37, Q41, Q53: Q_NMOS_GSD, Package_TO_SOT_SMD:SOT-23, symbol Device:Q_NMOS_GSD
- removed Q38: Q_PMOS_GSD, Package_TO_SOT_SMD:SOT-23, symbol Device:Q_PMOS_GSD
- removed Q40, Q52: Q_Dual_NPN_PNP_E1B1C2E2B2C1, Package_TO_SOT_SMD:SOT-363_SC-70-6, symbol Device:Q_Dual_NPN_PNP_E1B1C2E2B2C1
- removed R209, R212: 100k, Resistor_SMD:R_0603_1608Metric, symbol Device:R
- removed R210, R211, R214, R215, R241, R242, R243, R244, R245: 1k, Resistor_SMD:R_0603_1608Metric, symbol Device:R
- removed R213: 499k, Resistor_SMD:R_0603_1608Metric, symbol Device:R
- removed R216: 100R, Resistor_SMD:R_0603_1608Metric, symbol Device:R
- removed R223, R225, R229: 3R3, Resistor_SMD:R_0603_1608Metric, symbol Device:R
- removed R239, R240, R268: 51k0, Resistor_SMD:R_0805_2012Metric, symbol Device:R
- removed U18: FAN3216TMX-F085, Package_SO:SOIC-8_3.9x4.9mm_P1.27mm, symbol ICs:FAN3216TMX-F085
- added D14: D_Schottky, Diode_SMD:D_SOD-123F, symbol Device:D_Schottky
- added U18, U22: LTC7001, Package_SO:MSOP-10-1EP_3x3mm_P0.5mm_EP1.68x1.88mm_ThermalVias, symbol ICs:LTC7001
- C104, C107: footprint Capacitor_SMD:C_1206_3216Metric -> Capacitor_SMD:C_0603_1608Metric; Digikey_PN 445-5851-1-ND -> 490-4779-1-ND; MPN CGA5L3X7R2E104K160AA -> GCM188R71H104KA57D; Part Number CGA5L3X7R2E104K160AA -> GCM188R71H104KA57D
- C105: value 100nF -> 10uF; Digikey_PN 445-5851-1-ND -> 1276-6797-1-ND; MPN CGA5L3X7R2E104K160AA -> CL31B106KOHVPNE; Part Number CGA5L3X7R2E104K160AA -> CL31B106KOHVPNE
- C110: value 4u7 -> 1uF; footprint Capacitor_SMD:C_1206_3216Metric -> Capacitor_SMD:C_0603_1608Metric; Digikey_PN 445-172481-1-ND -> 445-12539-1-ND; MPN CGA5L3X7R1H475K160AE -> (none); Part Number CGA5L3X7R1H475K160AE -> CGA3E1X7R1C105K080AC; populate y -> (none)
- D16: footprint Diode_SMD:D_SMA -> Diode_SMD:D_SOD-123F; Digikey_PN 497-7545-1-ND -> S215FACT-ND; MPN STPS1150A -> RS1GFA; Part Number STPS1150A -> RS1GFA
- Q42, Q43, Q45, Q46, Q47, Q48, Q49, Q50: Digikey_PN (none) -> 488-NTB5D0N15MCCT-ND
- Q55, Q56: footprint Package_SO:PowerPAK_SO-8_Single -> Footprints:POWER_SO8
- R14, R20, R217, R237, R255, R270, R271, R272, R275, R276, R277: DNP < ... > -> (none)
- R191: value 1k -> 10k0; Digikey_PN RMCF0603FT1K00CT-ND -> 311-10KLDCT-ND; MPN RMCF0603FT1K00 -> AC0603FR-0710KL; Part Number RMCF0603FT1K00 -> AC0603FR-0710KL
- R207: value 51k0 -> 10k0; footprint Resistor_SMD:R_0805_2012Metric -> Resistor_SMD:R_0603_1608Metric; Digikey_PN RMCF0805JT51K0CT-ND -> 311-10KLDCT-ND; MPN RMCF0805JT51K0 -> AC0603FR-0710KL; Part Number RMCF0805JT51K0 -> AC0603FR-0710KL
- U19: Digikey_PN (none) -> 620-ACS72981LLRATR-100B5CT-ND; MPN (none) -> ACS72981LLRATR-100B5
- U20: Digikey_PN (none) -> 620-CT415-HSN820DRCT-ND; MPN (none) -> CT415-HSN820DR
- U21: MPN (none) -> LMV393MX/NOPB
Connections:
- net HV_cp_s1 is gone; now on net +5VA: C104.1
- net HV_cp_s3 is gone; now on net +5VA: C107.1
- net HV_ev_signal is gone; now on an unnamed net: D16.2 (A)
- net +5VA: now also C119.1, U18.1 (VCC), U22.1 (VCC)
- net +BATT: no longer C110.1, C119.1
- net DCDC_ENABLE: now also R207.1
- net EV_CHARGER_ENABLE: now also R191.1
- net GND: now also C104.2, C107.2, C119.2, U18.11 (GND), U18.2 (Vcc_UV), U18.3 (GND), U18.5 (OVLO), U22.11 (GND), U22.2 (Vcc_UV), U22.3 (GND), U22.5 (OVLO)
- net HV_dcdc_source: now also C110.2, U22.8 (TS)
- net HV_ev_source: now also C105.2, U18.8 (TS)
- net at Q44.1, R14.1, R190.1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: now also D14.1 (K)
- net at Q54.1, R20.1, R224.1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: now also D16.1 (K)
- net at R207.2: now also U22.4 (INP)
- net +3V3: no longer names the net of R191.2
- net +3V3: now also D14.2 (A), U18.4 (INP)
- removed net HV_CHARGEPUMP_POWER: C110.2, R207.1
- net HV_DCDC_gate_r: no longer names the net of R247.1, R248.1
- net HV_DCDC_gate_r: now also U22.6 (TGUP), U22.7 (TGDN)
- net HV_cp_s2: no longer names the net of C105.1
- net HV_cp_s2: now also U18.9 (BST)
- net HV_ev_g_R: no longer names the net of R218.1, R220.1
- net HV_ev_g_R: now also U18.6 (TGUP), U18.7 (TGDN)
- new net: C110.1, U22.9 (BST)
Other:
- note added: "DNP"
- note removed: "Charge Pump Batt + 10V"
- moved on the sheet: D25, Q55, Q56, R247, R248, R250, R251
